File: armboard/REV2/arm-board-rev2.sch (EAGLE design)
At the start: 55 parts, among them J2_12V ANDERSON_POWERPOLEPP45_PCB_HO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, J2_GND ANDERSON_POWERPOLEPP45_PCB_HO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, X1 53261-06

Commit message: moved some stuff around
Connections:
- net +5V: no longer PWR_MAIN5V.P$1
Other:
- moved on the sheet: J2_12V, J2_GND, PWR_MAIN12V, PWR_MAIN5V, PWR_MAINGND
Changed lines of the file:
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@@
 <part name="GND28" library="SparkFun-Aesthetics" deviceset="GND" device=""/>
 <part name="P+12" library="supply1" deviceset="+12V" device=""/>
+<part name="P+13" library="supply1" deviceset="+5V" device=""/>
 </parts>
 <sheets>
@@
 <description>Power</description>
 <plain>
-<wire x1="71.12" y1="55.88" x2="71.12" y2="25.4" width="0.1524" layer="97" style="shortdash"/>
-<wire x1="71.12" y1="25.4" x2="48.26" y2="25.4" width="0.1524" layer="97" style="shortdash"/>
+<wire x1="101.6" y1="55.88" x2="101.6" y2="25.4" width="0.1524" layer="97" style="shortdash"/>
+<wire x1="101.6" y1="25.4" x2="48.26" y2="25.4" width="0.1524" layer="97" style="shortdash"/>
 <wire x1="48.26" y1="25.4" x2="48.26" y2="55.88" width="0.1524" layer="97" style="shortdash"/>
-<wire x1="48.26" y1="55.88" x2="71.12" y2="55.88" width="0.1524" layer="97" style="shortdash"/>
-<wire x1="76.2" y1="55.88" x2="76.2" y2="25.4" width="0.1524" layer="97" style="shortdash"/>
-<wire x1="76.2" y1="25.4" x2="93.98" y2="25.4" width="0.1524" layer="97" style="shortdash"/>
-<wire x1="93.98" y1="25.4" x2="93.98" y2="55.88" width="0.1524" layer="97" style="shortdash"/>
-<wire x1="93.98" y1="55.88" x2="76.2" y2="55.88" width="0.1524" layer="97" style="shortdash"/>
-<text x="53.34" y="55.88" size="1.778" layer="97">MAIN POWER</text>
-<text x="81.28" y="55.88" size="1.778" layer="97">J2 POWER</text>
+<wire x1="48.26" y1="55.88" x2="101.6" y2="55.88" width="0.1524" layer="97" style="shortdash"/>
+<wire x1="-25.4" y1="-5.08" x2="-25.4" y2="-35.56" width="0.1524" layer="97" style="shortdash"/>
+<wire x1="-25.4" y1="-35.56" x2="-7.62" y2="-35.56" width="0.1524" layer="97" style="shortdash"/>
+<wire x1="-7.62" y1="-35.56" x2="-7.62" y2="-5.08" width="0.1524" layer="97" style="shortdash"/>
+<wire x1="-7.62" y1="-5.08" x2="-25.4" y2="-5.08" width="0.1524" layer="97" style="shortdash"/>
+<text x="83.82" y="55.88" size="1.778" layer="97">MAIN POWER</text>
+<text x="-20.32" y="-5.08" size="1.778" layer="97">J2 POWER</text>
 <wire x1="71.12" y1="7.62" x2="71.12" y2="-48.26" width="0.1524" layer="97" style="shortdash"/>
 <wire x1="71.12" y1="-48.26" x2="-5.08" y2="-48.26" width="0.1524" layer="97" style="shortdash"/>
@@
 <wire x1="-5.08" y1="7.62" x2="71.12" y2="7.62" width="0.1524" layer="97" style="shortdash"/>
 <wire x1="76.2" y1="7.62" x2="76.2" y2="-48.26" width="0.1524" layer="97" style="shortdash"/>
-<wire x1="76.2" y1="-48.26" x2="132.08" y2="-48.26" width="0.1524" layer="97" style="shortdash"/>
-<wire x1="132.08" y1="-48.26" x2="132.08" y2="7.62" width="0.1524" layer="97" style="shortdash"/>
-<wire x1="132.08" y1="7.62" x2="76.2" y2="7.62" width="0.1524" layer="97" style="shortdash"/>
+<wire x1="76.2" y1="-48.26" x2="149.86" y2="-48.26" width="0.1524" layer="97" style="shortdash"/>
+<wire x1="149.86" y1="-48.26" x2="149.86" y2="7.62" width="0.1524" layer="97" style="shortdash"/>
+<wire x1="149.86" y1="7.62" x2="76.2" y2="7.62" width="0.1524" layer="97" style="shortdash"/>
 <text x="35.56" y="7.62" size="1.778" layer="97">SOLENOID POWER</text>
 <text x="99.06" y="7.62" size="1.778" layer="97">END EFFECTOR POWER</text>
@@
 <instance part="GND2" gate="1" x="10.16" y="17.78"/>
 <instance part="P+2" gate="1" x="53.34" y="48.26"/>
-<instance part="P+3" gate="1" x="58.42" y="50.8"/>
-<instance part="GND13" gate="1" x="58.42" y="30.48"/>
+<instance part="P+3" gate="1" x="88.9" y="50.8"/>
+<instance part="GND13" gate="1" x="88.9" y="30.48"/>
 <instance part="P+4" gate="1" x="22.86" y="48.26"/>
 <instance part="DECAP" gate="G$1" x="22.86" y="38.1"/>
@@
 <instance part="P+14" gate="1" x="58.42" y="2.54"/>
 <instance part="P+15" gate="1" x="88.9" y="2.54"/>
-<instance part="P+10" gate="1" x="88.9" y="50.8"/>
-<instance part="GND9" gate="1" x="88.9" y="30.48"/>
+<instance part="P+10" gate="1" x="-12.7" y="-10.16"/>
+<instance part="GND9" gate="1" x="-12.7" y="-30.48"/>
 <instance part="GND11" gate="1" x="88.9" y="-43.18" rot="MR0"/>
 <instance part="FET_PWRSOL" gate="G$1" x="55.88" y="-20.32"/>
@@
 <instance part="SOL-12V" gate="G$1" x="68.58" y="-27.94"/>
 <instance part="EE-12V" gate="G$1" x="78.74" y="-27.94" rot="R180"/>
-<instance part="J2_GND" gate="G$1" x="78.74" y="35.56" rot="R180"/>
-<instance part="J2_12V" gate="G$1" x="78.74" y="45.72" rot="R180"/>
-<instance part="PWR_MAIN" gate="GND" x="68.58" y="35.56"/>
-<instance part="PWR_MAIN" gate="5V" x="68.58" y="40.64"/>
-<instance part="PWR_MAIN" gate="12V" x="68.58" y="45.72"/>
+<instance part="J2_GND" gate="G$1" x="-22.86" y="-25.4" rot="R180"/>
+<instance part="J2_12V" gate="G$1" x="-22.86" y="-15.24" rot="R180"/>
+<instance part="PWR_MAIN" gate="GND" x="99.06" y="35.56"/>
+<instance part="PWR_MAIN" gate="5V" x="99.06" y="40.64"/>
+<instance part="PWR_MAIN" gate="12V" x="99.06" y="45.72"/>
 <instance part="P+12" gate="1" x="10.16" y="48.26"/>
 </instances>
@@
 <net name="+12V" class="0">
 <segment>
-<wire x1="60.96" y1="45.72" x2="58.42" y2="45.72" width="0.1524" layer="91"/>
+<wire x1="91.44" y1="45.72" x2="88.9" y2="45.72" width="0.1524" layer="91"/>
 <pinref part="P+3" gate="1" pin="+12V"/>
-<wire x1="58.42" y1="45.72" x2="58.42" y2="48.26" width="0.1524" layer="91"/>
+<wire x1="88.9" y1="45.72" x2="88.9" y2="48.26" width="0.1524" layer="91"/>
 <pinref part="PWR_MAIN" gate="12V" pin="P$1"/>
 </segment>
@@
 </segment>
 <segment>
-<wire x1="86.36" y1="45.72" x2="88.9" y2="45.72" width="0.1524" layer="91"/>
+<wire x1="-15.24" y1="-15.24" x2="-12.7" y2="-15.24" width="0.1524" layer="91"/>
 <pinref part="P+10" gate="1" pin="+12V"/>
-<wire x1="88.9" y1="45.72" x2="88.9" y2="48.26" width="0.1524" layer="91"/>
+<wire x1="-12.7" y1="-15.24" x2="-12.7" y2="-12.7" width="0.1524" layer="91"/>
 <pinref part="J2_12V" gate="G$1" pin="P$1"/>
 </segment>
@@
 <net name="+5V" class="0">
 <segment>
-<wire x1="60.96" y1="40.64" x2="53.34" y2="40.64" width="0.1524" layer="91"/>
 <pinref part="P+2" gate="1" pin="+5V"/>
 <wire x1="53.34" y1="40.64" x2="53.34" y2="45.72" width="0.1524" layer="91"/>
-<pinref part="PWR_MAIN" gate="5V" pin="P$1"/>
 </segment>
 </net>
@@
 <segment>
 <pinref part="GND13" gate="1" pin="GND"/>
-<wire x1="58.42" y1="33.02" x2="58.42" y2="35.56" width="0.1524" layer="91"/>
-<wire x1="58.42" y1="35.56" x2="60.96" y2="35.56" width="0.1524" layer="91"/>
+<wire x1="88.9" y1="33.02" x2="88.9" y2="35.56" width="0.1524" layer="91"/>
+<wire x1="88.9" y1="35.56" x2="91.44" y2="35.56" width="0.1524" layer="91"/>
 <pinref part="PWR_MAIN" gate="GND" pin="P$1"/>
 </segment>
 <segment>
 <pinref part="GND9" gate="1" pin="GND"/>
-<wire x1="88.9" y1="33.02" x2="88.9" y2="35.56" width="0.1524" layer="91"/>
-<wire x1="88.9" y1="35.56" x2="86.36" y2="35.56" width="0.1524" layer="91"/>
+<wire x1="-12.7" y1="-27.94" x2="-12.7" y2="-25.4" width="0.1524" layer="91"/>
+<wire x1="-12.7" y1="-25.4" x2="-15.24" y2="-25.4" width="0.1524" layer="91"/>
 <pinref part="J2_GND" gate="G$1" pin="P$1"/>
 </segment>
@@
 <instance part="LT1910CAP-DYNA3" gate="G$1" x="213.36" y="-55.88"/>
 <instance part="GND28" gate="1" x="213.36" y="-48.26" rot="R180"/>
+<instance part="P+13" gate="1" x="119.38" y="43.18"/>
 </instances>
 <busses>
@@
 <pinref part="RES_LEDDYNASWD" gate="G$1" pin="2"/>
 <wire x1="119.38" y1="38.1" x2="119.38" y2="40.64" width="0.1524" layer="91"/>
-<label x="119.38" y="40.64" size="1.016" layer="95" rot="R90" xref="yes"/>
-</segment>
-<segment>
+<pinref part="P+13" gate="1" pin="+5V"/>
+</segment>
+<segment>

Commit message: finished design (not incl current sense), needs placement/routing
Parts:
- removed H1, H2: MOUNT-HOLE3.2, holes:MOUNT-HOLE3.2
- removed TRISTATEBUFFER: SN74LS241DW, 74LS241:SN74LS241DW
- removed X1: 53261-06, con-molex:53261-06
- removed XB: XBEE-1B3, SparkFun:XBEE-1B3
- removed ZENER_DYNA1, ZENER_DYNA2, ZENER_DYNA3: SMAJ5920, SparkFun-DiscreteSemi:DIODE-SCHOTTKY-MBRA140
- added FET_PWRJ2, FET_PWRMAIN: BUK9Y4R4-40EPOWER-SO8, MRDT-2015-General:BUK9Y4R4-40EPOWER-SO8
- added J2_DATA: M06, MRDT-Connectors:M06
- added LED_PWR1: RED, SparkFun-LED:LED1206
- added LT1910-J2, LT1910-MAIN: LT1910, Jake:LT1910
- added LT1910CAP-EE1, LT1910CAP-EE2: .1µF, SparkFun-Capacitors:CAP1206
- added RES_LEDPWR1: 390, SparkFun-Passives:RESISTOR1206
- added U$2: XBEE_802.15.4PTH, MRDT-RF:XBEE_802.15.4PTH
- added U$3: MOUNTING_HOLE#6, MRDT-Hardware:MOUNTING_HOLE#6
- DECAP: value (none) -> 1uF
- ENC_EI, ENC_EO, ENC_J1, ENC_J2, ENC_WI, ENC_WO: value 53261-03 -> M03; device con-molex:53261-03 -> MRDT-Connectors:M03
- LED_PWR: value RED -> YELLOW
- LED_XB_RX: value RED -> GREEN
- LED_XB_TX: value GREEN -> RED
- LT1910CAP-DYNA1, LT1910CAP-DYNA2, LT1910CAP-DYNA3, LT1910CAP-EE, LT1910CAP-SOL: device resistor:C-USC1206 -> SparkFun-Capacitors:CAP1206
- RES_LEDDYNASWD, RES_LEDXBRX, RES_LEDXBTX: value 1k -> 220
Connections:
- removed net DYNA_RX: TRISTATEBUFFER.1Y1, U$1.PC4
- removed net DYNA_TX: TRISTATEBUFFER.2A4, U$1.PC5
- removed net TRI_EN: TRISTATEBUFFER.~1G, TRISTATEBUFFER.~2G, U$1.PB2
- removed net XB_DIO11: XB.DIO11
- removed net XB_DIO12: XB.DIO12
- removed net XB_DIO9: XB.DIO9
- removed net XB_RES1: XB.RES@8
- removed net XB_RES2: XB.RES@14
- removed net XB_RSSI: XB.RSSI
- removed net XB_RX: LED_XB_RX.C, U$1.PC6, XB.DOUT
- removed net XB_TX: LED_XB_TX.C, U$1.PC7, XB.DIN
- removed net XB_XRESET: XB.RESET
- new net GATE-J2: FET_PWRJ2.G, LT1910-J2.GATE
- new net GATE-MAIN: FET_PWRMAIN.G, LT1910-MAIN.GATE
- new net N$5: LED_PWR1.A, RES_LEDPWR1.1
- new net RC1_TO_J2: U$1.PK5
- new net RX_FROM_J2_RS232: U$1.PK0
- new net RX_FROM_J2_TTL: U$1.PA4
- new net RX_FROM_XB: LED_XB_RX.C, U$1.PC6, U$2.DOUT
- new net SIG_J2: LT1910-J2.IN
- new net SIG_MAIN: LT1910-MAIN.IN
- new net SOURCE-J2: FET_PWRJ2.S, J2_12V.P$1
- new net SOURCE-MAIN: FET_PWRMAIN.S, PWR_MAIN12V.P$1
- new net TX_TO_DYNA: DYNA1.DATA, DYNA2.DATA, DYNA3.DATA, U$1.PC4, U$1.PC5
- new net TX_TO_J2_RS232: U$1.PK1
- new net TX_TO_J2_TTL: U$1.PA5
- new net TX_TO_XB: LED_XB_TX.C, U$1.PC7, U$2.DIN
- new net XB_PWM0: U$2.RSSI/PWM0
- new net XB_PWM1: U$2.PWM1
- new net XB_RESET: U$2.RESET
- net +12V: now also FET_PWRJ2.D, FET_PWRMAIN.D, LT1910-J2.SENSE, LT1910-J2.V+, LT1910-MAIN.SENSE, LT1910-MAIN.V+, LT1910CAP-EE1.2, LT1910CAP-EE2.2, RES_LEDPWR1.2; no longer J2_12V.P$1, PWR_MAIN12V.P$1
- net +3V3: now also U$2.VCC, U$2.VREF; no longer XB.VDD
- net +5V: now also ENC_EI.1, ENC_EO.1, ENC_J1.1, ENC_J2.1, ENC_WI.1, ENC_WO.1; no longer ENC_EI-1.S, ENC_EO-1.S, ENC_J1-1.S, ENC_J2-1.S, ENC_WI-1.S, ENC_WO-1.S, TRISTATEBUFFER.VCC
- net DYNA_SWD: no longer DYNA1.3, DYNA2.3, DYNA3.3, TRISTATEBUFFER.1A1, TRISTATEBUFFER.2Y4, ZENER_DYNA1.C, ZENER_DYNA2.C, ZENER_DYNA3.C
- net ENC_EI: now also ENC_EI.2; no longer ENC_EI-2.S
- net ENC_EO: now also ENC_EO.2; no longer ENC_EO-2.S
- net ENC_J1: now also ENC_J1.2; no longer ENC_J1-2.S
- net ENC_J2: now also ENC_J2.2; no longer ENC_J2-2.S
- net ENC_WI: now also ENC_WI.2; no longer ENC_WI-2.S
- net ENC_WO: now also ENC_WO.2; no longer ENC_WO-2.S
- net GATE-EE: now also FET_PWREE.G
- net GATE-SOL: now also FET_PWRSOL.G
- net GND: now also DYNA1.GND, DYNA2.GND, DYNA3.GND, ENC_EI.3, ENC_EO.3, ENC_J1.3, ENC_J2.3, ENC_WI.3, ENC_WO.3, J2_DATA.4, LED_PWR1.C, LT1910-J2.GND, LT1910-MAIN.GND, LT1910CAP-DYNA1.1, LT1910CAP-DYNA2.1, LT1910CAP-DYNA3.1, LT1910CAP-EE1.1, LT1910CAP-EE2.1, U$2.GND; no longer DYNA1.1, DYNA2.1, DYNA3.1, ENC_EI-3.S, ENC_EO-3.S, ENC_J1-3.S, ENC_J2-3.S, ENC_WI-3.S, ENC_WO-3.S, TRISTATEBUFFER.GND, X1-4.S, XB.GND, ZENER_DYNA1.A, ZENER_DYNA2.A, ZENER_DYNA3.A
- net J2_RC1: now also J2_DATA.3; no longer U$1.PK5, X1-3.S
- net J2_RS232RX: no longer U$1.PK0
- net J2_RS232TX: no longer U$1.PK1
- net J2_TTLRX: now also J2_DATA.6; no longer U$1.PA4, X1-6.S
- net J2_TTLTX: now also J2_DATA.5; no longer U$1.PA5, X1-5.S
- net R1IN: now also J2_DATA.2; no longer X1-2.S
- net SOURCE-DYNA1: now also DYNA1.VCC; no longer DYNA1.2
- net SOURCE-DYNA2: now also DYNA2.VCC; no longer DYNA2.2
- net SOURCE-DYNA3: now also DYNA3.VCC; no longer DYNA3.2
- net T1OUT: now also J2_DATA.1; no longer X1-1.S
- net XB_CTS: now also U$2.CTS/DIO7; no longer XB.CTS
- net XB_DIO0: now also U$2.AD0/DIO0; no longer XB.DIO0
- net XB_DIO1: now also U$2.AD1/DIO1; no longer XB.DIO1
- net XB_DIO2: now also U$2.AD2/DIO2; no longer XB.DIO2
- net XB_DIO3: now also U$2.AD3/DIO3; no longer XB.DIO3
- net XB_DIO4: now also U$2.AD4/DIO4; no longer XB.DIO4
- net XB_DIO5: now also U$2.AD5/DIO5; no longer XB.DIO5
- net XB_DTR: now also U$2.DTR/DI8; no longer XB.DTR
- net XB_RTS: now also U$2.RTS/DIO6; no longer XB.RTS

Commit message: routing sucks but its done...
Parts:
- removed LED_PWR: YELLOW, SparkFun-LED:LED1206
- removed LED_PWR1: RED, SparkFun-LED:LED1206
- removed LT1910CAP-EE1, LT1910CAP-EE2: .1µF, SparkFun-Capacitors:CAP1206
- added LED_12V: YELLOW, SparkFun-LED:LED0603
- added LED_12VU: ORANGE, SparkFun-LED:LED0603
- added LED_5V: RED, SparkFun-LED:LED0603
- added LT1910CAP-J2, LT1910CAP-MAIN: .1µF, SparkFun-Capacitors:CAP0603-CAP
- added RES_LEDPWR2: 1k, SparkFun-Resistors:RESISTOR0603
- added U$4, U$5: ACS722, MRDT-PowerICs:ACS722
- LED_DYNASWD, LED_XB_RX: device SparkFun-LED:LED1206 -> SparkFun-LED:LED0603
- LED_XB_TX: device SparkFun-LED:LED-GREEN1206 -> SparkFun-LED:LED0603
- LT1910CAP-DYNA1, LT1910CAP-DYNA2, LT1910CAP-DYNA3, LT1910CAP-EE, LT1910CAP-SOL, MAX232_C1_1, MAX232_C2_1, MAX232_DECAP_1, MAX232_VNCAP_1, MAX232_VPCAP_1: device SparkFun-Capacitors:CAP1206 -> SparkFun-Capacitors:CAP0603-CAP
- RES_LEDDYNASWD: device SparkFun-Resistors:RESISTOR1206 -> SparkFun-Resistors:RESISTOR0603
- RES_LEDPWR, RES_LEDPWR1, RES_LEDXBRX, RES_LEDXBTX: device SparkFun-Passives:RESISTOR1206 -> SparkFun-Resistors:RESISTOR0603
- U$2: value XBEE_802.15.4PTH -> XBEE_802.15.4SMD; device MRDT-RF:XBEE_802.15.4PTH -> MRDT-RF:XBEE_802.15.4SMD
Connections:
- removed net DYNA_SWD: LED_DYNASWD.C
- removed net J2_RC1: J2_DATA.3
- removed net J2_RS232RX: MAX232_1.R1OUT
- removed net J2_RS232TX: MAX232_1.T1IN
- removed net J2_TTLRX: J2_DATA.6
- removed net J2_TTLTX: J2_DATA.5
- removed net SOURCE-MAIN: FET_PWRMAIN.S, PWR_MAIN12V.P$1
- new net +12V_UNREG: FET_PWRMAIN.D, LT1910-MAIN.SENSE, LT1910-MAIN.V+, LT1910CAP-MAIN.2, PWR_MAIN12V.P$1, RES_LEDPWR.2
- new net IMEAS_12V_EE: U$1.PA6, U$5.VIOUT
- new net IMEAS_12V_MAIN: U$1.PK3, U$4.VIOUT
- new net N$10: EE-12V.P$1, U$5.IP-
- new net N$6: LED_12V.A, RES_LEDPWR2.1
- new net N$7: FET_PWRMAIN.S, U$4.IP+
- net +12V: now also LT1910CAP-J2.2, RES_LEDPWR2.2, U$4.IP-; no longer FET_PWRMAIN.D, LT1910-MAIN.SENSE, LT1910-MAIN.V+, LT1910CAP-EE1.2, LT1910CAP-EE2.2, RES_LEDPWR.2, RES_LEDPWR1.2
- net +3V3: now also MAX232_1.VCC, MAX232_DECAP_1.2, RES_LEDDYNASWD.2, U$4.VCC, U$5.VCC
- net +5V: now also PWR_MAIN5V.P$1, RES_LEDPWR1.2; no longer MAX232_1.VCC, MAX232_DECAP_1.2, RES_LEDDYNASWD.2
- net ENC_EI: now also U$1.PD1
- net ENC_EO: now also U$1.PD0
- net ENC_J1: now also U$1.PM2
- net ENC_J2: now also U$1.PM1
- net ENC_WI: now also U$1.PM3
- net ENC_WO: now also U$1.PL4
- net GATE-DYNA1: now also FET_DYNA1.G
- net GATE-DYNA2: now also FET_DYNA2.G
- net GATE-DYNA3: now also FET_DYNA3.G
- net GND: now also LED_12V.C, LED_12VU.C, LED_5V.C, LT1910CAP-J2.1, LT1910CAP-MAIN.1, U$4.FILTER, U$4.GND, U$5.FILTER, U$5.GND; no longer LED_PWR.C, LED_PWR1.C, LT1910CAP-EE1.1, LT1910CAP-EE2.1
- net N$4: now also LED_12VU.A; no longer LED_PWR.A
- net N$5: now also LED_5V.A; no longer LED_PWR1.A
- net RC1_TO_J2: now also J2_DATA.3
- net RX_FROM_J2_RS232: now also MAX232_1.R1OUT
- net RX_FROM_J2_TTL: now also J2_DATA.6
- net RX_FROM_XB: now also U$1.PP0; no longer U$1.PC6
- net SIG_DYNA1: now also U$1.PK7; no longer U$1.PE2
- net SIG_EE: now also U$1.PL3; no longer U$1.PH0
- net SIG_J2: now also U$1.PP4
- net SIG_MAIN: now also U$1.PK2
- net SIG_SOL: now also U$1.PL2; no longer U$1.PH1
- net SOURCE-EE: now also U$5.IP+; no longer EE-12V.P$1
- net TX_TO_DYNA: now also LED_DYNASWD.C
- net TX_TO_J2_RS232: now also MAX232_1.T1IN
- net TX_TO_J2_TTL: now also J2_DATA.5
- net TX_TO_XB: now also U$1.PP1; no longer U$1.PC7
- net XB_CTS: now also U$1.PE5
- net XB_DIO0: now also U$1.PB3
- net XB_DIO1: now also U$1.PB2
- net XB_DIO2: now also U$1.PM5
- net XB_DIO3: now also U$1.PM4
- net XB_DIO4: now also U$1.PC6
- net XB_DIO5: now also U$1.PD3
- net XB_DTR: now also U$1.PD4
- net XB_PWM0: now also U$1.PB5
- net XB_PWM1: now also U$1.PB4
- net XB_RESET: now also U$1.PD2
- net XB_RTS: now also U$1.PC7
Other:
- moved on the sheet: EE-12V, EE-GND, PWR_MAIN12V, PWR_MAIN5V, PWR_MAINGND

Commit message: added gerbers and stuff
dims 4.9x2.2in
Parts:
- added LED_5V1: white, SparkFun-LED:LED1206
- added RES_LEDPWR3: 390, SparkFun-Resistors:RESISTOR0603
- added U$7: SWITCH_SPDT_VERTSS12D07VG4NSGAPA, MRDT-Electromechanical:SWITCH_SPDT_VERTSS12D07VG4NSGAPA
Connections:
- new net N$11: LED_5V1.A, RES_LEDPWR3.1
- new net N$12: RES_LEDPWR3.2, U$7.P
- net +5V: now also U$7.O
- net GND: now also LED_5V1.C
Changed lines of the file:
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@@
 <part name="+3V7" library="supply1" deviceset="+3V3" device=""/>
 <part name="P+11" library="supply1" deviceset="+3V3" device=""/>
+<part name="RES_LEDPWR3" library="SparkFun-Resistors" deviceset="RESISTOR" device="0603" value="390"/>
+<part name="LED_5V1" library="SparkFun-LED" deviceset="LED" device="1206" value="white"/>
+<part name="GND26" library="SparkFun" deviceset="GND" device=""/>
+<part name="P+12" library="supply1" deviceset="+5V" device=""/>
+<part name="U$7" library="MRDT-Electromechanical" deviceset="SWITCH_SPDT_VERT" device="SS12D07VG4NSGAPA"/>
 </parts>
 <sheets>
@@
 <instance part="GND10" gate="1" x="149.86" y="-119.38"/>
 <instance part="+3V7" gate="G$1" x="149.86" y="-93.98"/>
+<instance part="RES_LEDPWR3" gate="G$1" x="-76.2" y="38.1" rot="R90"/>
+<instance part="LED_5V1" gate="G$1" x="-76.2" y="27.94"/>
+<instance part="GND26" gate="1" x="-76.2" y="17.78"/>
+<instance part="P+12" gate="1" x="-78.74" y="58.42"/>
+<instance part="U$7" gate="G$1" x="-76.2" y="48.26" rot="R90"/>
 </instances>
 <busses>
@@
 <junction x="149.86" y="-114.3"/>
 </segment>
+<segment>
+<wire x1="-76.2" y1="22.86" x2="-76.2" y2="20.32" width="0.1524" layer="91"/>
+<pinref part="LED_5V1" gate="G$1" pin="C"/>
+<pinref part="GND26" gate="1" pin="GND"/>
+</segment>
 </net>
 <net name="N$4" class="0">
@@
 <pinref part="P+2" gate="1" pin="+5V"/>
 </segment>
+<segment>
+<pinref part="U$7" gate="G$1" pin="O"/>
+<pinref part="P+12" gate="1" pin="+5V"/>
+<wire x1="-78.74" y1="53.34" x2="-78.74" y2="55.88" width="0.1524" layer="91"/>
+</segment>
 </net>
 <net name="N$6" class="0">
@@
 </segment>
 </net>
+<net name="N$11" class="0">
+<segment>
+<wire x1="-76.2" y1="30.48" x2="-76.2" y2="33.02" width="0.1524" layer="91"/>
+<pinref part="RES_LEDPWR3" gate="G$1" pin="1"/>
+<pinref part="LED_5V1" gate="G$1" pin="A"/>
+</segment>
+</net>
+<net name="N$12" class="0">
+<segment>
+<pinref part="RES_LEDPWR3" gate="G$1" pin="2"/>
+<pinref part="U$7" gate="G$1" pin="P"/>
+<wire x1="-76.2" y1="45.72" x2="-76.2" y2="43.18" width="0.1524" layer="91"/>
+</segment>
+</net>
