File: armboard/REV2/arm-board-rev2.sch (EAGLE design)
At the start: 65 parts, among them J2_12V ANDERSON_POWERPOLEPP45_PCB_HO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, J2_DATA M06, J2_GND ANDERSON_POWERPOLEPP45_PCB_HO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

Commit message: reroute
Parts:
- U$7: value SWITCH_SPDT_VERTSS12D07VG4NSGAPA -> SWITCH-SPST-HORIZ; device MRDT-Electromechanical:SWITCH_SPDT_VERTSS12D07VG4NSGAPA -> MRDT-Electromechanical:SWITCH-SPST-HORIZ
Connections:
- net N$7 renamed SOURCE-MAIN
- net +5V: now also U$7.S; no longer U$7.O
- net R1IN: now also J2_DATA.1; no longer J2_DATA.2
- net RX_FROM_J2_TTL: now also J2_DATA.5; no longer J2_DATA.6
- net T1OUT: now also J2_DATA.2; no longer J2_DATA.1
- net TX_TO_J2_TTL: now also J2_DATA.6; no longer J2_DATA.5
Changed lines of the file:
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@@
 <part name="GND26" library="SparkFun" deviceset="GND" device=""/>
 <part name="P+12" library="supply1" deviceset="+5V" device=""/>
-<part name="U$7" library="MRDT-Electromechanical" deviceset="SWITCH_SPDT_VERT" device="SS12D07VG4NSGAPA"/>
+<part name="U$7" library="MRDT-Electromechanical" deviceset="SWITCH-SPST-HORIZ" device=""/>
 </parts>
 <sheets>
@@
 <instance part="LED_5V1" gate="G$1" x="-76.2" y="27.94"/>
 <instance part="GND26" gate="1" x="-76.2" y="17.78"/>
-<instance part="P+12" gate="1" x="-78.74" y="58.42"/>
+<instance part="P+12" gate="1" x="-76.2" y="58.42"/>
 <instance part="U$7" gate="G$1" x="-76.2" y="48.26" rot="R90"/>
 </instances>
@@
 </segment>
 <segment>
-<pinref part="U$7" gate="G$1" pin="O"/>
 <pinref part="P+12" gate="1" pin="+5V"/>
-<wire x1="-78.74" y1="53.34" x2="-78.74" y2="55.88" width="0.1524" layer="91"/>
+<pinref part="U$7" gate="G$1" pin="S"/>
+<wire x1="-76.2" y1="55.88" x2="-76.2" y2="53.34" width="0.1524" layer="91"/>
 </segment>
 </net>
@@
 </segment>
 </net>
-<net name="N$7" class="0">
+<net name="SOURCE-MAIN" class="0">
 <segment>
 <pinref part="FET_PWRMAIN" gate="G$1" pin="S"/>
@@
 <segment>
 <pinref part="RES_LEDPWR3" gate="G$1" pin="2"/>
+<wire x1="-76.2" y1="45.72" x2="-76.2" y2="43.18" width="0.1524" layer="91"/>
 <pinref part="U$7" gate="G$1" pin="P"/>
-<wire x1="-76.2" y1="45.72" x2="-76.2" y2="43.18" width="0.1524" layer="91"/>
 </segment>
 </net>
@@
 </plain>
 <instances>
-<instance part="GND15" gate="1" x="132.08" y="7.62"/>
+<instance part="GND15" gate="1" x="149.86" y="7.62"/>
 <instance part="MAX232_1" gate="G$1" x="78.74" y="15.24"/>
 <instance part="MAX232_C1_1" gate="G$1" x="111.76" y="35.56" rot="R270"/>
@@
 <segment>
 <pinref part="GND15" gate="1" pin="GND"/>
-<wire x1="134.62" y1="17.78" x2="132.08" y2="17.78" width="0.1524" layer="91"/>
-<wire x1="132.08" y1="17.78" x2="132.08" y2="10.16" width="0.1524" layer="91"/>
+<wire x1="134.62" y1="17.78" x2="149.86" y2="17.78" width="0.1524" layer="91"/>
+<wire x1="149.86" y1="17.78" x2="149.86" y2="10.16" width="0.1524" layer="91"/>
 <pinref part="J2_DATA" gate="G$1" pin="4"/>
 </segment>
@@
 <net name="TX_TO_J2_TTL" class="0">
 <segment>
-<wire x1="134.62" y1="15.24" x2="129.54" y2="15.24" width="0.1524" layer="91"/>
+<label x="129.54" y="12.7" size="1.016" layer="95" rot="R180" xref="yes"/>
+<pinref part="J2_DATA" gate="G$1" pin="6"/>
+<wire x1="132.08" y1="12.7" x2="129.54" y2="12.7" width="0.1524" layer="91"/>
+<wire x1="132.08" y1="12.7" x2="134.62" y2="12.7" width="0.1524" layer="91"/>
+</segment>
+</net>
+<net name="RX_FROM_J2_TTL" class="0">
+<segment>
 <label x="129.54" y="15.24" size="1.016" layer="95" rot="R180" xref="yes"/>
 <pinref part="J2_DATA" gate="G$1" pin="5"/>
-</segment>
-</net>
-<net name="RX_FROM_J2_TTL" class="0">
-<segment>
-<wire x1="134.62" y1="12.7" x2="129.54" y2="12.7" width="0.1524" layer="91"/>
-<label x="129.54" y="12.7" size="1.016" layer="95" rot="R180" xref="yes"/>
-<pinref part="J2_DATA" gate="G$1" pin="6"/>
+<wire x1="132.08" y1="15.24" x2="129.54" y2="15.24" width="0.1524" layer="91"/>
+<wire x1="132.08" y1="15.24" x2="134.62" y2="15.24" width="0.1524" layer="91"/>
 </segment>
 </net>
@@
 <segment>
 <pinref part="MAX232_1" gate="G$1" pin="T1OUT"/>
-<wire x1="106.68" y1="25.4" x2="134.62" y2="25.4" width="0.1524" layer="91"/>
+<wire x1="106.68" y1="25.4" x2="132.08" y2="25.4" width="0.1524" layer="91"/>
 <label x="124.46" y="25.4" size="1.016" layer="95"/>
-<pinref part="J2_DATA" gate="G$1" pin="1"/>
+<pinref part="J2_DATA" gate="G$1" pin="2"/>
+<wire x1="132.08" y1="25.4" x2="134.62" y2="22.86" width="0.1524" layer="91"/>
 </segment>
 </net>
@@
 <pinref part="MAX232_1" gate="G$1" pin="R1IN"/>
 <label x="124.46" y="22.86" size="1.016" layer="95"/>
-<wire x1="106.68" y1="22.86" x2="111.76" y2="22.86" width="0.1524" layer="91"/>
-<wire x1="121.92" y1="22.86" x2="111.76" y2="22.86" width="0.1524" layer="91"/>
-<wire x1="121.92" y1="22.86" x2="134.62" y2="22.86" width="0.1524" layer="91"/>
-<pinref part="J2_DATA" gate="G$1" pin="2"/>
-</segment>
-</net>
+<wire x1="132.08" y1="22.86" x2="106.68" y2="22.86" width="0.1524" layer="91"/>
+<pinref part="J2_DATA" gate="G$1" pin="1"/>
+<wire x1="132.08" y1="22.86" x2="134.62" y2="25.4" width="0.1524" layer="91"/>
+</segment>
+</net>
