File: drillboard/drill-rev-1.brd (EAGLE design)
At the start: 160 x 100 mm, 31 parts

Commit message: started placement/routing
Parts:
- removed U$10, U$11, U$12, U$2, U$4, U$7, U$8, U$9: M03VERT, MRDT-Connectors:MOLEX0436500328
- added C1, C10, C11, C3, C4, C5, C6, C7, C8, C9: 47uf, SparkFun-Passives:1210
- added M1, M2, M3, M4, T1, T2, T3, T4: M03VERT, MRDT-Connectors:MOLEX0436500328
- C2: value 33pF -> 33nF
- R10, R4: value 1K -> 3K3
- R8: value 1K -> 10k
- moved U$15 138.5 mm to (31.1, 31.1), turned to 270 degrees
- moved U$5 130.7 mm to (42.5, 0.00)
- moved U$1 105.4 mm to (23.5, 15.2), turned to 180 degrees
- moved U$6 96.6 mm to (34.3, 18.4), turned to 270 degrees
- moved U$3 93.2 mm to (32.5, 0.00)
- moved U$13 49.4 mm to (18.4, 47.6), turned to 90 degrees
Connections:
- net +12V: now also C1.1, C10.1, C11.1, C3.1, C4.1, C5.1, C6.1, C7.1, C8.1, C9.1
- net +3V3: now also M1.P$2, M2.P$2, T1.P$2, T2.P$2, T3.P$2, T4.P$2; no longer U$10.P$2, U$2.P$2, U$4.P$2, U$7.P$2, U$8.P$2, U$9.P$2
- net D1: now also M3.P$3; no longer U$11.P$3
- net D2: now also M3.P$2; no longer U$11.P$2
- net D3: now also M4.P$3; no longer U$12.P$3
- net D4: now also M4.P$2; no longer U$12.P$2
- net GND: now also C1.2, C10.2, C11.2, C3.2, C4.2, C5.2, C6.2, C7.2, C8.2, C9.2, M1.P$3, M2.P$3, T1.P$3, T2.P$3, T3.P$3, T4.P$3; no longer U$10.P$3, U$2.P$3, U$4.P$3, U$7.P$3, U$8.P$3, U$9.P$3
- net MOIST_1: now also M1.P$1; no longer U$9.P$1
- net MOIST_2: now also M2.P$1; no longer U$10.P$1
- net MOIST_3: now also M3.P$1; no longer U$11.P$1
- net MOIST_4: now also M4.P$1; no longer U$12.P$1
- net TEMP_1: now also T1.P$1; no longer U$2.P$1
- net TEMP_2: now also T2.P$1; no longer U$4.P$1
- net TEMP_3: now also T3.P$1; no longer U$7.P$1
- net TEMP_4: now also T4.P$1; no longer U$8.P$1
Routing:
- added copper zone on layer 1, net +3V3
- added copper zone on layer 16, net GND
Other:
- board size 160 x 100 mm -> 52.7 x 56.4 mm

Commit message: finished routing/placement
Parts:
- moved R13 153.4 mm to (23.6, 3.56), flipped to the bottom
- moved R12 152.0 mm to (23.6, 1.65), flipped to the bottom
- moved C11 142.0 mm to (16.9, 11.0), flipped to the bottom, turned to 270 degrees
- moved C2 139.9 mm to (21.3, 26.4), flipped to the bottom, turned to 270 degrees
- moved C10 137.8 mm to (13.7, 11.0), flipped to the bottom, turned to 270 degrees
- moved R11 136.0 mm to (33.8, 34.8), flipped to the bottom, turned to 180 degrees
- moved C1 135.0 mm to (16.9, 16.1), flipped to the bottom, turned to 90 degrees
- moved C9 133.6 mm to (10.5, 11.0), flipped to the bottom, turned to 270 degrees
- moved C3 132.5 mm to (13.7, 16.1), flipped to the bottom, turned to 90 degrees
- moved R9 130.6 mm to (33.8, 33.1), flipped to the bottom, turned to 180 degrees
- moved C4 130.1 mm to (10.5, 16.1), flipped to the bottom, turned to 90 degrees
- moved R10 130.0 mm to (30.4, 34.8), flipped to the bottom, turned to 180 degrees
- moved C8 129.4 mm to (7.37, 11.0), flipped to the bottom, turned to 270 degrees
- moved C5 127.8 mm to (7.37, 16.1), flipped to the bottom, turned to 90 degrees
- moved R7 127.5 mm to (32.1, 26.3), flipped to the bottom, turned to 90 degrees
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Connections:
- net D3: now also U$13.P$28; no longer U$13.P$10
- net INA: now also U$13.P$11; no longer U$13.P$16
- net INB: now also U$13.P$12; no longer U$13.P$17
- net MOIST_1: now also U$13.P$25; no longer U$13.P$24
- net MOIST_2: now also U$13.P$24; no longer U$13.P$25
- net PWM: now also U$13.P$13; no longer U$13.P$5
- net TEMP_1: now also U$13.P$17; no longer U$13.P$6
- net TEMP_2: now also U$13.P$16; no longer U$13.P$11
- net TEMP_3: now also U$13.P$6; no longer U$13.P$12
- net TEMP_4: now also U$13.P$5; no longer U$13.P$13
Routing:
- net MOIST_2: track 0.00 -> 56.6 mm, vias 0 -> 3
- net OUTA: track 0.00 -> 55.9 mm, vias 0 -> 6
- net OUTB: track 0.00 -> 54.6 mm, vias 0 -> 6
- net +12V: track 0.00 -> 46.5 mm
- net MOIST_1: track 0.00 -> 44.7 mm, vias 0 -> 2
- net N$2: track 0.00 -> 40.9 mm, vias 0 -> 1
- net TEMP_3: track 0.00 -> 35.1 mm, vias 0 -> 2
- net N$10: track 0.00 -> 32.5 mm, vias 0 -> 1
- net XB_DIN: track 0.00 -> 32.1 mm, vias 0 -> 1
- net XB_DOUT: track 0.00 -> 27.2 mm, vias 0 -> 1
- net MOIST_3: track 0.00 -> 26.4 mm
- net N$8: track 0.00 -> 25.1 mm, vias 0 -> 1
- net TEMP_1: track 0.00 -> 24.3 mm, vias 0 -> 2
- net TEMP_4: track 0.00 -> 21.7 mm, vias 0 -> 1
- net N$3: track 0.00 -> 20.2 mm, vias 0 -> 3
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- added copper zone on layer 1, net +12V
- added copper zone on layer 16, net +12V
- added copper zone on layer 1, net GND
- added copper zone on layer 1, net OUTA
- added copper zone on layer 16, net OUTA
- added copper zone on layer 1, net OUTB
- added copper zone on layer 16, net OUTB
Other:
- board size 52.7 x 56.4 mm -> 51.4 x 52.6 mm
