File: drillboard/REV1/drill-rev-1_p.brd (EAGLE design)
At the start: 160.7 x 52.6 mm, 123 parts, among them M1 M03VERT, M10 M03VERT, M11 M03VERT, M12 M03VERT, M2 M03VERT, M3 M03VERT, M4 M03VERT, M5 M03VERT, M6 M03VERT, M7 M03VERT, M8 M03VERT, M9 M03VERT, T1 M03VERT, T10 M03VERT, T11 M03VERT, T12 M03VERT, T2 M03VERT, T3 M03VERT, T4 M03VERT, T5 M03VERT, T6 M03VERT, T7 M03VERT, T8 M03VERT, T9 M03VERT

Commit message: regen gerbers
Changed lines of the file:
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@@
 <board>
 <plain>
-<wire x1="160.655" y1="52.6288" x2="0" y2="52.6288" width="0" layer="20"/>
-<wire x1="0" y1="52.6288" x2="0" y2="0" width="0" layer="20"/>
+<wire x1="160.655" y1="52.629" x2="0" y2="52.629" width="0" layer="20"/>
+<wire x1="0" y1="52.629" x2="0" y2="0" width="0" layer="20"/>
 <text x="13.335" y="12.7" size="1.27" layer="21" align="bottom-center">Mars Rover Design Team
 Zenith | Drill Board
@@
 <text x="98.679" y="1.524" size="1.27" layer="125" rot="R90">U$1</text>
 <text x="73.66" y="5.588" size="0.4064" layer="125" rot="R90">U$15</text>
-<wire x1="160.655" y1="0" x2="160.655" y2="52.6288" width="0" layer="20"/>
+<wire x1="160.655" y1="0" x2="160.655" y2="52.629" width="0" layer="20"/>
 <text x="122.555" y="12.7" size="1.27" layer="21" align="bottom-center">Mars Rover Design Team
 Zenith | Drill Board
@@
 <text x="153.289" y="1.524" size="1.27" layer="125" rot="R90">U$1</text>
 <text x="128.27" y="5.588" size="0.4064" layer="125" rot="R90">U$15</text>
-<dimension x1="0" y1="0" x2="160.655" y2="0" x3="80.3275" y3="-15.24" textsize="1.778" layer="47" unit="inch" precision="6" visible="yes"/>
-<dimension x1="0" y1="52.6288" x2="0" y2="0" x3="-19.685" y3="26.3144" textsize="1.778" layer="47" unit="inch" precision="6" visible="yes"/>
 </plain>
 <attributes>
