File: armboard/REV3/arm-board-rev3.sch (EAGLE design)
At the start: 59 parts, among them J2_12V ANDERSON_POWERPOLEPP45_PCB_HO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, J2_DATA M062X3VERT, J2_GND ANDERSON_POWERPOLEPP45_PCB_HO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

Commit message: working on rev3
Parts:
- added LED_12V1, LED_12V2, LED_12V3, LED_12V4: YELLOW, SparkFun-LED:LED0603
- added RES_LEDDYNASWD1, RES_LEDDYNASWD11, RES_LEDDYNASWD3, RES_LEDDYNASWD5, RES_LEDDYNASWD7, RES_LEDDYNASWD9, RES_LEDPWR4, RES_LEDPWR5, RES_LEDPWR6, RES_LEDPWR7: 1k, SparkFun-Resistors:RESISTOR0603
- added RES_LEDDYNASWD10, RES_LEDDYNASWD12, RES_LEDDYNASWD2, RES_LEDDYNASWD4, RES_LEDDYNASWD6, RES_LEDDYNASWD8: 2k, SparkFun-Resistors:RESISTOR0603
- DYNA1: value DYNAMIXEL-1X03HORIZ -> DYNAMIXEL-1X03VERT; device MRDT-2015-Arm:DYNAMIXEL-1X03HORIZ -> MRDT-2015-Arm:DYNAMIXEL-1X03VERT
- renumbered U$10 to U$9
Connections:
- removed net ENC_EI: U$1.PD1
- removed net ENC_EO: U$1.PD0
- removed net ENC_J1: U$1.PM2
- removed net ENC_J2: U$1.PM1
- removed net ENC_WI: U$1.PM3
- removed net RC1_TO_J2: J2_DATA.2, U$1.PK5
- new net N$12: LED_12V2.C, RES_LEDPWR5.2
- new net N$14: LED_12V3.C, RES_LEDPWR6.2
- new net N$15: LED_12V4.C, RES_LEDPWR7.2
- new net N$7: LED_12V1.C, RES_LEDPWR4.2
- new net RC3_TO_J2: J2_DATA.2, U$1.PD5
- new net TX_TO_DYNA1: DYNA1.DATA, U$1.PK0, U$1.PK1
- new net TX_TO_DYNA23: DYNA2.DATA, DYNA3.DATA, U$1.PC4, U$1.PC5
- new net XB_VREF: U$2.VREF
- net +12V: now also LED_12V.A; no longer RES_LEDPWR2.2
- net +12V_UNREG: now also LED_12VU.A; no longer RES_LEDPWR.2
- net +3V3: now also LED_DYNASWD.A; no longer RES_LEDDYNASWD.2, U$2.VREF
- net +5V: now also LED_5V.A; no longer RES_LEDPWR1.2
- net ENC_EI_ANA: now also RES_LEDDYNASWD10.2, RES_LEDDYNASWD9.1
- net ENC_EI_PWM: now also RES_LEDDYNASWD9.2
- net ENC_EO_ANA: now also RES_LEDDYNASWD3.1, RES_LEDDYNASWD4.2
- net ENC_EO_PWM: now also RES_LEDDYNASWD3.2
- net ENC_J1_ANA: now also RES_LEDDYNASWD1.1, RES_LEDDYNASWD2.2, U$1.PD2
- net ENC_J1_PWM: now also RES_LEDDYNASWD1.2
- net ENC_J2_ANA: now also RES_LEDDYNASWD7.1, RES_LEDDYNASWD8.2, U$1.PD4
- net ENC_J2_PWM: now also RES_LEDDYNASWD7.2
- net ENC_WI_ANA: now also RES_LEDDYNASWD11.1, RES_LEDDYNASWD12.2
- net ENC_WI_PWM: now also RES_LEDDYNASWD11.2
- net ENC_WO_ANA: now also RES_LEDDYNASWD5.1, RES_LEDDYNASWD6.2
- net ENC_WO_PWM: now also RES_LEDDYNASWD5.2
- net GND: now also RES_LEDDYNASWD10.1, RES_LEDDYNASWD12.1, RES_LEDDYNASWD2.1, RES_LEDDYNASWD4.1, RES_LEDDYNASWD6.1, RES_LEDDYNASWD8.1, RES_LEDPWR.1, RES_LEDPWR1.1, RES_LEDPWR2.1, RES_LEDPWR4.1, RES_LEDPWR5.1, RES_LEDPWR6.1, RES_LEDPWR7.1; no longer LED_12V.C, LED_12VU.C, LED_5V.C
- net IMEAS_12V_MAIN: now also U$1.PB4; no longer U$1.PK3
- net N$3: now also LED_DYNASWD.C, RES_LEDDYNASWD.2; no longer LED_DYNASWD.A, RES_LEDDYNASWD.1
- net N$4: now also LED_12V.C, RES_LEDPWR2.2; no longer LED_12VU.A, RES_LEDPWR.1
- net N$5: now also LED_12VU.C, RES_LEDPWR.2; no longer LED_5V.A, RES_LEDPWR1.1
- net N$6: now also LED_5V.C, RES_LEDPWR1.2; no longer LED_12V.A, RES_LEDPWR2.1
- net RX_FROM_J2_TTL: now also J2_DATA.4; no longer J2_DATA.3
- net SIG_DYNA1: now also U$1.PB5; no longer U$1.PK7
- net SIG_J2: now also U$1.PM0; no longer U$1.PP4
- net SIG_MAIN: now also U$1.PK7; no longer U$1.PK2
- net SOURCE-DYNA1: now also LED_12V2.A
- net SOURCE-DYNA2: now also LED_12V3.A
- net SOURCE-DYNA3: now also LED_12V4.A
- net SOURCE-J2: now also LED_12V1.A
- net TX_TO_DYNA: now also RES_LEDDYNASWD.1; no longer DYNA1.DATA, DYNA2.DATA, DYNA3.DATA, LED_DYNASWD.C, U$1.PC4, U$1.PC5
- net TX_TO_J2_TTL: now also J2_DATA.3; no longer J2_DATA.4
- net XB_CTS: no longer U$1.PE5
- net XB_DIO0: no longer U$1.PB3
- net XB_DIO1: no longer U$1.PB2
- net XB_DIO2: no longer U$1.PM5
- net XB_DIO3: no longer U$1.PM4
- net XB_DIO4: no longer U$1.PC6
- net XB_DIO5: no longer U$1.PD3
- net XB_DTR: no longer U$1.PD4
- net XB_PWM0: no longer U$1.PB5
- net XB_PWM1: no longer U$1.PB4
- net XB_RESET: no longer U$1.PD2
- net XB_RTS: no longer U$1.PC7
Other:
- note added: "DROPS PWM DOWN FROM 5V TO 3V3 IN CASE LTC2645 DOES NOT WORK"
- note removed: "replace w 2x2 microfit"
- moved on the sheet: LED_12V, LED_12VU, LED_5V, LED_5V1, LED_DYNASWD, LTC2645-CAP-IOVCC-1, LTC2645-CAP-IOVCC-2, RES_LEDDYNASWD, RES_LEDPWR, RES_LEDPWR1, RES_LEDPWR2, RES_LEDPWR3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

Commit message: finished first draft, gened gerbs
Connections:
- removed net ENC_WO: U$1.PL4
- removed net SIG_SOL: U$1.PL2
- removed net TX_TO_DYNA: RES_LEDDYNASWD.1
- net ENC_EI_ANA: now also U$1.PB3, U$1.PE3, U$11.VOUT_B; no longer U$11.VOUT_A
- net ENC_EI_PWM: now also U$11.IN_B; no longer U$11.IN_A
- net ENC_EO_ANA: now also U$1.PD7, U$11.VOUT_C; no longer U$11.VOUT_B
- net ENC_EO_PWM: now also U$11.IN_C; no longer U$11.IN_B
- net ENC_WI_ANA: now also U$1.PB2, U$1.PE5, U$11.VOUT_A; no longer U$11.VOUT_C
- net ENC_WI_PWM: now also U$11.IN_A; no longer U$11.IN_C
- net ENC_WO_ANA: now also U$1.PD3
- net IMEAS_12V_EE: now also U$1.PE2; no longer U$1.PA6
- net SIG_DYNA2: now also U$1.PE1; no longer U$1.PE3
- net SIG_DYNA3: now also U$1.PF3; no longer U$1.PD7
- net TX_TO_DYNA23: now also RES_LEDDYNASWD.1
