File: main eagle files/arm board/Arm_Board_2018.sch (EAGLE design)
At the start: 149 parts, among them Q1 Q_IRF7437SMD, U1 TIVA-1294, U4 ACS722, U5 ACS722, U6 ACS722, U7 ACS722, U8 ACS722, U9 ACS722

Commit message: Further progress
Parts:
- removed OE_PULLUP: 10K, SparkFun-Passives:RESISTOR0402-RES
Connections:
- removed net MOTOR7_POWER: C6.1, MOT7_HB.VBAT, MOT7_HB.VCC
- removed net MOTOR8_POWER: C5.1, MOT8_HB.VBAT, MOT8_HB.VCC
- removed net PWM_OUTPUT_ENABLE: OE_PULLUP.2, PWM_DRIVER.#OE
- net 12VMOTOR_POWER: now also C5.1, C6.1, MOT7_HB.VBAT, MOT7_HB.VCC, MOT8_HB.VBAT, MOT8_HB.VCC
- net BUTTON1: now also U1.PM2
- net BUTTON2: now also U1.PM1
- net BUTTON3: now also U1.PM0
- net ENCODER_1: now also U1.PL4
- net ENCODER_2: now also U1.PD2
- net ENCODER_3: now also U1.PA4
- net ENCODER_4: now also U1.PA6
- net ENCODER_5: now also U1.PM4
- net ENCODER_6: now also U1.PB2
- net GND: now also PWM_DRIVER.#OE, U1.GND
- net LED1: now also U1.PB4
- net LED2: now also U1.PB5
- net LED3: now also U1.PD4
- net LED4: now also U1.PD5
- net LED5: now also U1.PQ0
- net LED6: now also U1.PP4
- net LIMIT_SWITCH_1: now also U1.PB3
- net LIMIT_SWITCH_2: now also U1.PC7
- net LIMIT_SWITCH_3: now also U1.PD3
- net LOGIC_3.3V: now also U1.+3V3; no longer OE_PULLUP.1
- net MAINLINE_CURRENT_SENSOR: now also U1.PK3
- net MASTER_POWER_ENABLE: now also U1.PQ1
- net MOTOR1_CURRENT_SENSOR: now also U1.PK2
- net MOTOR1_INA: now also U1.PQ2/PA3
- net MOTOR1_INB: now also U1.PQ3/PA2
- net MOTOR2_CURRENT_SENSOR: now also U1.PK1
- net MOTOR2_INA: now also U1.PK4
- net MOTOR2_INB: now also U1.PK5
- net MOTOR3_CURRENT_SENSOR: now also U1.PK0
- net MOTOR3_INA: now also U1.PC4
- net MOTOR3_INB: now also U1.PC5
- net MOTOR4_CURRENT_SENSOR: now also U1.PE2
- net MOTOR4_INA: now also U1.PC6
- net MOTOR4_INB: now also U1.PE5
- net MOTOR5_CURRENT_SENSOR: now also U1.PE1
- net MOTOR5_INA: now also U1.PE3
- net MOTOR5_INB: now also U1.PM5
- net MOTOR6_CURRENT_SENSOR: now also U1.PE0
- net MOTOR6_INA: now also U1.PF1
- net MOTOR6_INB: now also U1.PF2
- net MOTOR7_INA: now also U1.PH2
- net MOTOR7_INB: now also U1.PH3
- net MOTOR8_INA: now also U1.PD1
- net MOTOR8_INB: now also U1.PD0
- net PWM_DRIVER_SCL: now also U1.PN5
- net PWM_DRIVER_SDA: now also U1.PN4
- net SWITCH: now also U1.PH0

Commit message: all things routed
Parts:
- added H1: MOUNTING_HOLE#6, MRDT-Hardware:MOUNTING_HOLE#6
- added LOGO1: MRDT_LOGO, MRDT-Hardware:MRDT_LOGO
Changed lines of the file:
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@@
 <part name="GND17" library="SparkFun-Aesthetics" deviceset="GND" device=""/>
 <part name="GND18" library="SparkFun-Aesthetics" deviceset="GND" device=""/>
+<part name="H1" library="MRDT-Hardware" deviceset="MOUNTING_HOLE" device="#6"/>
+<part name="LOGO1" library="MRDT-Hardware" deviceset="MRDT_LOGO" device=""/>
 </parts>
 <sheets>
@@
 <instance part="U1" gate="G$1" x="182.88" y="114.3"/>
 <instance part="GND18" gate="1" x="223.52" y="223.52" rot="R90"/>
+<instance part="H1" gate="G$1" x="167.64" y="83.82"/>
+<instance part="LOGO1" gate="G$1" x="187.96" y="83.82"/>
 </instances>
 <busses>

Commit message: Some minor touch ups
Parts:
- removed C62: 2.2uF, SparkFun-Passives:CAP1206
- added C9: 100uF, SparkFun-Capacitors:CAP1210
- added H2, H3: MOUNTING_HOLE#6, MRDT-Hardware:MOUNTING_HOLE#6
- C1, C2, C3, C4, C5, C6, C7, C8: value (none) -> 100uF
- renumbered ENCODER1 to ENC1, ENCODER2 to ENC2, ENCODER3 to ENC3, ENCODER4 to ENC4, ENCODER5 to ENC5, ENCODER6 to ENC6, LIMIT_SWITCH_1 to LIMIT_1, LIMIT_SWITCH_2 to LIMIT_2, LIMIT_SWITCH_3 to LIMIT_3
Connections:
- net GND: now also C9.1; no longer C62.1
- net VCC_12V: now also C9.2; no longer C62.2
