File: ArmBoard_2019_Rev1/ArmBoardMC_2019_Rev1/ArmBoardMC_2019_Rev1.sch (KiCad schematic (older format))
At the start: 60 parts, among them U1 TM4C129E_Launchpad, U10 Limit_Switch5, U11 Limit_Switch7, U12 Limit_Switch2, U13 Limit_Switch4, U14 Limit_Switch6, U15 Limit_Switch8, U16 MAX_3232, U17 Encoder_1, U18 Encoder_3, U19 Encoder_2, U2 TM4C129E_Launchpad, U20 Encoder_4, U3 OKI, U4 VNH5019A_E, U5 VNH5019A_E, U6 VNH5019A_E, U7 VNH5019A_E, U8 Limit_Switch1, U9 Limit_Switch3

Commit message: Annotated Schematic
Parts:
- U10: renamed from U11; value Limit_Switch7 -> Limit_Switch
- U13: renamed from U14; value Limit_Switch6 -> Limit_Switch
- U14: renamed from U15; value Limit_Switch8 -> Limit_Switch
- renumbered C10 to C1, C8 to C10, C9 to C11, C11 to C2, C1 to C3, C6 to C4, C7 to C5, C2 to C6, C3 to C7, C4 to C8, C5 to C9, Conn2 to Conn1, Conn3 to Conn2, Conn4 to Conn3, Conn5 to Conn4, Conn6 to Conn5, Conn1 to Conn6, R5 to R1, R14 to R10, R15 to R11, R16 to R12, R17 to R13, R2 to R14, R3 to R15, R18 to R16, R19 to R17, R2 to R18, R4 to R19, R6 to R2, R1 to R22, R7 to R3, R8 to R4, R9 to R5, R10 to R6, R11 to R7, R12 to R8, R13 to R9, U4 to U1, U12 to U11, U13 to U12, U16 to U15, U3 to U16, U5 to U2, U1 to U3, U2 to U4, U6 to U5, U7 to U6, U8 to U7, U9 to U8, U10 to U9

Commit message: Gave Capacitors and Resistors values
Parts:
- removed R8: R_Small, symbol Device:R_Small
- C1, C10, C11, C2: value C_Small -> .1uF
- R1, R10, R11, R12, R13, R2, R3, R4, R5, R6, R7, R9: value R_Small -> 1K
Other:
- note removed: "1K"
Changed lines of the file:
@@
 Wire Wire Line
 	4400 4025 4275 4025
-$Comp
-L Device:R_Small R7
-U 1 1 5BD4DECC
-P 4175 4025
-F 0 "R7" V 4225 4025 31  0000 C CNN
-F 1 "R_Small" V 4070 4025 50  0001 C CNN
-F 2 "" H 4175 4025 50  0001 C CNN
-F 3 "~" H 4175 4025 50  0001 C CNN
-	1    4175 4025
-	0    1    1    0
-$EndComp
 Wire Wire Line
 	4075 4025 4000 4025
-Text Notes 4200 4050 2    31   ~ 0
-1K
 $Comp
 L Device:R_Small R11
@@
 P 4275 1875
 F 0 "R11" V 4325 1875 31  0000 C CNN
-F 1 "R_Small" V 4170 1875 50  0001 C CNN
+F 1 "1K" V 4275 1875 31  0000 C CNN
 F 2 "" H 4275 1875 50  0001 C CNN
 F 3 "~" H 4275 1875 50  0001 C CNN
@@
 	0    1    1    0
 $EndComp
-Text Notes 4300 1900 2    31   ~ 0
-1K
 Wire Wire Line
 	4175 1875 4100 1875
@@
 P 1225 4000
 F 0 "R5" V 1275 4000 31  0000 C CNN
-F 1 "R_Small" V 1120 4000 50  0001 C CNN
+F 1 "1K" V 1225 4000 31  0000 C CNN
 F 2 "" H 1225 4000 50  0001 C CNN
 F 3 "~" H 1225 4000 50  0001 C CNN
@@
 Wire Wire Line
 	1125 4000 1025 4000
-Text Notes 1250 4025 2    31   ~ 0
-1K
 Wire Wire Line
 	1375 1950 1300 1950
@@
 P 1200 1950
 F 0 "R1" V 1250 1950 31  0000 C CNN
-F 1 "R_Small" V 1095 1950 50  0001 C CNN
+F 1 "1K" V 1200 1950 31  0000 C CNN
 F 2 "" H 1200 1950 50  0001 C CNN
 F 3 "~" H 1200 1950 50  0001 C CNN
@@
 	0    1    1    0
 $EndComp
-Text Notes 1225 1975 2    31   ~ 0
-1K
 Wire Wire Line
 	1100 1950 1050 1950
@@
 Wire Wire Line
 	1375 2250 1300 2250
-$Comp
-L Device:R_Small R2
-U 1 1 5BDE1FC2
-P 1200 2250
-F 0 "R2" V 1275 2250 31  0000 C CNN
-F 1 "R_Small" V 1275 2250 50  0001 C CNN
-F 2 "" H 1200 2250 50  0001 C CNN
-F 3 "~" H 1200 2250 50  0001 C CNN
-	1    1200 2250
-	0    1    1    0
-$EndComp
 Wire Wire Line
 	1100 2250 1050 2250
@@
 P 1225 1650
 F 0 "R3" V 1150 1650 31  0000 C CNN
-F 1 "R_Small" V 1120 1650 50  0001 C CNN
+F 1 "1K" V 1225 1650 31  0000 C CNN
 F 2 "" H 1225 1650 50  0001 C CNN
 F 3 "~" H 1225 1650 50  0001 C CNN
@@
 P 1225 3700
 F 0 "R4" V 1150 3700 31  0000 C CNN
-F 1 "R_Small" V 1120 3700 50  0001 C CNN
+F 1 "1K" V 1225 3700 31  0000 C CNN
 F 2 "" H 1225 3700 50  0001 C CNN
 F 3 "~" H 1225 3700 50  0001 C CNN
@@
 Wire Wire Line
 	1400 4300 1350 4300
-$Comp
-L Device:R_Small R6
-U 1 1 5BE5B77C
-P 1250 4300
-F 0 "R6" V 1300 4300 31  0000 C CNN
-F 1 "R_Small" V 1145 4300 50  0001 C CNN
-F 2 "" H 1250 4300 50  0001 C CNN
-F 3 "~" H 1250 4300 50  0001 C CNN
-	1    1250 4300
-	0    1    1    0
-$EndComp
 Wire Wire Line
 	1150 4300 1100 4300
@@
 P 4300 1575
 F 0 "R13" V 4225 1575 31  0000 C CNN
-F 1 "R_Small" V 4195 1575 50  0001 C CNN
+F 1 "1K" V 4300 1575 31  0000 C CNN
 F 2 "" H 4300 1575 50  0001 C CNN
 F 3 "~" H 4300 1575 50  0001 C CNN
@@
 P 4275 2175
 F 0 "R12" V 4350 2175 31  0000 C CNN
-F 1 "R_Small" V 4170 2175 50  0001 C CNN
+F 1 "1K" V 4275 2175 31  0000 C CNN
 F 2 "" H 4275 2175 50  0001 C CNN
 F 3 "~" H 4275 2175 50  0001 C CNN
@@
 U 1 1 5BEE4968
 P 4250 3725
-F 0 "R10" V 4175 3750 31  0000 C CNN
-F 1 "R_Small" V 4145 3725 50  0001 C CNN
+F 0 "R10" V 4175 3725 31  0000 C CNN
+F 1 "1K" V 4250 3725 31  0000 C CNN
 F 2 "" H 4250 3725 50  0001 C CNN
 F 3 "~" H 4250 3725 50  0001 C CNN
@@
 P 4225 4325
 F 0 "R9" V 4300 4325 31  0000 C CNN
-F 1 "R_Small" V 4120 4325 50  0001 C CNN
+F 1 "1K" V 4225 4325 31  0000 C CNN
 F 2 "" H 4225 4325 50  0001 C CNN
 F 3 "~" H 4225 4325 50  0001 C CNN
@@
 Text GLabel 4075 4325 0    31   Input ~ 0
 IN_A4
-$Comp
-L Device:R_Small R8
-U 1 1 5BF2B87C
-P 4175 4025
-F 0 "R8" V 4250 4025 50  0001 C CNN
-F 1 "R_Small" V 4070 4025 50  0001 C CNN
-F 2 "" H 4175 4025 50  0001 C CNN
-F 3 "~" H 4175 4025 50  0001 C CNN
-	1    4175 4025
-	0    1    1    0
-$EndComp
-Connection ~ 4275 4025
-Connection ~ 4075 4025
-Text Notes 4250 4350 2    31   ~ 0
-1K
-Text Notes 4275 3750 2    31   ~ 0
-1K
-Text Notes 4300 2200 2    31   ~ 0
-1K
-Text Notes 4325 1600 2    31   ~ 0
-1K
-Text Notes 1275 4325 2    31   ~ 0
-1K
-Text Notes 1250 3725 2    31   ~ 0
-1K
-Text Notes 1225 2275 2    31   ~ 0
-1K
-Text Notes 1250 1675 2    31   ~ 0
-1K
 Wire Wire Line
 	6000 3075 6050 3075
@@
 Text Notes 3075 1500 0    31   ~ 0
 Out_B1\n
-Text Notes 3125 3150 0    31   ~ 0
-Out_A2\n
 Text Notes 3125 3550 0    31   ~ 0
 Out_B2\n
@@
 U 1 1 5C9225CC
 P 10675 1350
-F 0 "C10" H 10700 1425 50  0000 L CNN
-F 1 "C_Small" H 10767 1305 50  0001 L CNN
+F 0 "C10" H 10675 1400 31  0000 L CNN
+F 1 ".1uF" H 10675 1300 31  0000 L CNN
 F 2 "" H 10675 1350 50  0001 C CNN
 F 3 "~" H 10675 1350 50  0001 C CNN
@@
 U 1 1 5CA6FA04
 P 10675 1650
-F 0 "C11" H 10700 1725 50  0000 L CNN
-F 1 "C_Small" H 10767 1605 50  0001 L CNN
+F 0 "C11" H 10675 1700 31  0000 L CNN
+F 1 ".1uF" H 10675 1600 31  0000 L CNN
 F 2 "" H 10675 1650 50  0001 C CNN
 F 3 "~" H 10675 1650 50  0001 C CNN
@@
 U 1 1 5CAD4E6B
 P 9325 1650
-F 0 "C1" V 9275 1700 39  0000 L CNN
-F 1 "C_Small" H 9417 1605 50  0001 L CNN
+F 0 "C1" V 9300 1725 31  0000 C CNN
+F 1 ".1uF" V 9300 1550 31  0000 C CNN
 F 2 "" H 9325 1650 50  0001 C CNN
 F 3 "~" H 9325 1650 50  0001 C CNN
@@
 U 1 1 5CAD5071
 P 9325 1750
-F 0 "C2" V 9375 1800 39  0000 L CNN
-F 1 "C_Small" H 9417 1705 50  0001 L CNN
+F 0 "C2" V 9350 1800 31  0000 L CNN
+F 1 ".1uF" V 9350 1600 31  0000 L CNN
 F 2 "" H 9325 1750 50  0001 C CNN
 F 3 "~" H 9325 1750 50  0001 C CNN
@@
 Text Notes 3325 725  0    118  ~ 24
 H-Bridges
+$Comp
+L Device:R_Small R7
+U 1 1 5BD4DECC
+P 4175 4025
+F 0 "R7" V 4250 4025 31  0000 C CNN
+F 1 "1K" V 4175 4025 31  0000 C CNN
+F 2 "" H 4175 4025 50  0001 C CNN
+F 3 "~" H 4175 4025 50  0001 C CNN
+	1    4175 4025
+	0    1    1    0
+$EndComp
+$Comp
+L Device:R_Small R6
+U 1 1 5BE5B77C
+P 1250 4300
+F 0 "R6" V 1300 4300 31  0000 C CNN
+F 1 "1K" V 1250 4300 31  0000 C CNN
+F 2 "" H 1250 4300 50  0001 C CNN
+F 3 "~" H 1250 4300 50  0001 C CNN
+	1    1250 4300
+	0    1    1    0
+$EndComp
+$Comp
+L Device:R_Small R2
+U 1 1 5BDE1FC2
+P 1200 2250
+F 0 "R2" V 1275 2250 31  0000 C CNN
+F 1 "1K" V 1200 2250 31  0000 C CNN
+F 2 "" H 1200 2250 50  0001 C CNN
+F 3 "~" H 1200 2250 50  0001 C CNN
+	1    1200 2250
+	0    1    1    0
+$EndComp
+Text Notes 3125 3150 0    31   ~ 0
+Out_A2\n
 $EndSCHEMATC

Commit message: Added more values and assigned footprint libraries to schematic
Hopefully it transfers over to your end
Parts:
- C1, C10, C11, C2, C3, C4, C5, C6, C7, C8, C9: footprint (none) -> Capacitor_SMD:C_0603_1608Metric_Pad1.05x0.95mm_HandSolder
- Conn1, Conn2, Conn3, Conn4: value AndersonPP -> Anderson-2; footprint (none) -> MRDT_Connectors:Anderson_2_Horisontal_Side_by_Side
- Conn5: footprint (none) -> MRDT_Connectors:MOLEX_SL_05_Vertical
- Conn6: value AndersonPP -> Anderson-3; footprint (none) -> MRDT_Connectors:Anderson_3_Horisontal_Side_by_Side
- Conn6: renamed from Conn1; value AndersonPP -> Anderson-3; footprint (none) -> MRDT_Connectors:Anderson_3_Horisontal_Side_by_Side
- D1: footprint (none) -> Diode_SMD:D_1206_3216Metric
- R1, R10, R11, R12, R13, R2, R22, R3, R4, R5, R6, R7, R9: footprint (none) -> Resistor_SMD:R_0603_1608Metric_Pad1.05x0.95mm_HandSolder
- R14, R15, R16, R17, R18, R19, R20, R21: value R_Small -> 10K; footprint (none) -> Resistor_SMD:R_0603_1608Metric_Pad1.05x0.95mm_HandSolder
- U1, U2, U5, U6: footprint (none) -> MRDT_ICs:MultiPowerSO_30
- U10: value Limit_Switch -> Limit_Switch7; footprint (none) -> MRDT_Connectors:MOLEX_SL_02_Vertical
- U11, U12, U7, U8, U9: footprint (none) -> MRDT_Connectors:MOLEX_SL_02_Vertical
- U13: value Limit_Switch -> Limit_Switch6; footprint (none) -> MRDT_Connectors:MOLEX_SL_02_Vertical
- U14: value Limit_Switch -> Limit_Switch8; footprint (none) -> MRDT_Connectors:MOLEX_SL_02_Vertical
- U15: footprint (none) -> MRDT_ICs:SOIC_16_3.9x9.9mm_Pitch1.27mm
- U16: footprint (none) -> MRDT_Devices:OKI_Horizontal
- U17, U18, U19, U20: footprint (none) -> MRDT_Connectors:MOLEX_SL_03_Vertical
- U3, U4: footprint (none) -> MRDT_Shields:TM4C129E_Launchpad_X9
Other:
- note removed: "10K"

Commit message: Fixed Tiva issue
There was a copy of a section of it. Doesnt cause further problems.
Parts:
- removed U4: TM4C129E_Launchpad, MRDT_Shields:TM4C129E_Launchpad_X9, symbol MRDT_Shields:TM4C129E_Launchpad
- added unit 8 of U3
- U3: footprint MRDT_Shields:TM4C129E_Launchpad_X9 -> MRDT_Shields:TM4C129E_Launchpad_FULL
Connections:
- wire segments 308 -> 310
Changed lines of the file:
@@
 F 0 "U3" H 1850 6325 60  0000 L CNN
 F 1 "TM4C129E_Launchpad" H 1400 6225 60  0001 L CNN
-F 2 "MRDT_Shields:TM4C129E_Launchpad_X9" H 1800 6375 60  0001 C CNN
+F 2 "MRDT_Shields:TM4C129E_Launchpad_FULL" H 1800 6375 60  0001 C CNN
 F 3 "" H 1800 6375 60  0001 C CNN
 	1    1800 6375
@@
 F 0 "U3" H 2400 6325 60  0000 C CNN
 F 1 "TM4C129E_Launchpad" H 1825 7525 60  0000 C CNN
-F 2 "MRDT_Shields:TM4C129E_Launchpad_X9" H 2300 6375 60  0001 C CNN
+F 2 "MRDT_Shields:TM4C129E_Launchpad_FULL" H 2300 6375 60  0001 C CNN
 F 3 "" H 2300 6375 60  0001 C CNN
 	2    2300 6375
@@
 F 0 "U3" H 1850 7550 60  0000 L CNN
 F 1 "TM4C129E_Launchpad" H 2105 8092 60  0001 L CNN
-F 2 "MRDT_Shields:TM4C129E_Launchpad_X9" H 1800 7600 60  0001 C CNN
+F 2 "MRDT_Shields:TM4C129E_Launchpad_FULL" H 1800 7600 60  0001 C CNN
 F 3 "" H 1800 7600 60  0001 C CNN
 	3    1800 7600
@@
 F 0 "U3" H 2400 7550 60  0000 C CNN
 F 1 "TM4C129E_Launchpad" H 2150 8750 60  0001 C CNN
-F 2 "MRDT_Shields:TM4C129E_Launchpad_X9" H 2300 7600 60  0001 C CNN
+F 2 "MRDT_Shields:TM4C129E_Launchpad_FULL" H 2300 7600 60  0001 C CNN
 F 3 "" H 2300 7600 60  0001 C CNN
 	4    2300 7600
@@
 F 0 "U3" H 3700 6325 60  0000 L CNN
 F 1 "TM4C129E_Launchpad" H 3951 6867 60  0001 L CNN
-F 2 "MRDT_Shields:TM4C129E_Launchpad_X9" H 3650 6375 60  0001 C CNN
+F 2 "MRDT_Shields:TM4C129E_Launchpad_FULL" H 3650 6375 60  0001 C CNN
 F 3 "" H 3650 6375 60  0001 C CNN
 	5    3650 6375
@@
 F 0 "U3" H 4250 6325 60  0000 C CNN
 F 1 "TM4C129E_Launchpad" H 4182 7546 60  0001 C CNN
-F 2 "MRDT_Shields:TM4C129E_Launchpad_X9" H 4150 6375 60  0001 C CNN
+F 2 "MRDT_Shields:TM4C129E_Launchpad_FULL" H 4150 6375 60  0001 C CNN
 F 3 "" H 4150 6375 60  0001 C CNN
 	6    4150 6375
@@
 F 0 "U3" H 3700 7550 60  0000 L CNN
 F 1 "TM4C129E_Launchpad" H 3955 8092 60  0001 L CNN
-F 2 "MRDT_Shields:TM4C129E_Launchpad_X9" H 3650 7600 60  0001 C CNN
+F 2 "MRDT_Shields:TM4C129E_Launchpad_FULL" H 3650 7600 60  0001 C CNN
 F 3 "" H 3650 7600 60  0001 C CNN
 	7    3650 7600
 	1    0    0    -1
-$EndComp
-$Comp
-L MRDT_Shields:TM4C129E_Launchpad U4
-U 7 1 5BC25775
-P 4150 7600
-F 0 "U4" H 4300 7550 60  0000 C CNN
-F 1 "TM4C129E_Launchpad" H 4182 8771 60  0001 C CNN
-F 2 "MRDT_Shields:TM4C129E_Launchpad_X9" H 4150 7600 60  0001 C CNN
-F 3 "" H 4150 7600 60  0001 C CNN
-	7    4150 7600
-	-1   0    0    -1
 $EndComp
 Text Notes 2575 5150 0    118  ~ 24
@@
 	0    1    1    0
 $EndComp
+$Comp
+L MRDT_Shields:TM4C129E_Launchpad U3
+U 8 1 5CC0A057
+P 4150 7600
+F 0 "U3" H 4275 7550 60  0000 C CNN
+F 1 "TM4C129E_Launchpad" H 3200 7650 60  0001 C CNN
+F 2 "" H 4150 7600 60  0001 C CNN
+F 3 "" H 4150 7600 60  0001 C CNN
+	8    4150 7600
+	-1   0    0    -1
+$EndComp
+Text GLabel 4425 6650 2    31   UnSpc ~ 0
+GND
+Text GLabel 2600 6650 2    31   UnSpc ~ 0
+GND
+Wire Wire Line
+	4350 6650 4425 6650
+Wire Wire Line
+	2500 6650 2600 6650
 $EndSCHEMATC

Commit message: Placed Footprints onto PCB schematic Design
Parts:
- U3: footprint (none) -> MRDT_Shields:TM4C129E_Launchpad_FULL
Changed lines of the file:
@@
 F 0 "U3" H 4275 7550 60  0000 C CNN
 F 1 "TM4C129E_Launchpad" H 3200 7650 60  0001 C CNN
-F 2 "" H 4150 7600 60  0001 C CNN
+F 2 "MRDT_Shields:TM4C129E_Launchpad_FULL" H 4150 7600 60  0001 C CNN
 F 3 "" H 4150 7600 60  0001 C CNN
 	8    4150 7600

Commit message: Created and started workign on high level placement
Parts:
- U3: footprint MRDT_Shields:TM4C129E_Launchpad_FULL -> MRDT_Shields:TM4C129E_Launchpad_FULL_Bottom_SMD
Connections:
- wire segments 310 -> 312
Changed lines of the file:
@@
 F 0 "U3" H 1850 6325 60  0000 L CNN
 F 1 "TM4C129E_Launchpad" H 1400 6225 60  0001 L CNN
-F 2 "MRDT_Shields:TM4C129E_Launchpad_FULL" H 1800 6375 60  0001 C CNN
+F 2 "MRDT_Shields:TM4C129E_Launchpad_FULL_Bottom_SMD" H 1800 6375 60  0001 C CNN
 F 3 "" H 1800 6375 60  0001 C CNN
 	1    1800 6375
@@
 F 0 "U3" H 2400 6325 60  0000 C CNN
 F 1 "TM4C129E_Launchpad" H 1825 7525 60  0000 C CNN
-F 2 "MRDT_Shields:TM4C129E_Launchpad_FULL" H 2300 6375 60  0001 C CNN
+F 2 "MRDT_Shields:TM4C129E_Launchpad_FULL_Bottom_SMD" H 2300 6375 60  0001 C CNN
 F 3 "" H 2300 6375 60  0001 C CNN
 	2    2300 6375
@@
 F 0 "U3" H 1850 7550 60  0000 L CNN
 F 1 "TM4C129E_Launchpad" H 2105 8092 60  0001 L CNN
-F 2 "MRDT_Shields:TM4C129E_Launchpad_FULL" H 1800 7600 60  0001 C CNN
+F 2 "MRDT_Shields:TM4C129E_Launchpad_FULL_Bottom_SMD" H 1800 7600 60  0001 C CNN
 F 3 "" H 1800 7600 60  0001 C CNN
 	3    1800 7600
@@
 F 0 "U3" H 2400 7550 60  0000 C CNN
 F 1 "TM4C129E_Launchpad" H 2150 8750 60  0001 C CNN
-F 2 "MRDT_Shields:TM4C129E_Launchpad_FULL" H 2300 7600 60  0001 C CNN
+F 2 "MRDT_Shields:TM4C129E_Launchpad_FULL_Bottom_SMD" H 2300 7600 60  0001 C CNN
 F 3 "" H 2300 7600 60  0001 C CNN
 	4    2300 7600
@@
 F 0 "U3" H 3700 6325 60  0000 L CNN
 F 1 "TM4C129E_Launchpad" H 3951 6867 60  0001 L CNN
-F 2 "MRDT_Shields:TM4C129E_Launchpad_FULL" H 3650 6375 60  0001 C CNN
+F 2 "MRDT_Shields:TM4C129E_Launchpad_FULL_Bottom_SMD" H 3650 6375 60  0001 C CNN
 F 3 "" H 3650 6375 60  0001 C CNN
 	5    3650 6375
@@
 F 0 "U3" H 4250 6325 60  0000 C CNN
 F 1 "TM4C129E_Launchpad" H 4182 7546 60  0001 C CNN
-F 2 "MRDT_Shields:TM4C129E_Launchpad_FULL" H 4150 6375 60  0001 C CNN
+F 2 "MRDT_Shields:TM4C129E_Launchpad_FULL_Bottom_SMD" H 4150 6375 60  0001 C CNN
 F 3 "" H 4150 6375 60  0001 C CNN
 	6    4150 6375
@@
 F 0 "U3" H 3700 7550 60  0000 L CNN
 F 1 "TM4C129E_Launchpad" H 3955 8092 60  0001 L CNN
-F 2 "MRDT_Shields:TM4C129E_Launchpad_FULL" H 3650 7600 60  0001 C CNN
+F 2 "MRDT_Shields:TM4C129E_Launchpad_FULL_Bottom_SMD" H 3650 7600 60  0001 C CNN
 F 3 "" H 3650 7600 60  0001 C CNN
 	7    3650 7600
@@
 F 0 "U3" H 4275 7550 60  0000 C CNN
 F 1 "TM4C129E_Launchpad" H 3200 7650 60  0001 C CNN
-F 2 "MRDT_Shields:TM4C129E_Launchpad_FULL" H 4150 7600 60  0001 C CNN
+F 2 "MRDT_Shields:TM4C129E_Launchpad_FULL_Bottom_SMD" H 4150 7600 60  0001 C CNN
 F 3 "" H 4150 7600 60  0001 C CNN
 	8    4150 7600
@@
 Wire Wire Line
 	2500 6650 2600 6650
+Wire Wire Line
+	4450 1675 4375 1675
+Wire Wire Line
+	4450 1775 4375 1775
 $EndSCHEMATC

Commit message: Updated high level placement
Made decent progress but still a lot to do
Parts:
- removed unit 3 of Conn1
- removed unit 3 of Conn2
- removed unit 3 of Conn3
- removed unit 3 of Conn4
- added unit 2 of Conn1
- added unit 2 of Conn2
- added unit 2 of Conn3
- added unit 2 of Conn4
- Conn1, Conn2, Conn3, Conn4: value Anderson-2 -> AndersonPP
Connections:
- net labels added: Out_A1, Out_A3, Out_A4, Out_B1, Out_B2, Out_B3, Out_B4
- wire segments 312 -> 313
Other:
- note removed: "Out_A1\n"
- note removed: "Out_A2\n"
- note removed: "Out_A3\n"
- note removed: "Out_A4"
- note removed: "Out_B1\n"
- note removed: "Out_B2\n"
- note removed: "Out_B3\n"
- note removed: "Out_B4\n"
Changed lines of the file:
@@
 Wire Wire Line
 	6050 3575 6050 3675
-Text Notes 6125 3175 0    31   ~ 0
-Out_A4
 $Comp
 L MRDT_Connectors:AndersonPP Conn3
 U 1 1 5C0054EB
-P 6700 1325
-F 0 "Conn3" H 6900 1575 39  0000 R CNN
-F 1 "Anderson-2" V 6625 1425 60  0001 R CNN
-F 2 "MRDT_Connectors:Anderson_2_Horisontal_Side_by_Side" H 6550 775 60  0001 C CNN
-F 3 "" H 6550 775 60  0001 C CNN
-	1    6700 1325
+P 6700 925
+F 0 "Conn3" H 6900 1175 39  0000 R CNN
+F 1 "AndersonPP" V 6625 1025 60  0001 R CNN
+F 2 "MRDT_Connectors:Anderson_2_Horisontal_Side_by_Side" H 6550 375 60  0001 C CNN
+F 3 "" H 6550 375 60  0001 C CNN
+	1    6700 925
 	-1   0    0    1
 $EndComp
@@
 Wire Wire Line
 	6050 3575 6325 3575
-Text Notes 6100 3575 0    31   ~ 0
-Out_B4\n
 Wire Wire Line
 	6050 925  6125 925
@@
 	3100 3550 3300 3550
 Wire Wire Line
-	3100 3150 3300 3150
+	3100 3150 3275 3150
 Wire Wire Line
 	3050 1300 2975 1300
@@
 L MRDT_Connectors:AndersonPP Conn4
 U 1 1 5C47ACED
-P 6725 3475
-F 0 "Conn4" H 6925 3725 39  0000 R CNN
-F 1 "Anderson-2" V 6650 3575 60  0001 R CNN
-F 2 "MRDT_Connectors:Anderson_2_Horisontal_Side_by_Side" H 6575 2925 60  0001 C CNN
-F 3 "" H 6575 2925 60  0001 C CNN
-	1    6725 3475
+P 6725 3075
+F 0 "Conn4" H 6925 3325 39  0000 R CNN
+F 1 "AndersonPP" V 6650 3175 60  0001 R CNN
+F 2 "MRDT_Connectors:Anderson_2_Horisontal_Side_by_Side" H 6575 2525 60  0001 C CNN
+F 3 "" H 6575 2525 60  0001 C CNN
+	1    6725 3075
 	-1   0    0    1
 $EndComp
@@
 L MRDT_Connectors:AndersonPP Conn2
 U 1 1 5C47B742
-P 3700 3450
-F 0 "Conn2" H 3900 3700 39  0000 R CNN
-F 1 "Anderson-2" V 3625 3550 60  0001 R CNN
-F 2 "MRDT_Connectors:Anderson_2_Horisontal_Side_by_Side" H 3550 2900 60  0001 C CNN
-F 3 "" H 3550 2900 60  0001 C CNN
-	1    3700 3450
+P 3675 3050
+F 0 "Conn2" H 3875 3300 39  0000 R CNN
+F 1 "AndersonPP" V 3600 3150 60  0001 R CNN
+F 2 "MRDT_Connectors:Anderson_2_Horisontal_Side_by_Side" H 3525 2500 60  0001 C CNN
+F 3 "" H 3525 2500 60  0001 C CNN
+	1    3675 3050
 	-1   0    0    1
 $EndComp
@@
 L MRDT_Connectors:AndersonPP Conn1
 U 1 1 5C47BBD6
-P 3625 1400
-F 0 "Conn1" H 3825 1650 39  0000 R CNN
-F 1 "Anderson-2" V 3550 1500 60  0001 R CNN
-F 2 "MRDT_Connectors:Anderson_2_Horisontal_Side_by_Side" H 3475 850 60  0001 C CNN
-F 3 "" H 3475 850 60  0001 C CNN
-	1    3625 1400
-	-1   0    0    1
-$EndComp
-Text Notes 3075 1100 0    31   ~ 0
-Out_A1\n
-Text Notes 3075 1500 0    31   ~ 0
-Out_B1\n
-Text Notes 3125 3550 0    31   ~ 0
-Out_B2\n
-Text Notes 6150 1025 0    31   ~ 0
-Out_A3\n
-Text Notes 6150 1425 0    31   ~ 0
-Out_B3\n
+P 3625 1000
+F 0 "Conn1" H 3825 1250 39  0000 R CNN
+F 1 "AndersonPP" V 3550 1100 60  0001 R CNN
+F 2 "MRDT_Connectors:Anderson_2_Horisontal_Side_by_Side" H 3475 450 60  0001 C CNN
+F 3 "" H 3475 450 60  0001 C CNN
+	1    3625 1000
+	-1   0    0    1
+$EndComp
 Text Notes 6450 800  0    51   ~ 0
 Motor 3
@@
 	1    0    0    -1
 $EndComp
-$Comp
-L MRDT_Connectors:AndersonPP Conn4
-U 3 1 5CC350B6
-P 6725 3075
-F 0 "Conn4" H 6925 3325 39  0000 R CNN
-F 1 "Anderson-2" H 7000 3050 39  0000 R CNN
-F 2 "MRDT_Connectors:Anderson_2_Horisontal_Side_by_Side" H 6575 2525 60  0001 C CNN
-F 3 "" H 6575 2525 60  0001 C CNN
-	3    6725 3075
-	-1   0    0    1
-$EndComp
-$Comp
-L MRDT_Connectors:AndersonPP Conn3
-U 3 1 5CC35253
-P 6700 925
-F 0 "Conn3" H 6900 1175 39  0000 R CNN
-F 1 "Anderson-2" H 6975 875 39  0000 R CNN
-F 2 "MRDT_Connectors:Anderson_2_Horisontal_Side_by_Side" H 6550 375 60  0001 C CNN
-F 3 "" H 6550 375 60  0001 C CNN
-	3    6700 925
-	-1   0    0    1
-$EndComp
-$Comp
-L MRDT_Connectors:AndersonPP Conn2
-U 3 1 5CC35627
-P 3700 3050
-F 0 "Conn2" H 3900 3300 39  0000 R CNN
-F 1 "Anderson-2" H 3975 3000 39  0000 R CNN
-F 2 "MRDT_Connectors:Anderson_2_Horisontal_Side_by_Side" H 3550 2500 60  0001 C CNN
-F 3 "" H 3550 2500 60  0001 C CNN
-	3    3700 3050
-	-1   0    0    1
-$EndComp
-$Comp
-L MRDT_Connectors:AndersonPP Conn1
-U 3 1 5CC35999
-P 3625 1000
-F 0 "Conn1" H 3825 1250 39  0000 R CNN
-F 1 "Anderson-2" H 3875 975 39  0000 R CNN
-F 2 "MRDT_Connectors:Anderson_2_Horisontal_Side_by_Side" H 3475 450 60  0001 C CNN
-F 3 "" H 3475 450 60  0001 C CNN
-	3    3625 1000
-	-1   0    0    1
-$EndComp
 Wire Wire Line
 	7900 1325 7500 1325
@@
 	0    1    1    0
 $EndComp
-Text Notes 3125 3150 0    31   ~ 0
-Out_A2\n
 $Comp
 L Device:R_Small R15
@@
 Wire Wire Line
 	4450 1775 4375 1775
+$Comp
+L MRDT_Connectors:AndersonPP Conn2
+U 2 1 5BDBDE04
+P 3700 3450
+F 0 "Conn2" H 3673 3497 60  0000 R CNN
+F 1 "AndersonPP" H 3673 3603 60  0000 R CNN
+F 2 "MRDT_Connectors:Anderson_2_Horisontal_Side_by_Side" H 3550 2900 60  0001 C CNN
+F 3 "" H 3550 2900 60  0001 C CNN
+	2    3700 3450
+	-1   0    0    1
+$EndComp
+$Comp
+L MRDT_Connectors:AndersonPP Conn1
+U 2 1 5BDBE507
+P 3625 1400
+F 0 "Conn1" H 3598 1447 60  0000 R CNN
+F 1 "AndersonPP" H 3598 1553 60  0000 R CNN
+F 2 "MRDT_Connectors:Anderson_2_Horisontal_Side_by_Side" H 3475 850 60  0001 C CNN
+F 3 "" H 3475 850 60  0001 C CNN
+	2    3625 1400
+	-1   0    0    1
+$EndComp
+$Comp
+L MRDT_Connectors:AndersonPP Conn3
+U 2 1 5BDBE5AD
+P 6700 1325
+F 0 "Conn3" H 6673 1372 60  0000 R CNN
+F 1 "AndersonPP" H 6673 1478 60  0000 R CNN
+F 2 "MRDT_Connectors:Anderson_2_Horisontal_Side_by_Side" H 6550 775 60  0001 C CNN
+F 3 "" H 6550 775 60  0001 C CNN
+	2    6700 1325
+	-1   0    0    1
+$EndComp
+$Comp
+L MRDT_Connectors:AndersonPP Conn4
+U 2 1 5BDBE659
+P 6725 3475
+F 0 "Conn4" H 6698 3522 60  0000 R CNN
+F 1 "AndersonPP" H 6698 3628 60  0000 R CNN
+F 2 "MRDT_Connectors:Anderson_2_Horisontal_Side_by_Side" H 6575 2925 60  0001 C CNN
+F 3 "" H 6575 2925 60  0001 C CNN
+	2    6725 3475
+	-1   0    0    1
+$EndComp
+Text GLabel 7275 5575 0    31   Input ~ 0
+Logic_3.3V
+Connection ~ 3275 3150
+Wire Wire Line
+	3275 3150 3300 3150
+Text Label 3050 1100 0    39   ~ 0
+Out_A1
+Text Label 3050 1500 0    39   ~ 0
+Out_B1
+Text Label 3100 3150 0    39   ~ 0
+Out_B2
+Text Label 3100 3550 0    39   ~ 0
+Out_B2
+Text Label 6125 1025 0    39   ~ 0
+Out_A3
+Text Label 6125 1425 0    39   ~ 0
+Out_B3
+Text Label 6050 3175 0    39   ~ 0
+Out_A4
+Text Label 6050 3575 0    39   ~ 0
+Out_B4
 $EndSCHEMATC
