File: ArmBoard_2019_Rev1/ArmBoardMC_2019_Rev1/ArmBoardMC_2019_Rev1.sch (KiCad schematic (older format))
At the start: 58 parts, among them U1 VNH5019A_E, U10 Limit_Switch7, U11 Limit_Switch2, U12 Limit_Switch4, U13 Limit_Switch6, U14 Limit_Switch8, U15 MAX_3232, U16 OKI, U17 Encoder_1, U18 Encoder_3, U19 Encoder_2, U2 VNH5019A_E, U20 Encoder_4, U3 TM4C129E_Launchpad, U5 VNH5019A_E, U6 VNH5019A_E, U7 Limit_Switch1, U8 Limit_Switch3, U9 Limit_Switch5

Commit message: Finished high level placement and adjusted schematic
High level placement for PDR is finished. I had to change up the schematic a bit in order for it to work
Parts:
- Conn5: footprint MRDT_Connectors:MOLEX_SL_05_Vertical -> MRDT_Connectors:MOLEX_SL_05_Horizontal
Connections:
- net labels added: I_Sense_1, I_Sense_2, I_Sense_3, I_Sense_4
Other:
- note added: "A0"
- note added: "A1"
- note added: "A2"
- note added: "A3"
Changed lines of the file:
@@
 F 0 "Conn5" H 8075 2200 60  0000 L CNN
 F 1 "Molex_SL_05" H 7925 2125 60  0000 L CNN
-F 2 "MRDT_Connectors:MOLEX_SL_05_Vertical" H 8100 1575 60  0001 C CNN
+F 2 "MRDT_Connectors:MOLEX_SL_05_Horizontal" H 8100 1575 60  0001 C CNN
 F 3 "" H 8100 1575 60  0001 C CNN
 	1    8100 1575
@@
 Text GLabel 1525 6125 0    31   Input ~ 0
 LS_4
-Text GLabel 2550 5625 2    31   Input ~ 0
+Text GLabel 2500 6025 2    31   Input ~ 0
 LS_5
-Text GLabel 2550 5725 2    31   Input ~ 0
+Text GLabel 2500 6125 2    31   Input ~ 0
 LS_6
-Text GLabel 2550 5825 2    31   Input ~ 0
+Text GLabel 2500 6225 2    31   Input ~ 0
 LS_7
-Text GLabel 2550 5925 2    31   Input ~ 0
+Text GLabel 2500 6325 2    31   Input ~ 0
 LS_8
 Wire Wire Line
@@
 Text Label 6050 3575 0    39   ~ 0
 Out_B4
+Text GLabel 1375 2050 0    39   Output ~ 0
+I_Sense_1
+Text GLabel 1400 4100 0    39   Output ~ 0
+I_Sense_2
+Text GLabel 4450 1975 0    39   Output ~ 0
+I_Sense_3
+Text GLabel 2550 5925 2    39   Input ~ 0
+I_Sense_4
+Text GLabel 2550 5625 2    39   Input ~ 0
+I_Sense_1
+Text GLabel 2550 5725 2    39   Input ~ 0
+I_Sense_2
+Text GLabel 2550 5825 2    39   Input ~ 0
+I_Sense_3
+Text GLabel 4400 4125 0    39   Output ~ 0
+I_Sense_4
+Text Notes 2900 5650 0    39   ~ 0
+A3
+Text Notes 2900 5750 0    39   ~ 0
+A2
+Text Notes 2900 5850 0    39   ~ 0
+A1
+Text Notes 2900 5950 0    39   ~ 0
+A0
 $EndSCHEMATC
