File: ArmPatchPanel_2019_Rev1/PatchPanel.sch (KiCad schematic (older format))
At the start: 0 parts

Commit message: completed patchpanel, wait on driveboard
completed all designs for patch panel, it's ready to go.
Laser, solenoid, servos ports were added. Waiting for futher instruction on laser, and solenoid input format.
Parts:
- added Conn1: AndersonPP, MRDT_Connectors:Anderson_3_Horisontal_Side_by_Side, symbol MRDT_Connectors:AndersonPP
- added Conn2, Conn3, Conn4: AndersonPP, Project Library:Anderson_3_Horisontal_Side_by_Side, symbol MRDT_Connectors:AndersonPP
Connections:
- net labels removed: +12V, GND
- wire segments 0 -> 9
Other:
- note added: "DriveBoard"
- note added: "MC1"
- note added: "MC2"
- note added: "Vin"
Changed lines of the file:
@@
 EESchema Schematic File Version 4
+LIBS:PatchPanel-cache
 EELAYER 26 0
 EELAYER END
@@
 $EndDescr
 $Comp
-L power:GND #PWR?
-U 1 1 5BC66334
-P 2950 2500
-F 0 "#PWR?" H 2950 2250 50  0001 C CNN
-F 1 "GND" H 2955 2327 50  0000 C CNN
-F 2 "" H 2950 2500 50  0001 C CNN
-F 3 "" H 2950 2500 50  0001 C CNN
-	1    2950 2500
+L MRDT_Connectors:AndersonPP Conn1
+U 1 1 5BCA5207
+P 3250 2500
+F 0 "Conn1" H 3000 2650 60  0000 C CNN
+F 1 "AndersonPP" H 3456 2781 60  0001 C CNN
+F 2 "MRDT_Connectors:Anderson_3_Horisontal_Side_by_Side" H 3100 1950 60  0001 C CNN
+F 3 "" H 3100 1950 60  0001 C CNN
+	1    3250 2500
 	1    0    0    -1
 $EndComp
 $Comp
-L power:+12V #PWR?
-U 1 1 5BC6636B
-P 2950 2050
-F 0 "#PWR?" H 2950 1900 50  0001 C CNN
-F 1 "+12V" H 2965 2223 50  0000 C CNN
-F 2 "" H 2950 2050 50  0001 C CNN
-F 3 "" H 2950 2050 50  0001 C CNN
-	1    2950 2050
+L MRDT_Connectors:AndersonPP Conn1
+U 2 1 5BCA52E0
+P 3250 2700
+F 0 "Conn1" H 3000 2850 60  0000 C CNN
+F 1 "AndersonPP" H 3456 2981 60  0001 C CNN
+F 2 "MRDT_Connectors:Anderson_3_Horisontal_Side_by_Side" H 3100 2150 60  0001 C CNN
+F 3 "" H 3100 2150 60  0001 C CNN
+	2    3250 2700
 	1    0    0    -1
 $EndComp
+$Comp
+L MRDT_Connectors:AndersonPP Conn1
+U 3 1 5BCA6ABA
+P 3250 2900
+F 0 "Conn1" H 3000 3050 60  0000 C CNN
+F 1 "AndersonPP" H 3456 3181 60  0001 C CNN
+F 2 "MRDT_Connectors:Anderson_3_Horisontal_Side_by_Side" H 3100 2350 60  0001 C CNN
+F 3 "" H 3100 2350 60  0001 C CNN
+	3    3250 2900
+	1    0    0    -1
+$EndComp
+$Comp
+L MRDT_Connectors:AndersonPP Conn2
+U 1 1 5BCA6C87
+P 4200 2500
+F 0 "Conn2" H 3950 2650 60  0000 C CNN
+F 1 "AndersonPP" H 4406 2781 60  0001 C CNN
+F 2 "Project Library:Anderson_3_Horisontal_Side_by_Side" H 4050 1950 60  0001 C CNN
+F 3 "" H 4050 1950 60  0001 C CNN
+	1    4200 2500
+	1    0    0    -1
+$EndComp
+$Comp
+L MRDT_Connectors:AndersonPP Conn2
+U 2 1 5BCA6C8E
+P 4200 2700
+F 0 "Conn2" H 3950 2850 60  0000 C CNN
+F 1 "AndersonPP" H 4406 2981 60  0001 C CNN
+F 2 "Project Library:Anderson_3_Horisontal_Side_by_Side" H 4050 2150 60  0001 C CNN
+F 3 "" H 4050 2150 60  0001 C CNN
+	2    4200 2700
+	1    0    0    -1
+$EndComp
+$Comp
+L MRDT_Connectors:AndersonPP Conn2
+U 3 1 5BCA6C95
+P 4200 2900
+F 0 "Conn2" H 3950 3050 60  0000 C CNN
+F 1 "AndersonPP" H 4406 3181 60  0001 C CNN
+F 2 "Project Library:Anderson_3_Horisontal_Side_by_Side" H 4050 2350 60  0001 C CNN
+F 3 "" H 4050 2350 60  0001 C CNN
+	3    4200 2900
+	1    0    0    -1
+$EndComp
+$Comp
+L MRDT_Connectors:AndersonPP Conn3
+U 1 1 5BCA6F40
+P 5150 2500
+F 0 "Conn3" H 4900 2650 60  0000 C CNN
+F 1 "AndersonPP" H 5356 2781 60  0001 C CNN
+F 2 "Project Library:Anderson_3_Horisontal_Side_by_Side" H 5000 1950 60  0001 C CNN
+F 3 "" H 5000 1950 60  0001 C CNN
+	1    5150 2500
+	1    0    0    -1
+$EndComp
+$Comp
+L MRDT_Connectors:AndersonPP Conn3
+U 2 1 5BCA6F47
+P 5150 2700
+F 0 "Conn3" H 4900 2850 60  0000 C CNN
+F 1 "AndersonPP" H 5356 2981 60  0001 C CNN
+F 2 "Project Library:Anderson_3_Horisontal_Side_by_Side" H 5000 2150 60  0001 C CNN
+F 3 "" H 5000 2150 60  0001 C CNN
+	2    5150 2700
+	1    0    0    -1
+$EndComp
+$Comp
+L MRDT_Connectors:AndersonPP Conn3
+U 3 1 5BCA6F4E
+P 5150 2900
+F 0 "Conn3" H 4900 3050 60  0000 C CNN
+F 1 "AndersonPP" H 5356 3181 60  0001 C CNN
+F 2 "Project Library:Anderson_3_Horisontal_Side_by_Side" H 5000 2350 60  0001 C CNN
+F 3 "" H 5000 2350 60  0001 C CNN
+	3    5150 2900
+	1    0    0    -1
+$EndComp
+$Comp
+L MRDT_Connectors:AndersonPP Conn4
+U 1 1 5BCA6F55
+P 6100 2500
+F 0 "Conn4" H 5850 2650 60  0000 C CNN
+F 1 "AndersonPP" H 6306 2781 60  0001 C CNN
+F 2 "Project Library:Anderson_3_Horisontal_Side_by_Side" H 5950 1950 60  0001 C CNN
+F 3 "" H 5950 1950 60  0001 C CNN
+	1    6100 2500
+	1    0    0    -1
+$EndComp
+$Comp
+L MRDT_Connectors:AndersonPP Conn4
+U 2 1 5BCA6F5C
+P 6100 2700
+F 0 "Conn4" H 5850 2850 60  0000 C CNN
+F 1 "AndersonPP" H 6306 2981 60  0001 C CNN
+F 2 "Project Library:Anderson_3_Horisontal_Side_by_Side" H 5950 2150 60  0001 C CNN
+F 3 "" H 5950 2150 60  0001 C CNN
+	2    6100 2700
+	1    0    0    -1
+$EndComp
+$Comp
+L MRDT_Connectors:AndersonPP Conn4
+U 3 1 5BCA6F63
+P 6100 2900
+F 0 "Conn4" H 5850 3050 60  0000 C CNN
+F 1 "AndersonPP" H 6306 3181 60  0001 C CNN
+F 2 "Project Library:Anderson_3_Horisontal_Side_by_Side" H 5950 2350 60  0001 C CNN
+F 3 "" H 5950 2350 60  0001 C CNN
+	3    6100 2900
+	1    0    0    -1
+$EndComp
+Wire Wire Line
+	3650 2400 4600 2400
+Wire Wire Line
+	5550 2400 4600 2400
+Connection ~ 4600 2400
+Wire Wire Line
+	5550 2400 6500 2400
+Connection ~ 5550 2400
+Wire Wire Line
+	3650 2600 4600 2600
+Connection ~ 4600 2600
+Wire Wire Line
+	4600 2600 5550 2600
+Connection ~ 5550 2600
+Wire Wire Line
+	5550 2600 6500 2600
+Wire Wire Line
+	3650 2800 4600 2800
+Connection ~ 4600 2800
+Wire Wire Line
+	4600 2800 5550 2800
+Connection ~ 5550 2800
+Wire Wire Line
+	5550 2800 6500 2800
+Text Notes 3250 2200 0    79   ~ 0
+Vin
+Text Notes 4000 2200 0    79   ~ 0
+DriveBoard
+Text Notes 5150 2200 0    79   ~ 0
+MC1
+Text Notes 6100 2200 0    79   ~ 0
+MC2
 $EndSCHEMATC

Commit message: added another molex2 on patch panel
Parts:
- added C1, C2: 10uF, Capacitor_SMD:C_0603_1608Metric_Pad1.05x0.95mm_HandSolder, symbol Device:C
- added Conn5: Molex_SL_02, MRDT_Connectors:MOLEX_SL_02_Vertical, symbol MRDT_Connectors:Molex_SL_02
- added U1: OKI, MRDT_Devices:OKI_Horizontal, symbol MRDT_Devices:OKI
Connections:
- net labels added: +5V, GND
- wire segments 9 -> 23
Changed lines of the file:
@@
 Text Notes 6100 2200 0    79   ~ 0
 MC2
+$Comp
+L Device:C C1
+U 1 1 5BD391BD
+P 6700 2450
+F 0 "C1" H 6815 2496 50  0000 L CNN
+F 1 "10uF" H 6815 2405 50  0000 L CNN
+F 2 "Capacitor_SMD:C_0603_1608Metric_Pad1.05x0.95mm_HandSolder" H 6738 2300 50  0001 C CNN
+F 3 "~" H 6700 2450 50  0001 C CNN
+	1    6700 2450
+	1    0    0    -1
+$EndComp
+$Comp
+L Device:C C2
+U 1 1 5BD39264
+P 7800 2450
+F 0 "C2" H 7915 2496 50  0000 L CNN
+F 1 "10uF" H 7915 2405 50  0000 L CNN
+F 2 "Capacitor_SMD:C_0603_1608Metric_Pad1.05x0.95mm_HandSolder" H 7838 2300 50  0001 C CNN
+F 3 "~" H 7800 2450 50  0001 C CNN
+	1    7800 2450
+	1    0    0    -1
+$EndComp
+$Comp
+L MRDT_Connectors:Molex_SL_02 Conn5
+U 1 1 5BD39375
+P 8550 2500
+F 0 "Conn5" H 8677 2658 60  0000 L CNN
+F 1 "Molex_SL_02" H 8677 2552 60  0000 L CNN
+F 2 "MRDT_Connectors:MOLEX_SL_02_Vertical" H 8550 2400 60  0001 C CNN
+F 3 "" H 8550 2400 60  0001 C CNN
+	1    8550 2500
+	1    0    0    -1
+$EndComp
+Wire Wire Line
+	6500 2600 6700 2600
+Connection ~ 6500 2600
+Connection ~ 6700 2600
+Wire Wire Line
+	6500 2400 6500 2300
+Wire Wire Line
+	6500 2300 6700 2300
+Connection ~ 6500 2400
+Wire Wire Line
+	6700 2600 7150 2600
+$Comp
+L MRDT_Devices:OKI U1
+U 1 1 5BD39164
+P 7250 2400
+F 0 "U1" H 7300 2350 60  0001 C CNN
+F 1 "OKI" H 7450 2680 60  0000 C CNN
+F 2 "MRDT_Devices:OKI_Horizontal" H 7050 2300 60  0001 C CNN
+F 3 "" H 7050 2300 60  0001 C CNN
+	1    7250 2400
+	0    -1   -1   0
+$EndComp
+Wire Wire Line
+	6700 2300 7450 2300
+Wire Wire Line
+	7450 2300 7450 2200
+Connection ~ 6700 2300
+Wire Wire Line
+	7450 2300 7450 2600
+Wire Wire Line
+	7450 2600 7800 2600
+Connection ~ 7450 2300
+Wire Wire Line
+	7150 1800 7800 1800
+Wire Wire Line
+	7800 1800 7800 2300
+Wire Wire Line
+	7800 2300 8350 2300
+Wire Wire Line
+	8350 2300 8350 2350
+Connection ~ 7800 2300
+Wire Wire Line
+	7800 2600 8350 2600
+Wire Wire Line
+	8350 2600 8350 2450
+Connection ~ 7800 2600
+Text Label 8250 2300 0    50   ~ 0
++5V
+Text Label 8350 2550 0    50   ~ 0
+GND
 $EndSCHEMATC
