File: ArmDriveBoard_2019_Rev1/DriveBoard_Hardware.sch (KiCad schematic (older format))
At the start: 12 parts, among them U1 TM4C129E_Launchpad, U2 MAX_3232

Commit message: completed patchpanel, wait on driveboard
completed all designs for patch panel, it's ready to go.
Laser, solenoid, servos ports were added. Waiting for futher instruction on laser, and solenoid input format.
Parts:
- added Conn?: Servo 2, symbol MRDT_Connectors:Molex_SL_03
- added Conn?: Servo 1, symbol MRDT_Connectors:Molex_SL_03
- added Conn?: Servo 3, symbol MRDT_Connectors:Molex_SL_03
- added Conn?: Laser 1, symbol MRDT_Connectors:Molex_SL_02
- added Conn?: Laser 2, symbol MRDT_Connectors:Molex_SL_02
- added Conn?: Solenoid, symbol MRDT_Connectors:Molex_SL_02
- Conn2: value Molex_SL_05 -> MoCo 1
Connections:
- net labels added: Servo1_PWM, Servo2_PWM, Servo3_PWM
Changed lines of the file:
@@
 EESchema Schematic File Version 4
+LIBS:DriveBoard_Hardware-cache
 EELAYER 26 0
 EELAYER END
@@
 Text Notes 7800 2800 0    98   ~ 20
 Conectors
-Wire Notes Line
-	5000 2650 8800 2650
-Wire Notes Line
-	8800 4350 8800 1550
-Wire Notes Line
-	7450 4350 7450 2650
-Wire Notes Line
-	5000 1550 5000 4350
-Wire Notes Line
-	3150 1550 3150 4350
-Wire Notes Line
-	3150 4350 8800 4350
 Wire Wire Line
 	5350 3500 5450 3500
@@
 Wire Wire Line
 	6250 2100 5900 2100
-Wire Notes Line
-	3150 1550 8800 1550
 $Comp
 L power:+5V #PWR0101
@@
 P 8350 3450
 F 0 "Conn2" H 8477 3758 60  0000 L CNN
-F 1 "Molex_SL_05" H 8477 3652 60  0000 L CNN
+F 1 "MoCo 1" H 8477 3652 60  0000 L CNN
 F 2 "" H 8350 3450 60  0001 C CNN
 F 3 "" H 8350 3450 60  0001 C CNN
@@
 	1    0    0    -1
 $EndComp
+$Comp
+L MRDT_Connectors:Molex_SL_03 Conn?
+U 1 1 5BCAB0BE
+P 8350 5150
+F 0 "Conn?" H 8478 5358 60  0000 L CNN
+F 1 "Servo 2" H 8478 5252 60  0000 L CNN
+F 2 "" H 8350 5150 60  0001 C CNN
+F 3 "" H 8350 5150 60  0001 C CNN
+	1    8350 5150
+	1    0    0    -1
+$EndComp
+Text GLabel 8150 4900 0    50   UnSpc ~ 0
+GND
+Text GLabel 8150 5000 0    50   Input ~ 0
++5V
+Text GLabel 8150 5100 0    50   Input ~ 0
+Servo2_PWM
+Text GLabel 3600 3600 0    50   Input ~ 0
+Servo1_PWM
+$Comp
+L MRDT_Connectors:Molex_SL_03 Conn?
+U 1 1 5BCAC1D7
+P 8350 4650
+F 0 "Conn?" H 8478 4858 60  0000 L CNN
+F 1 "Servo 1" H 8478 4752 60  0000 L CNN
+F 2 "" H 8350 4650 60  0001 C CNN
+F 3 "" H 8350 4650 60  0001 C CNN
+	1    8350 4650
+	1    0    0    -1
+$EndComp
+Text GLabel 8150 4400 0    50   UnSpc ~ 0
+GND
+Text GLabel 8150 4500 0    50   Input ~ 0
++5V
+Text GLabel 8150 4600 0    50   Input ~ 0
+Servo1_PWM
+$Comp
+L MRDT_Connectors:Molex_SL_03 Conn?
+U 1 1 5BCAC820
+P 8350 5550
+F 0 "Conn?" H 8478 5758 60  0000 L CNN
+F 1 "Servo 3" H 8478 5652 60  0000 L CNN
+F 2 "" H 8350 5550 60  0001 C CNN
+F 3 "" H 8350 5550 60  0001 C CNN
+	1    8350 5550
+	1    0    0    -1
+$EndComp
+Text GLabel 8150 5300 0    50   UnSpc ~ 0
+GND
+Text GLabel 8150 5400 0    50   Input ~ 0
++5V
+Text GLabel 8150 5500 0    50   Input ~ 0
+Servo3_PWM
+Text GLabel 3600 3700 0    50   Input ~ 0
+Servo2_PWM
+Text GLabel 3600 3800 0    50   Input ~ 0
+Servo3_PWM
+$Comp
+L MRDT_Connectors:Molex_SL_02 Conn?
+U 1 1 5BCADF34
+P 6350 4600
+F 0 "Conn?" H 6478 4758 60  0000 L CNN
+F 1 "Laser 1" H 6478 4652 60  0000 L CNN
+F 2 "" H 6350 4500 60  0001 C CNN
+F 3 "" H 6350 4500 60  0001 C CNN
+	1    6350 4600
+	1    0    0    -1
+$EndComp
+$Comp
+L MRDT_Connectors:Molex_SL_02 Conn?
+U 1 1 5BCADFB6
+P 6350 5000
+F 0 "Conn?" H 6478 5158 60  0000 L CNN
+F 1 "Laser 2" H 6478 5052 60  0000 L CNN
+F 2 "" H 6350 4900 60  0001 C CNN
+F 3 "" H 6350 4900 60  0001 C CNN
+	1    6350 5000
+	1    0    0    -1
+$EndComp
+$Comp
+L MRDT_Connectors:Molex_SL_02 Conn?
+U 1 1 5BCAE57B
+P 6350 5350
+F 0 "Conn?" H 6477 5508 60  0000 L CNN
+F 1 "Solenoid" H 6477 5402 60  0000 L CNN
+F 2 "" H 6350 5250 60  0001 C CNN
+F 3 "" H 6350 5250 60  0001 C CNN
+	1    6350 5350
+	1    0    0    -1
+$EndComp
+Text GLabel 6150 4550 0    50   UnSpc ~ 0
+GND
+Text GLabel 6150 4950 0    50   UnSpc ~ 0
+GND
+Text GLabel 6150 5300 0    50   UnSpc ~ 0
+GND
 $EndSCHEMATC

Commit message: fixed driveboard, and add power filter on MotorController
Parts:
- added Conn10: AndersonPP, symbol MRDT_Connectors:AndersonPP
- added Q1, Q2: Q_NMOS_DGS, symbol Device:Q_NMOS_DGS
- gave numbers to parts that had none: 7
Connections:
- net labels added: +12V_Act, +12V_log, Laser_control, Solenoial_Control
- net labels removed: +12V
- wire segments 33 -> 45
Changed lines of the file:
@@
 $EndComp
 Text Label 5950 2100 0    60   ~ 0
-+12V
++12V_log
 Text Notes 8450 3350 1    60   ~ 0
 Motor 1
@@
 Text Notes 3900 1750 0    98   ~ 20
 TIVA
-Text Notes 6200 1900 0    98   ~ 20
+Text Notes 5950 1500 0    98   ~ 20
 Power Filtering
 Text Notes 7800 2800 0    98   ~ 20
@@
 $EndComp
 $Comp
-L MRDT_Devices:OKI U?
+L MRDT_Devices:OKI U3
 U 1 1 5BC6E00E
 P 6600 2200
-F 0 "U?" H 6650 2150 60  0001 C CNN
+F 0 "U3" H 6650 2150 60  0001 C CNN
 F 1 "OKI" H 6800 2481 60  0000 C CNN
 F 2 "" H 6400 2100 60  0001 C CNN
@@
 $EndComp
 $Comp
-L MRDT_Connectors:Molex_SL_03 Conn?
+L MRDT_Connectors:Molex_SL_03 Conn8
 U 1 1 5BCAB0BE
 P 8350 5150
-F 0 "Conn?" H 8478 5358 60  0000 L CNN
+F 0 "Conn8" H 8478 5358 60  0000 L CNN
 F 1 "Servo 2" H 8478 5252 60  0000 L CNN
 F 2 "" H 8350 5150 60  0001 C CNN
@@
 Servo1_PWM
 $Comp
-L MRDT_Connectors:Molex_SL_03 Conn?
+L MRDT_Connectors:Molex_SL_03 Conn7
 U 1 1 5BCAC1D7
 P 8350 4650
-F 0 "Conn?" H 8478 4858 60  0000 L CNN
+F 0 "Conn7" H 8478 4858 60  0000 L CNN
 F 1 "Servo 1" H 8478 4752 60  0000 L CNN
 F 2 "" H 8350 4650 60  0001 C CNN
@@
 Servo1_PWM
 $Comp
-L MRDT_Connectors:Molex_SL_03 Conn?
+L MRDT_Connectors:Molex_SL_03 Conn9
 U 1 1 5BCAC820
 P 8350 5550
-F 0 "Conn?" H 8478 5758 60  0000 L CNN
+F 0 "Conn9" H 8478 5758 60  0000 L CNN
 F 1 "Servo 3" H 8478 5652 60  0000 L CNN
 F 2 "" H 8350 5550 60  0001 C CNN
@@
 Servo3_PWM
 $Comp
-L MRDT_Connectors:Molex_SL_02 Conn?
+L MRDT_Connectors:Molex_SL_02 Conn4
 U 1 1 5BCADF34
 P 6350 4600
-F 0 "Conn?" H 6478 4758 60  0000 L CNN
+F 0 "Conn4" H 6478 4758 60  0000 L CNN
 F 1 "Laser 1" H 6478 4652 60  0000 L CNN
 F 2 "" H 6350 4500 60  0001 C CNN
@@
 $EndComp
 $Comp
-L MRDT_Connectors:Molex_SL_02 Conn?
+L MRDT_Connectors:Molex_SL_02 Conn5
 U 1 1 5BCADFB6
 P 6350 5000
-F 0 "Conn?" H 6478 5158 60  0000 L CNN
+F 0 "Conn5" H 6478 5158 60  0000 L CNN
 F 1 "Laser 2" H 6478 5052 60  0000 L CNN
 F 2 "" H 6350 4900 60  0001 C CNN
@@
 $EndComp
 $Comp
-L MRDT_Connectors:Molex_SL_02 Conn?
+L MRDT_Connectors:Molex_SL_02 Conn6
 U 1 1 5BCAE57B
 P 6350 5350
-F 0 "Conn?" H 6477 5508 60  0000 L CNN
+F 0 "Conn6" H 6477 5508 60  0000 L CNN
 F 1 "Solenoid" H 6477 5402 60  0000 L CNN
 F 2 "" H 6350 5250 60  0001 C CNN
@@
 Text GLabel 6150 5300 0    50   UnSpc ~ 0
 GND
+Wire Wire Line
+	6150 4450 5900 4450
+Wire Wire Line
+	6150 5200 5900 5200
+Wire Wire Line
+	5900 4850 6150 4850
+Wire Wire Line
+	5900 4450 5900 4850
+Wire Wire Line
+	5250 4400 5250 4600
+Wire Wire Line
+	5250 4600 5400 4600
+$Comp
+L Device:Q_NMOS_DGS Q1
+U 1 1 5BCAC99A
+P 5300 4800
+F 0 "Q1" H 5505 4846 50  0000 L CNN
+F 1 "Q_NMOS_DGS" H 5505 4755 50  0000 L CNN
+F 2 "" H 5500 4900 50  0001 C CNN
+F 3 "~" H 5300 4800 50  0001 C CNN
+	1    5300 4800
+	1    0    0    -1
+$EndComp
+Wire Wire Line
+	5900 5000 5900 4850
+Connection ~ 5900 4850
+$Comp
+L Device:Q_NMOS_DGS Q2
+U 1 1 5BCADB61
+P 5300 5350
+F 0 "Q2" H 5505 5396 50  0000 L CNN
+F 1 "Q_NMOS_DGS" H 5505 5305 50  0000 L CNN
+F 2 "" H 5500 5450 50  0001 C CNN
+F 3 "~" H 5300 5350 50  0001 C CNN
+	1    5300 5350
+	1    0    0    -1
+$EndComp
+Wire Wire Line
+	5400 5000 5900 5000
+Wire Wire Line
+	5250 4600 5250 5150
+Wire Wire Line
+	5250 5150 5400 5150
+Connection ~ 5250 4600
+Wire Wire Line
+	5400 5550 5900 5550
+Wire Wire Line
+	5900 5550 5900 5200
+$Comp
+L MRDT_Connectors:AndersonPP Conn10
+U 3 1 5BCB1124
+P 5500 1850
+F 0 "Conn10" H 5550 2100 60  0000 C CNN
+F 1 "AndersonPP" H 5750 2250 60  0001 C CNN
+F 2 "" H 5350 1300 60  0001 C CNN
+F 3 "" H 5350 1300 60  0001 C CNN
+	3    5500 1850
+	1    0    0    -1
+$EndComp
+Text GLabel 5900 1750 2    50   Input ~ 0
++12V_Act
+Text GLabel 5250 4400 2    50   Input ~ 0
++12V_Act
+Text GLabel 3600 2500 0    50   Input ~ 0
+Laser_control
+Text GLabel 5100 4800 0    50   Input ~ 0
+Laser_control
+Text GLabel 3600 2600 0    50   Input ~ 0
+Solenoial_Control
+Text GLabel 5100 5350 0    50   Input ~ 0
+Solenoial_Control
 $EndSCHEMATC

Commit message: Changed positioning a bit
Connections:
- net labels added: Solenoid_Control
Other:
- note added: "Connectors"
- note added: "Laser & Solenoid Control"
- note removed: "Conectors"

Commit message: finish PDR requirement check list
Parts:
- removed Q1: Q_NMOS_DGS, symbol Device:Q_NMOS_DGS
- added Q1: Q_NMOS_DGS, Package_TO_SOT_SMD:SOT-23, symbol Device:Q_NMOS_GSD
- Conn1: footprint (none) -> MRDT_Connectors:Anderson_3_Horisontal_Side_by_Side
- Conn1: renamed from Conn10; footprint (none) -> MRDT_Connectors:Anderson_3_Horisontal_Side_by_Side
- Conn2: footprint (none) -> MRDT_Connectors:MOLEX_SL_03_Horizontal; symbol MRDT_Connectors:Molex_SL_05 -> MRDT_Connectors:Molex_SL_03
- Conn3: value Molex_SL_05 -> MoCo 2; footprint (none) -> MRDT_Connectors:MOLEX_SL_03_Horizontal; symbol MRDT_Connectors:Molex_SL_05 -> MRDT_Connectors:Molex_SL_03
- Conn4, Conn5, Conn6: footprint (none) -> MRDT_Connectors:MOLEX_SL_02_Horizontal
- Conn7, Conn8, Conn9: footprint (none) -> MRDT_Connectors:MOLEX_SL_03_Vertical
- Q2: footprint (none) -> Package_TO_SOT_SMD:SOT-23; symbol Device:Q_NMOS_DGS -> Device:Q_NMOS_GSD
- U1: footprint (none) -> MRDT_Shields:TM4C129E_Launchpad_X7
- U2: footprint (none) -> MRDT_ICs:SOIC_16_3.9x9.9mm_Pitch1.27mm
- U3: footprint (none) -> MRDT_Devices:OKI_Horizontal
Connections:
- no-connect marks 4 -> 0
Other:
- note removed: "Motor 1"
Changed lines of the file:
@@
 Text Label 5950 1750 0    60   ~ 0
 +12V_log
-Text Notes 8450 3350 1    60   ~ 0
-Motor 1
 $Comp
 L Device:C_Small C4
@@
 Text GLabel 4200 2600 2    60   Output ~ 0
 TX_2_IC
-NoConn ~ 8150 3000
-NoConn ~ 8150 3100
-NoConn ~ 8150 3700
-NoConn ~ 8150 3800
 Text GLabel 6800 4000 2    60   Output ~ 0
 TX_2_SL
@@
 F 0 "U1" H 3300 3000 60  0000 L CNN
 F 1 "TM4C129E_Launchpad" H 3250 4250 60  0001 L CNN
-F 2 "" H 3500 3050 60  0001 C CNN
+F 2 "MRDT_Shields:TM4C129E_Launchpad_X7" H 3500 3050 60  0001 C CNN
 F 3 "" H 3500 3050 60  0001 C CNN
 	5    3500 3050
@@
 F 0 "U1" H 4050 3000 60  0000 L CNN
 F 1 "TM4C129E_Launchpad" H 3750 4250 60  0000 L CNN
-F 2 "" H 4000 3050 60  0001 C CNN
+F 2 "MRDT_Shields:TM4C129E_Launchpad_X7" H 4000 3050 60  0001 C CNN
 F 3 "" H 4000 3050 60  0001 C CNN
 	6    4000 3050
@@
 F 0 "U1" H 3500 4200 60  0000 L CNN
 F 1 "TM4C129E_Launchpad" H 2750 4050 60  0001 L CNN
-F 2 "" H 3500 4250 60  0001 C CNN
+F 2 "MRDT_Shields:TM4C129E_Launchpad_X7" H 3500 4250 60  0001 C CNN
 F 3 "" H 3500 4250 60  0001 C CNN
 	7    3500 4250
@@
 F 0 "U1" H 4050 4200 60  0000 L CNN
 F 1 "TM4C129E_Launchpad" H 3250 4050 60  0001 L CNN
-F 2 "" H 4000 4250 60  0001 C CNN
+F 2 "MRDT_Shields:TM4C129E_Launchpad_X7" H 4000 4250 60  0001 C CNN
 F 3 "" H 4000 4250 60  0001 C CNN
 	8    4000 4250
@@
 F 0 "Conn1" H 5550 2100 60  0000 C CNN
 F 1 "AndersonPP" H 5250 1950 60  0000 C CNN
-F 2 "" H 5350 1300 60  0001 C CNN
+F 2 "MRDT_Connectors:Anderson_3_Horisontal_Side_by_Side" H 5350 1300 60  0001 C CNN
 F 3 "" H 5350 1300 60  0001 C CNN
 	2    5500 1850
@@
 F 0 "Conn1" H 5550 2100 60  0000 C CNN
 F 1 "AndersonPP" H 5250 2250 60  0000 C CNN
-F 2 "" H 5350 1600 60  0001 C CNN
+F 2 "MRDT_Connectors:Anderson_3_Horisontal_Side_by_Side" H 5350 1600 60  0001 C CNN
 F 3 "" H 5350 1600 60  0001 C CNN
 	1    5500 2150
@@
 F 0 "U3" H 6650 1800 60  0001 C CNN
 F 1 "OKI" H 6800 2131 60  0000 C CNN
-F 2 "" H 6400 1750 60  0001 C CNN
+F 2 "MRDT_Devices:OKI_Horizontal" H 6400 1750 60  0001 C CNN
 F 3 "" H 6400 1750 60  0001 C CNN
 	1    6600 1850
@@
 F 0 "U2" H 5950 4000 60  0000 C CNN
 F 1 "MAX_3232" H 6250 5281 60  0000 C CNN
-F 2 "" H 5900 3450 60  0001 C CNN
+F 2 "MRDT_ICs:SOIC_16_3.9x9.9mm_Pitch1.27mm" H 5900 3450 60  0001 C CNN
 F 3 "" H 5900 3450 60  0001 C CNN
 	1    5900 4050
@@
 $EndComp
 $Comp
-L MRDT_Connectors:Molex_SL_05 Conn2
-U 1 1 5BC6E438
-P 8350 3450
-F 0 "Conn2" H 8477 3758 60  0000 L CNN
-F 1 "MoCo 1" H 8477 3652 60  0000 L CNN
-F 2 "" H 8350 3450 60  0001 C CNN
-F 3 "" H 8350 3450 60  0001 C CNN
-	1    8350 3450
-	1    0    0    -1
-$EndComp
-$Comp
-L MRDT_Connectors:Molex_SL_05 Conn3
+L MRDT_Connectors:Molex_SL_03 Conn3
 U 1 1 5BC6E491
 P 8350 4150
 F 0 "Conn3" H 8477 4458 60  0000 L CNN
-F 1 "Molex_SL_05" H 8477 4352 60  0000 L CNN
-F 2 "" H 8350 4150 60  0001 C CNN
+F 1 "MoCo 2" H 8477 4352 60  0000 L CNN
+F 2 "MRDT_Connectors:MOLEX_SL_03_Horizontal" H 8350 4150 60  0001 C CNN
 F 3 "" H 8350 4150 60  0001 C CNN
 	1    8350 4150
@@
 F 0 "Conn8" H 8478 5358 60  0000 L CNN
 F 1 "Servo 2" H 8478 5252 60  0000 L CNN
-F 2 "" H 8350 5150 60  0001 C CNN
+F 2 "MRDT_Connectors:MOLEX_SL_03_Vertical" H 8350 5150 60  0001 C CNN
 F 3 "" H 8350 5150 60  0001 C CNN
 	1    8350 5150
@@
 F 0 "Conn7" H 8478 4858 60  0000 L CNN
 F 1 "Servo 1" H 8478 4752 60  0000 L CNN
-F 2 "" H 8350 4650 60  0001 C CNN
+F 2 "MRDT_Connectors:MOLEX_SL_03_Vertical" H 8350 4650 60  0001 C CNN
 F 3 "" H 8350 4650 60  0001 C CNN
 	1    8350 4650
@@
 F 0 "Conn9" H 8478 5758 60  0000 L CNN
 F 1 "Servo 3" H 8478 5652 60  0000 L CNN
-F 2 "" H 8350 5550 60  0001 C CNN
+F 2 "MRDT_Connectors:MOLEX_SL_03_Vertical" H 8350 5550 60  0001 C CNN
 F 3 "" H 8350 5550 60  0001 C CNN
 	1    8350 5550
@@
 F 0 "Conn4" H 6428 5108 60  0000 L CNN
 F 1 "Laser 1" H 6428 5002 60  0000 L CNN
-F 2 "" H 6300 4850 60  0001 C CNN
+F 2 "MRDT_Connectors:MOLEX_SL_02_Horizontal" H 6300 4850 60  0001 C CNN
 F 3 "" H 6300 4850 60  0001 C CNN
 	1    6300 4950
@@
 F 0 "Conn5" H 6428 5508 60  0000 L CNN
 F 1 "Laser 2" H 6428 5402 60  0000 L CNN
-F 2 "" H 6300 5250 60  0001 C CNN
+F 2 "MRDT_Connectors:MOLEX_SL_02_Horizontal" H 6300 5250 60  0001 C CNN
 F 3 "" H 6300 5250 60  0001 C CNN
 	1    6300 5350
@@
 F 0 "Conn6" H 6427 5858 60  0000 L CNN
 F 1 "Solenoid" H 6427 5752 60  0000 L CNN
-F 2 "" H 6300 5600 60  0001 C CNN
+F 2 "MRDT_Connectors:MOLEX_SL_02_Horizontal" H 6300 5600 60  0001 C CNN
 F 3 "" H 6300 5600 60  0001 C CNN
 	1    6300 5700
@@
 Wire Wire Line
 	5200 4950 5350 4950
-$Comp
-L Device:Q_NMOS_DGS Q1
-U 1 1 5BCAC99A
-P 5250 5150
-F 0 "Q1" H 5455 5196 50  0000 L CNN
-F 1 "Q_NMOS_DGS" H 5455 5105 50  0000 L CNN
-F 2 "" H 5450 5250 50  0001 C CNN
-F 3 "~" H 5250 5150 50  0001 C CNN
-	1    5250 5150
-	1    0    0    -1
-$EndComp
 Wire Wire Line
 	5850 5350 5850 5200
 Connection ~ 5850 5200
 $Comp
-L Device:Q_NMOS_DGS Q2
+L Device:Q_NMOS_GSD Q2
 U 1 1 5BCADB61
 P 5250 5700
 F 0 "Q2" H 5455 5746 50  0000 L CNN
 F 1 "Q_NMOS_DGS" H 5455 5655 50  0000 L CNN
-F 2 "" H 5450 5800 50  0001 C CNN
+F 2 "Package_TO_SOT_SMD:SOT-23" H 5450 5800 50  0001 C CNN
 F 3 "~" H 5250 5700 50  0001 C CNN
 	1    5250 5700
@@
 	5850 5900 5850 5550
 $Comp
-L MRDT_Connectors:AndersonPP Conn10
+L MRDT_Connectors:AndersonPP Conn1
 U 3 1 5BCB1124
 P 5500 1500
-F 0 "Conn10" H 5550 1750 60  0000 C CNN
+F 0 "Conn1" H 5550 1750 60  0000 C CNN
 F 1 "AndersonPP" H 5750 1900 60  0001 C CNN
-F 2 "" H 5350 950 60  0001 C CNN
+F 2 "MRDT_Connectors:Anderson_3_Horisontal_Side_by_Side" H 5350 950 60  0001 C CNN
 F 3 "" H 5350 950 60  0001 C CNN
 	3    5500 1500
@@
 Wire Wire Line
 	5200 4750 5200 4950
+$Comp
+L Device:Q_NMOS_GSD Q1
+U 1 1 5BD01A10
+P 5250 5150
+F 0 "Q1" H 5455 5196 50  0000 L CNN
+F 1 "Q_NMOS_DGS" H 5455 5105 50  0000 L CNN
+F 2 "Package_TO_SOT_SMD:SOT-23" H 5450 5250 50  0001 C CNN
+F 3 "~" H 5250 5150 50  0001 C CNN
+	1    5250 5150
+	1    0    0    -1
+$EndComp
+$Comp
+L MRDT_Connectors:Molex_SL_03 Conn2
+U 1 1 5BC6E438
+P 8350 3450
+F 0 "Conn2" H 8477 3758 60  0000 L CNN
+F 1 "MoCo 1" H 8477 3652 60  0000 L CNN
+F 2 "MRDT_Connectors:MOLEX_SL_03_Horizontal" H 8350 3450 60  0001 C CNN
+F 3 "" H 8350 3450 60  0001 C CNN
+	1    8350 3450
+	1    0    0    -1
+$EndComp
 $EndSCHEMATC

Commit message: Made changes to schematics and boards
Approved for PDR by Andrew
Changed lines of the file:
@@
 	0    1    1    0
 $EndComp
-Text Notes 2900 2150 0    60   ~ 0
+Text Notes 2900 2250 0    60   ~ 0
 Serial 6
 Text Notes 4250 2450 0    60   ~ 0
@@
 Text GLabel 8150 3400 0    60   Output ~ 0
 RX_1_SL
-Text GLabel 3300 2300 0    60   Output ~ 0
+Text GLabel 3300 2400 0    60   Output ~ 0
 TX_1_IC
-Text GLabel 3300 2200 0    60   Input ~ 0
+Text GLabel 3300 2300 0    60   Input ~ 0
 RX_1_IC
 Text GLabel 5700 4000 0    60   Input ~ 0
@@
 Text GLabel 5200 4750 2    50   Input ~ 0
 +12V_Act
-Text GLabel 3300 2500 0    50   Input ~ 0
+Text GLabel 3300 2700 0    50   Input ~ 0
 Laser_control
 Text GLabel 5050 5150 0    50   Input ~ 0
 Laser_control
-Text GLabel 3300 2600 0    50   Input ~ 0
+Text GLabel 3300 2800 0    50   Input ~ 0
 Solenoial_Control
 Text GLabel 5050 5700 0    50   Input ~ 0

Commit message: Schematic layout
Parts:
- added Conn10, Conn11, Conn12: AndersonPP, Project Library:Anderson_3_Horisontal_Side_by_Side, symbol MRDT_Connectors:AndersonPP
- added Conn13: Molex_SL_02, MRDT_Connectors:MOLEX_SL_02_Horizontal, symbol MRDT_Connectors:Molex_SL_02
- Conn7, Conn8, Conn9: footprint MRDT_Connectors:MOLEX_SL_03_Vertical -> MRDT_Connectors:MOLEX_SL_03_Horizontal
- U1: footprint MRDT_Shields:TM4C129E_Launchpad_X7 -> Project Library:TM4C129E_Launchpad_FULL_ext
Connections:
- wire segments 45 -> 55
Other:
- note added: "DriveBoard"
- note added: "MC1"
- note added: "MC2"
- note added: "Power Filtering & Patch Panel"
- note added: "Vin"
- note removed: "Power Filtering"
