File: ArmDriveBoard_2019_Rev1/DriveBoard_Hardware.kicad_pcb (KiCad board)
At the start: 2 copper layers, 20 parts, among them Q1 Q_NMOS_DGS, Q2 Q_NMOS_DGS, U1 TM4C129E_Launchpad, U2 MAX_3232, U3 OKI

Commit message: Schematic layout
Parts:
- added Conn10: AndersonPP, Project Library:Anderson_3_Horisontal_Side_by_Side, F.Cu at (160.5, 114.2)
- added Conn11: AndersonPP, Project Library:Anderson_3_Horisontal_Side_by_Side, F.Cu at (174.2, 114.2)
- added Conn12: AndersonPP, Project Library:Anderson_3_Horisontal_Side_by_Side, F.Cu at (148.3, 114.2)
- added Conn13: Molex_SL_02, MRDT_Connectors:MOLEX_SL_02_Horizontal, F.Cu at (214.4, 63.9)
- Conn7, Conn8, Conn9: footprint MRDT_Connectors:MOLEX_SL_03_Vertical -> MRDT_Connectors:MOLEX_SL_03_Horizontal
- U1: footprint MRDT_Shields:TM4C129E_Launchpad_X7 -> Project Library:TM4C129E_Launchpad_FULL_ext
- moved U3 93.1 mm to (227.3, 94.4), turned to 90 degrees
- moved C3 93.0 mm to (222.9, 90.7), turned to 90 degrees
- moved Conn2 90.0 mm to (238.6, 63.9)
- moved Conn3 89.3 mm to (226.1, 63.9)
- moved C1 84.3 mm to (222.1, 87.1), turned to 0 degrees
- moved Conn6 77.2 mm to (202.1, 63.9)
- moved Conn5 68.9 mm to (184.5, 63.9)
- moved Conn4 68.3 mm to (174.7, 63.9)
- moved U2 67.6 mm to (211.8, 94.4)
- moved C4 63.2 mm to (201.7, 91.0)
- moved C5 63.0 mm to (201.5, 94.6)
- moved C6 60.3 mm to (184.7, 91.2), turned to 90 degrees
- moved C2 59.8 mm to (197.5, 91.0), turned to 90 degrees
- moved Q1 58.4 mm to (174.3, 76.1), turned to 270 degrees
- moved Q2 57.0 mm to (180.0, 76.3), turned to 270 degrees
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Connections:
- U1 pad PD2: RX_1_IC -> Net-(U1-PadPD2)
- U1 pad PD4: Laser_control -> Net-(U1-PadPD4)
- U1 pad PD5: Solenoial_Control -> Net-(U1-PadPD5)
- U1 pad PP0: TX_1_IC -> RX_1_IC
- U1 pad PP1: Net-(U1-PadPP1) -> TX_1_IC
- U1 pad PP4: Net-(U1-PadPP4) -> Solenoial_Control
- U1 pad PQ0: Net-(U1-PadPQ0) -> Laser_control

Commit message: finshed wiring
Parts:
- moved Conn3 12.5 mm to (238.6, 64.0)
- moved Conn2 11.6 mm to (226.9, 64.0)
Routing:
- net GND: track 0.00 -> 400.1 mm, vias 0 -> 11
- net +5V: track 0.00 -> 278.8 mm, vias 0 -> 12
- net /+12V_log: track 0.00 -> 101.6 mm, vias 0 -> 2
- net Servo3_PWM: track 0.00 -> 93.6 mm, vias 0 -> 2
- net +12V_Act: track 0.00 -> 87.7 mm, vias 0 -> 2
- net Laser_control: track 0.00 -> 86.3 mm, vias 0 -> 4
- net Net-(U1-PadRese): track 0.00 -> 82.5 mm, vias 0 -> 3
- net Servo2_PWM: track 0.00 -> 76.9 mm, vias 0 -> 2
- net TX_2_SL: track 0.00 -> 75.5 mm, vias 0 -> 4
- net RX_2_SL: track 0.00 -> 70.4 mm, vias 0 -> 2
- net Net-(U1-Pad+3V3): track 0.00 -> 70.1 mm, vias 0 -> 1
- net TX_1_IC: track 0.00 -> 64.6 mm, vias 0 -> 5
- net RX_1_IC: track 0.00 -> 63.5 mm, vias 0 -> 5
- net Servo1_PWM: track 0.00 -> 59.7 mm
- net RX_2_IC: track 0.00 -> 52.6 mm, vias 0 -> 2
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
Commit message: schematic
Parts:
- Conn13: value Molex_SL_02 -> PowerOut
- moved Conn7 25.3 mm to (125.7, 63.9)
- moved Conn9 25.2 mm to (150.9, 63.9)
Routing:
- net Servo1_PWM: track 59.7 -> 86.3 mm, vias 0 -> 2
- net Servo3_PWM: track 93.6 -> 68.4 mm
Changed lines of the file:
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@@
     (thickness 1.6)
     (drawings 0)
-    (tracks 381)
+    (tracks 388)
     (zones 0)
     (modules 24)
@@
   )
   (module MRDT_Connectors:MOLEX_SL_03_Horizontal (layer F.Cu)
-    (at 125.6665 64.0715)
+    (at 150.876 63.9445)
     (fp_text reference Conn9 (at -1.27 2.54) (layer F.SilkS) hide
       (effects (font (size 1 1) (thickness 0.15)))
@@
   )
   (module MRDT_Connectors:MOLEX_SL_03_Horizontal (layer F.Cu)
-    (at 150.9395 63.9445)
+    (at 125.6665 63.881)
     (fp_text reference Conn7 (at -1.27 2.54) (layer F.SilkS) hide
       (effects (font (size 1 1) (thickness 0.15)))
@@
       (effects (font (size 1 1) (thickness 0.15)))
     )
-    (fp_text value Molex_SL_02 (at 0.127 -3.556) (layer F.Fab)
+    (fp_text value PowerOut (at 0.127 -3.556) (layer F.Fab)
       (effects (font (size 1 1) (thickness 0.15)))
     )
@@
   (via (at 138.303 66.294) (size 0.8) (drill 0.4) (layers F.Cu B.Cu) (net 9))
   (segment (start 133.731 66.294) (end 138.303 66.294) (width 0.25) (layer B.Cu) (net 9))
-  (segment (start 138.303 66.294) (end 138.303 63.881) (width 0.25) (layer F.Cu) (net 9))
   (via (at 125.6665 66.294) (size 0.8) (drill 0.4) (layers F.Cu B.Cu) (net 9))
   (segment (start 133.731 66.294) (end 125.6665 66.294) (width 0.25) (layer B.Cu) (net 9))
@@
   (segment (start 213.1695 82.7405) (end 213.0425 82.7405) (width 0.25) (layer F.Cu) (net 9))
   (segment (start 213.0425 82.7405) (end 198.247 82.7405) (width 0.25) (layer F.Cu) (net 9))
+  (segment (start 138.303 66.294) (end 138.303 63.881) (width 0.25) (layer F.Cu) (net 9))
   (segment (start 141.577602 110.488) (end 151.892 110.488) (width 0.25) (layer F.Cu) (net 10))
   (segment (start 137.9855 110.488) (end 141.577602 110.488) (width 0.25) (layer F.Cu) (net 10))
@@
   (segment (start 179.0725 75.2635) (end 179.0725 71.6255) (width 0.25) (layer F.Cu) (net 16))
   (segment (start 192.278 82.423) (end 192.278 79.9465) (width 0.25) (layer F.Cu) (net 17))
-  (segment (start 153.543 82.423) (end 192.278 82.423) (width 0.25) (layer F.Cu) (net 17))
-  (segment (start 153.4795 63.9445) (end 153.4795 82.3595) (width 0.25) (layer F.Cu) (net 17))
   (segment (start 153.4795 82.3595) (end 153.543 82.423) (width 0.25) (layer F.Cu) (net 17))
-  (via (at 140.843 68.834) (size 0.8) (drill 0.4) (layers F.Cu B.Cu) (net 18))
-  (segment (start 140.843 63.881) (end 140.843 68.834) (width 0.25) (layer F.Cu) (net 18))
   (via (at 140.843 73.533) (size 0.8) (drill 0.4) (layers F.Cu B.Cu) (net 18))
-  (segment (start 140.843 68.834) (end 140.843 73.533) (width 0.25) (layer B.Cu) (net 18))
   (segment (start 140.843 73.533) (end 149.9235 73.533) (width 0.25) (layer F.Cu) (net 18))
   (segment (start 149.9235 73.533) (end 149.9235 83.3755) (width 0.25) (layer F.Cu) (net 18))
   (segment (start 149.9235 83.3755) (end 194.818 83.3755) (width 0.25) (layer F.Cu) (net 18))
   (segment (start 194.818 83.3755) (end 194.818 79.9465) (width 0.25) (layer F.Cu) (net 18))
-  (segment (start 128.2065 64.0715) (end 128.2065 65.14913) (width 0.25) (layer F.Cu) (net 19))
-  (segment (start 128.2065 65.14913) (end 128.2065 68.3895) (width 0.25) (layer F.Cu) (net 19))
-  (via (at 128.2065 68.961) (size 0.8) (drill 0.4) (layers F.Cu B.Cu) (net 19))
-  (segment (start 128.2065 68.3895) (end 128.2065 68.961) (width 0.25) (layer F.Cu) (net 19))
-  (segment (start 128.2065 68.961) (end 128.2065 71.5645) (width 0.25) (layer B.Cu) (net 19))
-  (segment (start 148.463 84.201) (end 148.5265 84.2645) (width 0.25) (layer F.Cu) (net 19))
-  (segment (start 148.463 84.201) (end 197.358 84.201) (width 0.25) (layer F.Cu) (net 19))
+  (segment (start 128.2065 64.0715) (end 128.2065 65.14913) (width 0.25) (layer F.Cu) (net 17))
+  (via (at 154.8765 66.9925) (size 0.8) (drill 0.4) (layers F.Cu B.Cu) (net 17))
+  (segment (start 154.8765 82.423) (end 154.8765 66.9925) (width 0.25) (layer F.Cu) (net 17))
+  (segment (start 154.8765 82.423) (end 192.278 82.423) (width 0.25) (layer F.Cu) (net 17))
+  (segment (start 153.543 82.423) (end 154.8765 82.423) (width 0.25) (layer F.Cu) (net 17))
+  (via (at 134.493 67.019) (size 0.8) (drill 0.4) (layers F.Cu B.Cu) (net 17))
+  (segment (start 151.287502 67.019) (end 134.493 67.019) (width 0.25) (layer B.Cu) (net 17))
+  (segment (start 154.8765 66.9925) (end 151.314002 66.9925) (width 0.25) (layer B.Cu) (net 17))
+  (segment (start 151.314002 66.9925) (end 151.287502 67.019) (width 0.25) (layer B.Cu) (net 17))
+  (segment (start 133.927315 67.019) (end 133.900815 66.9925) (width 0.25) (layer F.Cu) (net 17))
+  (segment (start 134.493 67.019) (end 133.927315 67.019) (width 0.25) (layer F.Cu) (net 17))
+  (segment (start 133.900815 66.9925) (end 128.2065 66.9925) (width 0.25) (layer F.Cu) (net 17))
+  (segment (start 128.2065 66.9925) (end 128.2065 65.14913) (width 0.25) (layer F.Cu) (net 17))
+  (via (at 140.843 68.8975) (size 0.8) (drill 0.4) (layers F.Cu B.Cu) (net 18))
+  (segment (start 140.843 63.881) (end 140.843 68.8975) (width 0.25) (layer F.Cu) (net 18))
+  (segment (start 140.843 69.463185) (end 140.843 73.533) (width 0.25) (layer B.Cu) (net 18))
+  (segment (start 140.843 68.8975) (end 140.843 69.463185) (width 0.25) (layer B.Cu) (net 18))
   (segment (start 197.358 84.201) (end 197.358 79.9465) (width 0.25) (layer F.Cu) (net 19))
-  (via (at 128.2065 74.93) (size 0.8) (drill 0.4) (layers F.Cu B.Cu) (net 19))
-  (segment (start 128.2065 71.5645) (end 128.2065 74.93) (width 0.25) (layer B.Cu) (net 19))
-  (segment (start 148.3995 74.93) (end 148.463 74.9935) (width 0.25) (layer F.Cu) (net 19))
-  (segment (start 128.2065 74.93) (end 148.3995 74.93) (width 0.25) (layer F.Cu) (net 19))
-  (segment (start 148.463 74.9935) (end 148.463 84.201) (width 0.25) (layer F.Cu) (net 19))
+  (segment (start 153.416 63.9445) (end 153.416 75.057) (width 0.25) (layer F.Cu) (net 19))
+  (via (at 153.4795 80.899) (size 0.8) (drill 0.4) (layers F.Cu B.Cu) (net 19))
+  (segment (start 153.416 75.057) (end 153.416 80.8355) (width 0.25) (layer F.Cu) (net 19))
+  (segment (start 153.416 80.8355) (end 153.4795 80.899) (width 0.25) (layer F.Cu) (net 19))
+  (via (at 153.4795 84.201) (size 0.8) (drill 0.4) (layers F.Cu B.Cu) (net 19))
+  (segment (start 153.4795 80.899) (end 153.4795 84.201) (width 0.25) (layer B.Cu) (net 19))
+  (segment (start 153.4795 84.201) (end 197.358 84.201) (width 0.25) (layer F.Cu) (net 19))
   (via (at 176.8475 75.057) (size 0.8) (drill 0.4) (layers F.Cu B.Cu) (net 20))
   (segment (start 175.26 75.057) (end 176.8475 75.057) (width 0.25) (layer F.Cu) (net 20))

Commit message: finished board design
Parts:
- added D1: LED, LED_SMD:LED_0603_1608Metric_Pad1.05x0.95mm_HandSolder, F.Cu at (140.0, 55.3)
- added D10: LED, LED_SMD:LED_0603_1608Metric_Pad1.05x0.95mm_HandSolder, F.Cu at (175.7, 55.0)
- added D3: LED, LED_SMD:LED_0603_1608Metric_Pad1.05x0.95mm_HandSolder, F.Cu at (152.1, 55.0)
- added D4: LED, LED_SMD:LED_0603_1608Metric_Pad1.05x0.95mm_HandSolder, F.Cu at (225.3, 55.0)
- added D5: LED, LED_SMD:LED_0603_1608Metric_Pad1.05x0.95mm_HandSolder, F.Cu at (239.8, 55.0)
- added D6: LED, LED_SMD:LED_0603_1608Metric_Pad1.05x0.95mm_HandSolder, F.Cu at (206.8, 55.0)
- added D7: LED, LED_SMD:LED_0603_1608Metric_Pad1.05x0.95mm_HandSolder, F.Cu at (221.0, 55.0)
- added D8: LED, LED_SMD:LED_0603_1608Metric_Pad1.05x0.95mm_HandSolder, F.Cu at (203.8, 55.0)
- added D9: LED, LED_SMD:LED_0603_1608Metric_Pad1.05x0.95mm_HandSolder, F.Cu at (190.0, 55.0)
- added R1: 1.5k, Resistor_SMD:R_0603_1608Metric_Pad1.05x0.95mm_HandSolder, F.Cu at (140.0, 58.8)
- added R10: 500, Resistor_SMD:R_0603_1608Metric_Pad1.05x0.95mm_HandSolder, F.Cu at (175.7, 58.7)
- added R3: 1.5k, Resistor_SMD:R_0603_1608Metric_Pad1.05x0.95mm_HandSolder, F.Cu at (152.1, 58.7)
- added R4: 500, Resistor_SMD:R_0603_1608Metric_Pad1.05x0.95mm_HandSolder, F.Cu at (225.3, 58.8)
- added R5: 500, Resistor_SMD:R_0603_1608Metric_Pad1.05x0.95mm_HandSolder, F.Cu at (239.8, 58.8)
- added R6: 500, Resistor_SMD:R_0603_1608Metric_Pad1.05x0.95mm_HandSolder, F.Cu at (206.8, 58.7)
- added R7: 500, Resistor_SMD:R_0603_1608Metric_Pad1.05x0.95mm_HandSolder, F.Cu at (221.0, 58.7)
- added R8: 500, Resistor_SMD:R_0603_1608Metric_Pad1.05x0.95mm_HandSolder, F.Cu at (203.8, 58.8)
- added R9: 500, Resistor_SMD:R_0603_1608Metric_Pad1.05x0.95mm_HandSolder, F.Cu at (190.0, 58.8)
- moved Conn13 92.1 mm to (122.3, 62.7)
- moved Conn7 71.0 mm to (196.7, 63.0)
- moved Conn5 50.4 mm to (134.1, 63.0)
- moved U3 45.6 mm to (181.9, 98.6)
- moved Conn8 44.6 mm to (182.9, 63.0)
- moved Conn6 44.0 mm to (158.1, 63.0)
- moved C3 43.5 mm to (179.6, 95.1)
- moved C4 34.6 mm to (225.4, 65.8), turned to 180 degrees
- moved C5 32.5 mm to (222.2, 69.5)
- moved C2 31.6 mm to (220.7, 69.5)
- moved Conn4 28.8 mm to (145.9, 63.0)
- moved Q2 28.4 mm to (151.6, 76.2), turned to 180 degrees
- moved Q1 26.8 mm to (147.6, 76.2), turned to 180 degrees
- moved Conn3 24.8 mm to (213.9, 63.0)
- moved U2 21.5 mm to (222.6, 75.9), turned to 270 degrees
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Routing:
- net GND: track 400.1 -> 5.32 mm, vias 11 -> 2
- net /+12V_log: track 101.6 -> 48.1 mm, vias 2 -> 0
- net RX_2_SL: track 70.4 -> 17.8 mm, vias 2 -> 0
- net TX_2_SL: track 75.5 -> 26.1 mm, vias 4 -> 0
- net Servo2_PWM: track 76.9 -> 40.7 mm, vias 2 -> 0
- net Servo1_PWM: track 86.3 -> 51.3 mm, vias 2 -> 0
- net Net-(C1-Pad1): track 22.6 -> 2.88 mm, vias 2 -> 0
- net Servo3_PWM: track 68.4 -> 49.4 mm, vias 2 -> 0
- net Net-(U1-PadRese): track 82.5 -> 66.3 mm, vias 3 -> 0
- net Net-(C2-Pad1): track 16.0 -> 2.85 mm
- net Net-(Conn6-Pad1): track 33.0 -> 20.1 mm, vias 2 -> 0
- net RX_1_SL: track 44.8 -> 32.6 mm, vias 4 -> 0
- net TX_1_SL: track 40.8 -> 29.3 mm, vias 4 -> 0
- net +12V_Act: track 87.7 -> 76.7 mm
- net RX_1_IC: track 63.5 -> 73.6 mm, vias 5 -> 0
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- added copper zone on B.Cu, net GND
- added copper zone on F.Cu, net GND
