File: ArmMotorController_Hardware/ArmBoardMC_2019_Rev1.sch (KiCad schematic (older format))
At the start: 72 parts, among them U1 VNH5019A_E, U10 Limit_Switch7, U11 Limit_Switch2, U12 Limit_Switch4, U13 Limit_Switch6, U14 Limit_Switch8, U15 MAX_3232, U16 OKI, U17 Encoder_1, U18 Encoder_3, U19 Encoder_2, U2 VNH5019A_E, U20 Encoder_4, U3 TM4C129E_Launchpad, U5 VNH5019A_E, U6 VNH5019A_E, U7 Limit_Switch1, U8 Limit_Switch3, U9 Limit_Switch5

Commit message: Began properly orginizing schematic
Parts:
- removed D1, D? (x3): LED, Diode_SMD:D_1206_3216Metric, symbol Device:LED
- removed R22: 330, Resistor_SMD:R_0603_1608Metric_Pad1.05x0.95mm_HandSolder, symbol Device:R
- removed R? (x3): 330, 1.5k, symbol Device:R_Small
Connections:
- net labels removed: V+Log
- wire segments 327 -> 314

Commit message: Added AP1509 3.3v
Parts:
- added C? (x4): 10u, Capacitor_SMD:C_0603_1608Metric_Pad1.05x0.95mm_HandSolder, symbol Device:C
- added Conn? (x4): Anderson-3, MRDT_Connectors:Anderson_3_Horisontal_Side_by_Side, symbol MRDT_Connectors:AndersonPP
- added D? (x2): D_Schottky, symbol Device:D_Schottky
- added L? (x2): 47uH, symbol pspice:INDUCTOR
- added U? (x2): AP1059, symbol MRDT_ICs:AP1059
Connections:
- wire segments 314 -> 362

Commit message: Put components into sections, renamed a few pins, changed library for Encoder and Limit Switch
Parts:
- removed D? (x2): LED, Diode_SMD:D_1206_3216Metric, symbol Device:LED
- removed D? (x2): LED, symbol Device:LED
- removed R15, R16, R17, R18, R19, R20, R21: 10K, Resistor_SMD:R_0603_1608Metric_Pad1.05x0.95mm_HandSolder, symbol Device:R_Small
- removed R? (x2): 330, 1.5k, symbol Device:R_Small
- removed R?: 1.5k, 1.5k, symbol Device:R_Small
- removed R?: 1.5k, symbol Device:R_Small
- removed U10: Limit_Switch7, MRDT_Connectors:MOLEX_SL_02_Vertical, symbol MRDT_Switches:Limit_Switch
- removed U11: Limit_Switch2, MRDT_Connectors:MOLEX_SL_02_Vertical, symbol MRDT_Switches:Limit_Switch
- removed U12: Limit_Switch4, MRDT_Connectors:MOLEX_SL_02_Vertical, symbol MRDT_Switches:Limit_Switch
- removed U13: Limit_Switch6, MRDT_Connectors:MOLEX_SL_02_Vertical, symbol MRDT_Switches:Limit_Switch
- removed U14: Limit_Switch8, MRDT_Connectors:MOLEX_SL_02_Vertical, symbol MRDT_Switches:Limit_Switch
- removed U17: Encoder_1, MRDT_Connectors:MOLEX_SL_03_Vertical, symbol MRDT_Sensors:AbsoluteEncoder
- removed U18: Encoder_3, MRDT_Connectors:MOLEX_SL_03_Vertical, symbol MRDT_Sensors:AbsoluteEncoder
- removed U19: Encoder_2, MRDT_Connectors:MOLEX_SL_03_Vertical, symbol MRDT_Sensors:AbsoluteEncoder
- removed U20: Encoder_4, MRDT_Connectors:MOLEX_SL_03_Vertical, symbol MRDT_Sensors:AbsoluteEncoder
- removed U7: Limit_Switch1, MRDT_Connectors:MOLEX_SL_02_Vertical, symbol MRDT_Switches:Limit_Switch
- removed U8: Limit_Switch3, MRDT_Connectors:MOLEX_SL_02_Vertical, symbol MRDT_Switches:Limit_Switch
- removed U9: Limit_Switch5, MRDT_Connectors:MOLEX_SL_02_Vertical, symbol MRDT_Switches:Limit_Switch
- added Conn?: Encoder_3, symbol MRDT_Connectors:Picoblade_3
- added Conn?: Encoder_4, symbol MRDT_Connectors:Picoblade_3
- added Conn?: Encoder_2, symbol MRDT_Connectors:Picoblade_3
- added Conn?: Encoder_1, symbol MRDT_Connectors:Picoblade_3
- added Conn?: Limit_Switch_1, symbol MRDT_Connectors:Molex_SL_02
- added Conn?: Limit_Switch_2, symbol MRDT_Connectors:Molex_SL_02
- added Conn?: Limit_Switch_3, symbol MRDT_Connectors:Molex_SL_02
- added Conn?: Limit_Switch_4, symbol MRDT_Connectors:Molex_SL_02
- added Conn?: Limit_Switch_5, symbol MRDT_Connectors:Molex_SL_02
- added Conn?: Limit_Switch_6, symbol MRDT_Connectors:Molex_SL_02
- added Conn?: Limit_Switch_7, symbol MRDT_Connectors:Molex_SL_02
- added Conn?: Limit_Switch_8, symbol MRDT_Connectors:Molex_SL_02
- added R? (x7): 10K, Resistor_SMD:R_0603_1608Metric_Pad1.05x0.95mm_HandSolder, symbol Device:R_Small
Connections:
- net labels added: +5V, ENC1, ENC2, ENC3, ENC4
- net labels removed: Encoder1_PWM, Encoder2_PWM, Encoder3_PWM, Encoder4_PWM, Logic_3.3V, Out_A1, Out_A2, Out_A3, Out_A4, Out_B1, Out_B2, Out_B3, Out_B4
- wire segments 362 -> 356
Other:
- note added: "Out_A1\n\n"
- note added: "Out_A2\n\n\n"
- note added: "Out_A3\n"
- note added: "Out_A4\n\n\n\n"
- note added: "Out_B1\n\n"
- note added: "Out_B2\n\n\n"
- note added: "Out_B3\n"
- note added: "Out_B4\n\n\n\n"
- note removed: "Orange"
- note removed: "Orange\n"
