File: ArmBoard_Hardware/ArmBoard_Hardware.sch (KiCad schematic (older format))
At the start: 116 parts, among them Q1 Q_NMOS_GSD, Q2 Q_NMOS_GSD, U1 TM4C129E_Launchpad, U2 MAX_3232, U3 OKI, U4 OKI, U5 VNH5019A_E, U6 MAX_3232

Commit message: If anyone touches this I will kill them, and then myself
Parts:
- C11, C14: value 47u -> 47uF
- C12, C13, C5, C6, C7, C8: value 10u -> 10uF
- C15, C16, C19, C2, C20, C21, C22, C3, C4: value .1u -> .1uF
Changed lines of the file:
@@
 P 3400 1200
 F 0 "C2" H 3400 1100 50  0000 L CNN
-F 1 ".1u" H 3250 1300 50  0000 L CNN
+F 1 ".1uF" H 3200 1300 50  0000 L CNN
 F 2 "Capacitor_SMD:C_0603_1608Metric_Pad1.05x0.95mm_HandSolder" H 3438 1050 50  0001 C CNN
 F 3 "~" H 3400 1200 50  0001 C CNN
@@
 $EndComp
 $Comp
-L Device:C C7
-U 1 1 5BCA6E9A
-P 3600 1200
-F 0 "C7" H 3600 1100 50  0000 L CNN
-F 1 "10u" H 3450 1300 50  0000 L CNN
-F 2 "Capacitor_SMD:C_0603_1608Metric_Pad1.05x0.95mm_HandSolder" H 3638 1050 50  0001 C CNN
-F 3 "~" H 3600 1200 50  0001 C CNN
-	1    3600 1200
-	1    0    0    -1
-$EndComp
-$Comp
 L Device:C C8
 U 1 1 5BCA6EB8
 P 3800 1200
 F 0 "C8" H 3800 1100 50  0000 L CNN
-F 1 "10u" H 3650 1300 50  0000 L CNN
+F 1 "10uF" H 3600 1300 50  0000 L CNN
 F 2 "Capacitor_SMD:C_0603_1608Metric_Pad1.05x0.95mm_HandSolder" H 3838 1050 50  0001 C CNN
 F 3 "~" H 3800 1200 50  0001 C CNN
@@
 P 4000 1200
 F 0 "C9" H 4000 1100 50  0000 L CNN
-F 1 "10u" H 3850 1300 50  0000 L CNN
+F 1 "10u" H 3800 1300 50  0000 L CNN
 F 2 "Capacitor_SMD:C_0603_1608Metric_Pad1.05x0.95mm_HandSolder" H 4038 1050 50  0001 C CNN
 F 3 "~" H 4000 1200 50  0001 C CNN
@@
 P 3500 1800
 F 0 "C5" H 3450 1900 50  0000 C CNN
-F 1 "10u" H 3600 1700 50  0000 C CNN
+F 1 "10uF" H 3650 1700 50  0000 C CNN
 F 2 "Capacitor_SMD:C_0603_1608Metric_Pad1.05x0.95mm_HandSolder" H 3538 1650 50  0001 C CNN
 F 3 "~" H 3500 1800 50  0001 C CNN
@@
 U 1 1 5CF9D7A2
 P 4550 1800
-F 0 "C12" H 4500 1900 50  0000 C CNN
-F 1 "10u" H 4650 1700 50  0000 C CNN
+F 0 "C12" H 4450 1900 50  0000 C CNN
+F 1 "10uF" H 4700 1700 50  0000 C CNN
 F 2 "Capacitor_SMD:C_0603_1608Metric_Pad1.05x0.95mm_HandSolder" H 4588 1650 50  0001 C CNN
 F 3 "~" H 4550 1800 50  0001 C CNN
@@
 P 3500 2500
 F 0 "C6" H 3450 2600 50  0000 C CNN
-F 1 "10u" H 3600 2400 50  0000 C CNN
+F 1 "10uF" H 3650 2400 50  0000 C CNN
 F 2 "Capacitor_SMD:C_0603_1608Metric_Pad1.05x0.95mm_HandSolder" H 3538 2350 50  0001 C CNN
 F 3 "~" H 3500 2500 50  0001 C CNN
@@
 U 1 1 5D1DB1A8
 P 4550 2500
-F 0 "C13" H 4500 2600 50  0000 C CNN
-F 1 "10u" H 4650 2400 50  0000 C CNN
+F 0 "C13" H 4450 2600 50  0000 C CNN
+F 1 "10uF" H 4700 2400 50  0000 C CNN
 F 2 "Capacitor_SMD:C_0603_1608Metric_Pad1.05x0.95mm_HandSolder" H 4588 2350 50  0001 C CNN
 F 3 "~" H 4550 2500 50  0001 C CNN
@@
 P 4200 1200
 F 0 "C10" H 4200 1100 50  0000 L CNN
-F 1 "10u" H 4050 1300 50  0000 L CNN
+F 1 "10u" H 4000 1300 50  0000 L CNN
 F 2 "Capacitor_SMD:C_0603_1608Metric_Pad1.05x0.95mm_HandSolder" H 4238 1050 50  0001 C CNN
 F 3 "~" H 4200 1200 50  0001 C CNN
@@
 P 4400 1200
 F 0 "C11" H 4400 1100 50  0000 L CNN
-F 1 "47u" H 4400 1300 50  0000 L CNN
+F 1 "47uF" H 4200 1300 50  0000 L CNN
 F 2 "Capacitor_THT:CP_Radial_D5.0mm_P2.50mm" H 4400 1200 50  0001 C CNN
 F 3 "~" H 4400 1200 50  0001 C CNN
@@
 P 4600 1200
 F 0 "C14" H 4600 1100 50  0000 L CNN
-F 1 "47u" H 4600 1300 50  0000 L CNN
+F 1 "47uF" H 4400 1300 50  0000 L CNN
 F 2 "Capacitor_THT:CP_Radial_D5.0mm_P2.50mm" H 4600 1200 50  0001 C CNN
 F 3 "~" H 4600 1200 50  0001 C CNN
@@
 P 13100 4150
 F 0 "C15" H 13250 4100 50  0000 R TNN
-F 1 ".1u" H 13100 4250 50  0000 L CNN
+F 1 ".1uF" H 13100 4250 50  0000 L CNN
 F 2 "Capacitor_SMD:C_0603_1608Metric_Pad1.05x0.95mm_HandSolder" H 13100 4150 50  0001 C CNN
 F 3 "~" H 13100 4150 50  0001 C CNN
@@
 P 13100 4450
 F 0 "C16" H 13250 4400 50  0000 R TNN
-F 1 ".1u" H 13100 4550 50  0000 L CNN
+F 1 ".1uF" H 13100 4550 50  0000 L CNN
 F 2 "Capacitor_SMD:C_0603_1608Metric_Pad1.05x0.95mm_HandSolder" H 13100 4450 50  0001 C CNN
 F 3 "~" H 13100 4450 50  0001 C CNN
@@
 P 11800 4450
 F 0 "C3" V 11750 4550 50  0000 C CNN
-F 1 ".1u" V 11750 4350 50  0000 C CNN
+F 1 ".1uF" V 11750 4350 50  0000 C CNN
 F 2 "Capacitor_SMD:C_0603_1608Metric_Pad1.05x0.95mm_HandSolder" H 11800 4450 50  0001 C CNN
 F 3 "~" H 11800 4450 50  0001 C CNN
@@
 P 11800 4550
 F 0 "C4" V 11850 4575 50  0000 L CNN
-F 1 ".1u" V 11850 4400 50  0000 L CNN
+F 1 ".1uF" V 11850 4350 50  0000 L CNN
 F 2 "Capacitor_SMD:C_0603_1608Metric_Pad1.05x0.95mm_HandSolder" H 11800 4550 50  0001 C CNN
 F 3 "~" H 11800 4550 50  0001 C CNN
@@
 P 13050 5550
 F 0 "C21" H 13200 5500 50  0000 R TNN
-F 1 ".1u" H 13050 5650 50  0000 L CNN
+F 1 ".1uF" H 13050 5650 50  0000 L CNN
 F 2 "Capacitor_SMD:C_0603_1608Metric_Pad1.05x0.95mm_HandSolder" H 13050 5550 50  0001 C CNN
 F 3 "~" H 13050 5550 50  0001 C CNN
@@
 P 13050 5850
 F 0 "C22" H 13200 5800 50  0000 R TNN
-F 1 ".1u" H 13050 5950 50  0000 L CNN
+F 1 ".1uF" H 13050 5950 50  0000 L CNN
 F 2 "Capacitor_SMD:C_0603_1608Metric_Pad1.05x0.95mm_HandSolder" H 13050 5850 50  0001 C CNN
 F 3 "~" H 13050 5850 50  0001 C CNN
@@
 P 11750 5850
 F 0 "C19" V 11700 5950 50  0000 C CNN
-F 1 ".1u" V 11700 5750 50  0000 C CNN
+F 1 ".1uF" V 11700 5700 50  0000 C CNN
 F 2 "Capacitor_SMD:C_0603_1608Metric_Pad1.05x0.95mm_HandSolder" H 11750 5850 50  0001 C CNN
 F 3 "~" H 11750 5850 50  0001 C CNN
@@
 P 11750 5950
 F 0 "C20" V 11800 5975 50  0000 L CNN
-F 1 ".1u" V 11800 5800 50  0000 L CNN
+F 1 ".1uF" V 11800 5750 50  0000 L CNN
 F 2 "Capacitor_SMD:C_0603_1608Metric_Pad1.05x0.95mm_HandSolder" H 11750 5950 50  0001 C CNN
 F 3 "~" H 11750 5950 50  0001 C CNN
@@
 Text GLabel 8050 7000 1    50   Input ~ 0
 LS_1
+$Comp
+L Device:C C7
+U 1 1 5BCA6E9A
+P 3600 1200
+F 0 "C7" H 3600 1100 50  0000 L CNN
+F 1 "10uF" H 3400 1300 50  0000 L CNN
+F 2 "Capacitor_SMD:C_0603_1608Metric_Pad1.05x0.95mm_HandSolder" H 3638 1050 50  0001 C CNN
+F 3 "~" H 3600 1200 50  0001 C CNN
+	1    3600 1200
+	1    0    0    -1
+$EndComp
 $EndSCHEMATC

Commit message: Hurt me daddy
Parts:
- removed C1, C18: 10uF, Capacitor_SMD:C_0603_1608Metric_Pad1.05x0.95mm_HandSolder, symbol Device:C_Small
- removed C13, C6: 10uF, Capacitor_SMD:C_0603_1608Metric_Pad1.05x0.95mm_HandSolder, symbol Device:C
- removed C15, C16, C19, C20, C21, C22, C3, C4: .1uF, Capacitor_SMD:C_0603_1608Metric_Pad1.05x0.95mm_HandSolder, symbol Device:C_Small
- removed U2, U6: MAX_3232, MRDT_ICs:SOIC_16_3.9x9.9mm_Pitch1.27mm, symbol MRDT_ICs:MAX_3232
- removed U4: OKI, MRDT_Devices:OKI_Horizontal, symbol MRDT_Devices:OKI
- added D9: LED, LED_SMD:LED_0603_1608Metric_Pad1.05x0.95mm_HandSolder, symbol Device:LED
- added R16: 1.5k, Resistor_SMD:R_0603_1608Metric_Pad1.05x0.95mm_HandSolder, symbol Device:R
Connections:
- net RX_1_SL is gone; now on net RX_1_Tiva: Conn23.1
- net RX_2_SL is gone; now on net RX_2_Tiva: Conn7.1
- net RX_3_SL is gone; now on net RX_3_Tiva: Conn6.1
- net TX_1_SL is gone; now on net TX_1_Tiva: Conn23.3
- net TX_2_SL is gone; now on net TX_2_Tiva: Conn7.3
- net TX_3_SL is gone; now on net TX_3_Tiva: Conn6.3
- net +12VA: now also R16.1
- net at Conn19.2, Q1.3 (D): now also D9.1 (K)
- new net: D9.2 (A), R16.2
- no-connect marks 54 -> 50
Other:
- note added: "Purple"
- note added: "Rx5"
- note added: "Rx7"
- note added: "Tx3"
- note added: "Tx5"
- note added: "Tx7"
- note removed: "Level Shifter"
- note removed: "Yellow"
- moved on the sheet: C10, C11, C12, C14, C2, C5, C7, C8, C9, Conn10, Conn11, Conn12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

Commit message: Suck my toes
Other:
- moved on the sheet: C12, C5
Changed lines of the file:
@@
 $EndComp
 Wire Wire Line
-	3450 2150 4000 2150
+	3450 2500 4000 2500
 $Comp
 L Device:C C5
 U 1 1 5CCD2350
-P 3450 1950
-F 0 "C5" H 3400 2050 50  0000 C CNN
-F 1 "10uF" H 3600 1850 50  0000 C CNN
-F 2 "Capacitor_SMD:C_0603_1608Metric_Pad1.05x0.95mm_HandSolder" H 3488 1800 50  0001 C CNN
-F 3 "~" H 3450 1950 50  0001 C CNN
-	1    3450 1950
+P 3450 2300
+F 0 "C5" H 3400 2400 50  0000 C CNN
+F 1 "10uF" H 3600 2200 50  0000 C CNN
+F 2 "Capacitor_SMD:C_0603_1608Metric_Pad1.05x0.95mm_HandSolder" H 3488 2150 50  0001 C CNN
+F 3 "~" H 3450 2300 50  0001 C CNN
+	1    3450 2300
 	-1   0    0    1
 $EndComp
@@
 L MRDT_Devices:OKI U3
 U 1 1 5C208612
-P 3800 1850
-F 0 "U3" H 3850 1800 60  0001 C CNN
-F 1 "OKI" H 4000 2131 60  0000 C CNN
-F 2 "MRDT_Devices:OKI_Horizontal" H 3600 1750 60  0001 C CNN
-F 3 "" H 3600 1750 60  0001 C CNN
-	1    3800 1850
-	1    0    0    -1
-$EndComp
-Wire Wire Line
-	4500 1750 4500 1700
+P 3800 2200
+F 0 "U3" H 3850 2150 60  0001 C CNN
+F 1 "OKI" H 4000 2481 60  0000 C CNN
+F 2 "MRDT_Devices:OKI_Horizontal" H 3600 2100 60  0001 C CNN
+F 3 "" H 3600 2100 60  0001 C CNN
+	1    3800 2200
+	1    0    0    -1
+$EndComp
+Wire Wire Line
+	4500 2100 4500 2050
 $Comp
 L power:+12L #PWR019
 U 1 1 5EDFDEDB
-P 3450 1650
-F 0 "#PWR019" H 3450 1500 50  0001 C CNN
-F 1 "+12L" H 3465 1823 50  0000 C CNN
-F 2 "" H 3450 1650 50  0001 C CNN
-F 3 "" H 3450 1650 50  0001 C CNN
-	1    3450 1650
+P 3450 2000
+F 0 "#PWR019" H 3450 1850 50  0001 C CNN
+F 1 "+12L" H 3465 2173 50  0000 C CNN
+F 2 "" H 3450 2000 50  0001 C CNN
+F 3 "" H 3450 2000 50  0001 C CNN
+	1    3450 2000
 	1    0    0    -1
 $EndComp
@@
 L power:GND #PWR029
 U 1 1 5D05E895
-P 4650 2200
-F 0 "#PWR029" H 4650 1950 50  0001 C CNN
-F 1 "GND" H 4650 2050 50  0000 C CNN
-F 2 "" H 4650 2200 50  0001 C CNN
-F 3 "" H 4650 2200 50  0001 C CNN
-	1    4650 2200
+P 4650 2550
+F 0 "#PWR029" H 4650 2300 50  0001 C CNN
+F 1 "GND" H 4650 2400 50  0000 C CNN
+F 2 "" H 4650 2550 50  0001 C CNN
+F 3 "" H 4650 2550 50  0001 C CNN
+	1    4650 2550
 	1    0    0    -1
 $EndComp
@@
 L power:+3.3V #PWR028
 U 1 1 5CFFE006
-P 4500 1700
-F 0 "#PWR028" H 4500 1550 50  0001 C CNN
-F 1 "+3.3V" H 4400 1850 50  0000 L CNN
-F 2 "" H 4500 1700 50  0001 C CNN
-F 3 "" H 4500 1700 50  0001 C CNN
-	1    4500 1700
+P 4500 2050
+F 0 "#PWR028" H 4500 1900 50  0001 C CNN
+F 1 "+3.3V" H 4400 2200 50  0000 L CNN
+F 2 "" H 4500 2050 50  0001 C CNN
+F 3 "" H 4500 2050 50  0001 C CNN
+	1    4500 2050
 	1    0    0    -1
 $EndComp
@@
 L Device:C C12
 U 1 1 5CF9D7A2
-P 4500 1950
-F 0 "C12" H 4400 2050 50  0000 C CNN
-F 1 "10uF" H 4650 1850 50  0000 C CNN
-F 2 "Capacitor_SMD:C_0603_1608Metric_Pad1.05x0.95mm_HandSolder" H 4538 1800 50  0001 C CNN
-F 3 "~" H 4500 1950 50  0001 C CNN
-	1    4500 1950
+P 4500 2300
+F 0 "C12" H 4400 2400 50  0000 C CNN
+F 1 "10uF" H 4650 2200 50  0000 C CNN
+F 2 "Capacitor_SMD:C_0603_1608Metric_Pad1.05x0.95mm_HandSolder" H 4538 2150 50  0001 C CNN
+F 3 "~" H 4500 2300 50  0001 C CNN
+	1    4500 2300
 	-1   0    0    1
 $EndComp
@@
 	4700 1400 4500 1400
 Wire Wire Line
-	4400 1750 4500 1750
-Wire Wire Line
-	3450 1650 3450 1750
-Wire Wire Line
-	3450 1750 3600 1750
-Wire Wire Line
-	4500 1800 4500 1750
-Connection ~ 4500 1750
-Wire Wire Line
-	3450 1800 3450 1750
-Connection ~ 3450 1750
-Wire Wire Line
-	3450 2100 3450 2150
-Wire Wire Line
-	4500 2100 4500 2150
-Wire Wire Line
-	4000 2050 4000 2150
-Connection ~ 4000 2150
-Wire Wire Line
-	4000 2150 4500 2150
+	4400 2100 4500 2100
+Wire Wire Line
+	3450 2000 3450 2100
+Wire Wire Line
+	3450 2100 3600 2100
+Wire Wire Line
+	4500 2150 4500 2100
+Connection ~ 4500 2100
+Wire Wire Line
+	3450 2150 3450 2100
+Connection ~ 3450 2100
+Wire Wire Line
+	3450 2450 3450 2500
+Wire Wire Line
+	4500 2450 4500 2500
+Wire Wire Line
+	4000 2400 4000 2500
+Connection ~ 4000 2500
+Wire Wire Line
+	4000 2500 4500 2500
 Wire Notes Line
 	5250 3200 5250 400
@@
 TIVA
 Wire Wire Line
-	4500 2150 4650 2150
-Wire Wire Line
-	4650 2150 4650 2200
-Connection ~ 4500 2150
+	4500 2500 4650 2500
+Wire Wire Line
+	4650 2500 4650 2550
+Connection ~ 4500 2500
 Wire Wire Line
 	2200 1450 2750 1450

Commit message: 3 up, three down, suck my toes
Parts:
- removed D7: LED, LED_SMD:LED_0603_1608Metric_Pad1.05x0.95mm_HandSolder, symbol Device:LED
- removed R14: 500, Resistor_SMD:R_0603_1608Metric_Pad1.05x0.95mm_HandSolder, symbol Device:R_Small
Connections:
- net ENC_1_PWM: now also U1.PD4 (A2_5); no longer U1.PB4 (B2_3)
- net ENC_2_PWM: now also U1.PM7 (D2_2); no longer U1.PK3 (B2_8)
- net ENC_3_PWM: now also U1.PM2 (C2_6); no longer U1.PB5 (B2_4)
- net ENC_4_PWM: now also U1.PM0 (C2_4); no longer U1.PK2 (B2_7)
- net ENC_5_PWM: now also U1.PA7 (D2_4); no longer U1.PK0 (B2_5)
- net ENC_6_PWM: now also U1.PM1 (C2_5); no longer U1.PK1 (B2_6)
Other:
- moved on the sheet: D3, D5, R10, R12
Changed lines of the file:
@@
 L Device:R_Small R10
 U 1 1 5D1DFACC
-P 9800 4450
-F 0 "R10" V 9850 4450 50  0000 C TNN
-F 1 "1000" V 9800 4450 50  0000 C CNN
-F 2 "Resistor_SMD:R_0603_1608Metric_Pad1.05x0.95mm_HandSolder" H 9800 4450 50  0001 C CNN
-F 3 "~" H 9800 4450 50  0001 C CNN
-	1    9800 4450
+P 9900 4450
+F 0 "R10" V 9950 4450 50  0000 C TNN
+F 1 "1000" V 9900 4450 50  0000 C CNN
+F 2 "Resistor_SMD:R_0603_1608Metric_Pad1.05x0.95mm_HandSolder" H 9900 4450 50  0001 C CNN
+F 3 "~" H 9900 4450 50  0001 C CNN
+	1    9900 4450
 	-1   0    0    1
 $EndComp
@@
 L Device:LED D3
 U 1 1 5D1DFAD3
-P 9800 4750
-F 0 "D3" H 9850 4650 50  0000 R CNN
-F 1 "LED" V 9900 4900 50  0000 R CNN
-F 2 "LED_SMD:LED_0603_1608Metric_Pad1.05x0.95mm_HandSolder" H 9800 4750 50  0001 C CNN
-F 3 "~" H 9800 4750 50  0001 C CNN
-	1    9800 4750
+P 9900 4750
+F 0 "D3" H 9950 4650 50  0000 R CNN
+F 1 "LED" V 10000 4900 50  0000 R CNN
+F 2 "LED_SMD:LED_0603_1608Metric_Pad1.05x0.95mm_HandSolder" H 9900 4750 50  0001 C CNN
+F 3 "~" H 9900 4750 50  0001 C CNN
+	1    9900 4750
 	0    -1   -1   0
 $EndComp
@@
 L power:GND #PWR046
 U 1 1 5D1DFADA
-P 9800 4950
-F 0 "#PWR046" H 9800 4700 50  0001 C CNN
-F 1 "GND" H 9800 4800 50  0000 C CNN
-F 2 "" H 9800 4950 50  0001 C CNN
-F 3 "" H 9800 4950 50  0001 C CNN
-	1    9800 4950
-	1    0    0    -1
-$EndComp
-Wire Wire Line
-	9800 4550 9800 4600
-Wire Wire Line
-	9800 4900 9800 4950
-Text Notes 9750 4700 3    39   ~ 0
+P 9900 4950
+F 0 "#PWR046" H 9900 4700 50  0001 C CNN
+F 1 "GND" H 9900 4800 50  0000 C CNN
+F 2 "" H 9900 4950 50  0001 C CNN
+F 3 "" H 9900 4950 50  0001 C CNN
+	1    9900 4950
+	1    0    0    -1
+$EndComp
+Wire Wire Line
+	9900 4550 9900 4600
+Wire Wire Line
+	9900 4900 9900 4950
+Text Notes 9850 4700 3    39   ~ 0
 Green\n
 $Comp
 L Device:R_Small R12
 U 1 1 5D243A0D
-P 10100 4450
-F 0 "R12" V 10150 4450 50  0000 C TNN
-F 1 "330" V 10100 4450 50  0000 C CNN
-F 2 "Resistor_SMD:R_0603_1608Metric_Pad1.05x0.95mm_HandSolder" H 10100 4450 50  0001 C CNN
-F 3 "~" H 10100 4450 50  0001 C CNN
-	1    10100 4450
+P 10200 4450
+F 0 "R12" V 10250 4450 50  0000 C TNN
+F 1 "330" V 10200 4450 50  0000 C CNN
+F 2 "Resistor_SMD:R_0603_1608Metric_Pad1.05x0.95mm_HandSolder" H 10200 4450 50  0001 C CNN
+F 3 "~" H 10200 4450 50  0001 C CNN
+	1    10200 4450
 	-1   0    0    1
 $EndComp
@@
 L Device:LED D5
 U 1 1 5D243A14
-P 10100 4750
-F 0 "D5" H 10150 4650 50  0000 R CNN
-F 1 "LED" V 10200 4900 50  0000 R CNN
-F 2 "LED_SMD:LED_0603_1608Metric_Pad1.05x0.95mm_HandSolder" H 10100 4750 50  0001 C CNN
-F 3 "~" H 10100 4750 50  0001 C CNN
-	1    10100 4750
+P 10200 4750
+F 0 "D5" H 10250 4650 50  0000 R CNN
+F 1 "LED" V 10300 4900 50  0000 R CNN
+F 2 "LED_SMD:LED_0603_1608Metric_Pad1.05x0.95mm_HandSolder" H 10200 4750 50  0001 C CNN
+F 3 "~" H 10200 4750 50  0001 C CNN
+	1    10200 4750
 	0    -1   -1   0
 $EndComp
@@
 L power:GND #PWR050
 U 1 1 5D243A1B
-P 10100 4950
-F 0 "#PWR050" H 10100 4700 50  0001 C CNN
-F 1 "GND" H 10100 4800 50  0000 C CNN
-F 2 "" H 10100 4950 50  0001 C CNN
-F 3 "" H 10100 4950 50  0001 C CNN
-	1    10100 4950
-	1    0    0    -1
-$EndComp
-Wire Wire Line
-	10100 4550 10100 4600
-Wire Wire Line
-	10100 4900 10100 4950
-Text Notes 10050 4850 1    39   ~ 0
+P 10200 4950
+F 0 "#PWR050" H 10200 4700 50  0001 C CNN
+F 1 "GND" H 10200 4800 50  0000 C CNN
+F 2 "" H 10200 4950 50  0001 C CNN
+F 3 "" H 10200 4950 50  0001 C CNN
+	1    10200 4950
+	1    0    0    -1
+$EndComp
+Wire Wire Line
+	10200 4550 10200 4600
+Wire Wire Line
+	10200 4900 10200 4950
+Text Notes 10150 4850 1    39   ~ 0
 Green
 Wire Wire Line
-	10100 4300 10100 4350
-Wire Wire Line
-	9800 4300 9800 4350
+	10200 4300 10200 4350
+Wire Wire Line
+	9900 4300 9900 4350
 NoConn ~ 7200 2650
 Wire Wire Line
@@
 L power:+3.3V #PWR049
 U 1 1 5D19AAEB
-P 10100 4300
-F 0 "#PWR049" H 10100 4150 50  0001 C CNN
-F 1 "+3.3V" H 10000 4450 50  0000 L CNN
-F 2 "" H 10100 4300 50  0001 C CNN
-F 3 "" H 10100 4300 50  0001 C CNN
-	1    10100 4300
-	1    0    0    -1
-$EndComp
-$Comp
-L Device:R_Small R14
-U 1 1 5DD5F861
-P 10400 4450
-F 0 "R14" V 10450 4450 50  0000 C TNN
-F 1 "500" V 10400 4450 50  0000 C CNN
-F 2 "Resistor_SMD:R_0603_1608Metric_Pad1.05x0.95mm_HandSolder" H 10400 4450 50  0001 C CNN
-F 3 "~" H 10400 4450 50  0001 C CNN
-	1    10400 4450
-	-1   0    0    1
-$EndComp
-$Comp
-L Device:LED D7
-U 1 1 5DD5F868
-P 10400 4750
-F 0 "D7" H 10450 4650 50  0000 R CNN
-F 1 "LED" V 10500 4900 50  0000 R CNN
-F 2 "LED_SMD:LED_0603_1608Metric_Pad1.05x0.95mm_HandSolder" H 10400 4750 50  0001 C CNN
-F 3 "~" H 10400 4750 50  0001 C CNN
-	1    10400 4750
-	0    -1   -1   0
-$EndComp
-$Comp
-L power:GND #PWR055
-U 1 1 5DD5F86F
-P 10400 4950
-F 0 "#PWR055" H 10400 4700 50  0001 C CNN
-F 1 "GND" H 10400 4800 50  0000 C CNN
-F 2 "" H 10400 4950 50  0001 C CNN
-F 3 "" H 10400 4950 50  0001 C CNN
-	1    10400 4950
-	1    0    0    -1
-$EndComp
-Wire Wire Line
-	10400 4550 10400 4600
-Wire Wire Line
-	10400 4900 10400 4950
-Text Notes 10350 4850 1    39   ~ 0
-Green
-Wire Wire Line
-	10400 4300 10400 4350
-$Comp
-L power:+5V #PWR054
-U 1 1 5DD9DFAA
-P 10400 4300
-F 0 "#PWR054" H 10400 4150 50  0001 C CNN
-F 1 "+5V" H 10400 4450 50  0000 C CNN
-F 2 "" H 10400 4300 50  0001 C CNN
-F 3 "" H 10400 4300 50  0001 C CNN
-	1    10400 4300
+P 10200 4300
+F 0 "#PWR049" H 10200 4150 50  0001 C CNN
+F 1 "+3.3V" H 10100 4450 50  0000 L CNN
+F 2 "" H 10200 4300 50  0001 C CNN
+F 3 "" H 10200 4300 50  0001 C CNN
+	1    10200 4300
 	1    0    0    -1
 $EndComp
@@
 L power:+12VA #PWR0108
 U 1 1 61115BFD
-P 9800 4300
-F 0 "#PWR0108" H 9800 4150 50  0001 C CNN
-F 1 "+12VA" H 9815 4473 50  0000 C CNN
-F 2 "" H 9800 4300 50  0001 C CNN
-F 3 "" H 9800 4300 50  0001 C CNN
-	1    9800 4300
+P 9900 4300
+F 0 "#PWR0108" H 9900 4150 50  0001 C CNN
+F 1 "+12VA" H 9915 4473 50  0000 C CNN
+F 2 "" H 9900 4300 50  0001 C CNN
+F 3 "" H 9900 4300 50  0001 C CNN
+	1    9900 4300
 	1    0    0    -1
 $EndComp
@@
 Text GLabel 4050 5950 2    50   Output ~ 0
 M_PWM
-Text GLabel 4050 4050 2    50   Input ~ 0
+Text GLabel 3050 4250 0    50   Input ~ 0
 ENC_1_PWM
-Text GLabel 4050 4550 2    50   Input ~ 0
+Text GLabel 4050 5150 2    50   Input ~ 0
 ENC_2_PWM
-Text GLabel 4050 4150 2    50   Input ~ 0
+Text GLabel 3050 5550 0    50   Input ~ 0
 ENC_3_PWM
 Text GLabel 4050 5750 2    50   Output ~ 0
@@
 L power:GND #PWR027
 U 1 1 5BFE4810
-P 4100 5100
-F 0 "#PWR027" H 4100 4850 50  0001 C CNN
-F 1 "GND" H 4200 5100 50  0000 C CNN
-F 2 "" H 4100 5100 50  0001 C CNN
-F 3 "" H 4100 5100 50  0001 C CNN
-	1    4100 5100
+P 4150 4950
+F 0 "#PWR027" H 4150 4700 50  0001 C CNN
+F 1 "GND" H 4250 4950 50  0000 C CNN
+F 2 "" H 4150 4950 50  0001 C CNN
+F 3 "" H 4150 4950 50  0001 C CNN
+	1    4150 4950
 	1    0    0    -1
 $EndComp
@@
 	3000 3850 3100 3850
 Wire Wire Line
-	4000 5050 4100 5050
+	4050 4900 4150 4900
 NoConn ~ 3100 3950
 NoConn ~ 4000 3850
 NoConn ~ 4000 5450
-Text GLabel 4050 4250 2    50   Input ~ 0
+Text GLabel 4050 5350 2    50   Input ~ 0
 ENC_5_PWM
-Text GLabel 4050 4350 2    50   Input ~ 0
+Text GLabel 3050 5450 0    50   Input ~ 0
 ENC_6_PWM
 NoConn ~ 4000 5550
 NoConn ~ 3100 5050
-Text GLabel 4050 4450 2    50   Input ~ 0
+Text GLabel 3050 5350 0    50   Input ~ 0
 ENC_4_PWM
 Text GLabel 4050 4650 2    50   Output ~ 0
@@
 TX_2_Tiva
 Wire Wire Line
-	4000 4150 4050 4150
-Wire Wire Line
-	4000 4250 4050 4250
-Wire Wire Line
-	4000 4350 4050 4350
-Wire Wire Line
-	4000 4550 4050 4550
-Wire Wire Line
-	4000 4050 4050 4050
-Wire Wire Line
-	4000 4450 4050 4450
+	4000 5350 4050 5350
+Wire Wire Line
+	3100 5550 3050 5550
+Wire Wire Line
+	3100 5450 3050 5450
+Wire Wire Line
+	4000 5150 4050 5150
+Wire Wire Line
+	3050 4250 3100 4250
+Wire Wire Line
+	3100 5350 3050 5350
 Wire Wire Line
 	4000 5750 4050 5750
@@
 NoConn ~ 3100 4050
 NoConn ~ 3100 4150
-NoConn ~ 3100 4250
-NoConn ~ 3100 5450
-NoConn ~ 3100 5550
 NoConn ~ 3100 5650
 NoConn ~ 3100 5750
@@
 Wire Wire Line
 	4000 4750 4050 4750
-NoConn ~ 4000 5350
-NoConn ~ 3100 5350
-NoConn ~ 4000 5150
 NoConn ~ 4000 5250
 NoConn ~ 3100 5250
@@
 	4050 3850 4150 3850
 Wire Wire Line
-	4100 5100 4100 5050
+	4150 4950 4150 4900
 Wire Wire Line
 	2200 3950 2200 4000
@@
 Wire Wire Line
 	11400 2300 11400 2250
+Wire Wire Line
+	4000 5050 4050 5050
+Wire Wire Line
+	4050 5050 4050 4900
+NoConn ~ 4000 4550
+NoConn ~ 4000 4450
+NoConn ~ 4000 4350
+NoConn ~ 4000 4250
+NoConn ~ 4000 4150
+NoConn ~ 4000 4050
 $EndSCHEMATC

Commit message: This board is a basterdization of what it once was
Connections:
- net ENC_1_PWM: now also U1.PD5 (A2_6); no longer U1.PD4 (A2_5)
- net ENC_2_PWM: now also U1.PD0 (D1_7); no longer U1.PM7 (D2_2)
- net ENC_3_PWM: now also U1.PD4 (A2_5); no longer U1.PM2 (C2_6)
- net ENC_5_PWM: now also U1.PM7 (D2_2); no longer U1.PA7 (D2_4)
- net I_SENSE: now also U1.PD1 (D1_6); no longer U1.PD5 (A2_6)
- no-connect marks 50 -> 61
Changed lines of the file:
@@
 Text GLabel 4050 5950 2    50   Output ~ 0
 M_PWM
+Text GLabel 3050 4350 0    50   Input ~ 0
+ENC_1_PWM
+Text GLabel 2150 5650 2    50   Input ~ 0
+ENC_2_PWM
 Text GLabel 3050 4250 0    50   Input ~ 0
-ENC_1_PWM
-Text GLabel 4050 5150 2    50   Input ~ 0
-ENC_2_PWM
-Text GLabel 3050 5550 0    50   Input ~ 0
 ENC_3_PWM
 Text GLabel 4050 5750 2    50   Output ~ 0
@@
 NoConn ~ 4000 3850
 NoConn ~ 4000 5450
-Text GLabel 4050 5350 2    50   Input ~ 0
+Text GLabel 4050 5150 2    50   Input ~ 0
 ENC_5_PWM
 Text GLabel 3050 5450 0    50   Input ~ 0
@@
 TX_2_Tiva
 Wire Wire Line
-	4000 5350 4050 5350
-Wire Wire Line
-	3100 5550 3050 5550
-Wire Wire Line
 	3100 5450 3050 5450
+Wire Wire Line
+	2100 5650 2150 5650
 Wire Wire Line
 	4000 5150 4050 5150
@@
 NoConn ~ 1200 5450
 NoConn ~ 1200 5650
-NoConn ~ 2100 5650
-NoConn ~ 2100 5550
 NoConn ~ 1200 4350
 NoConn ~ 1200 4450
 NoConn ~ 2100 4350
 NoConn ~ 2100 4250
-Text GLabel 3050 4350 0    50   Input ~ 0
+Text GLabel 2150 5550 2    50   Input ~ 0
 I_SENSE
 Wire Wire Line
@@
 NoConn ~ 4000 4150
 NoConn ~ 4000 4050
+NoConn ~ 2200 4550
+NoConn ~ 3100 5550
+NoConn ~ 3000 5550
+NoConn ~ 2500 4250
+NoConn ~ 4600 5150
+NoConn ~ 850  4750
+NoConn ~ 2150 5100
+NoConn ~ 2500 4350
+NoConn ~ 4000 5350
+NoConn ~ 4100 5350
+NoConn ~ 4500 4600
+NoConn ~ 4500 4800
+NoConn ~ 1100 5450
+Wire Wire Line
+	2100 5550 2150 5550
 $EndSCHEMATC

Commit message: Generated Gerbs
Parts:
- Conn2, Conn5, Conn8: footprint MRDT_Connectors:Anderson_3_Vertical_Side_by_Side -> MRDT_Connectors:Anderson_2_Vertical_Sidy_by_Side
