File: Hardware/ArmBoard_Hardware/ArmBoard_Hardware.kicad_pcb (KiCad board)
At the start: 2 copper layers, 203.2 x 103.5 mm, 200 parts, among them Q1 BSS138, Q10 BSS138, Q11 BSS138, Q12 BSS138, Q13 BSS138, Q14 BSS138, Q15 BSS138, Q16 BSS138, Q2 BSS138, Q3 BSS138, Q31 BUK7M6R3-40EX, Q32 BUK7M6R3-40EX, Q33 BUK7M6R3-40EX, Q34 BUK7M6R3-40EX, Q35 BUK7M6R3-40EX, Q36 BUK7M6R3-40EX, Q37 BUK7M6R3-40EX, Q4 BSS138, Q5 BSS138, Q6 BSS138, Q7 BSS138, Q8 BSS138, Q9 BSS138, SW1 SW_Push, SW2 SW_Push, SW3 SW_Push, SW4 SW_Push, SW5 SW_Push, SW6 SW_Push, SW7 SW_Push, U1 TM4C129E_Launchpad, U2 OKI, U3 VNH5019A_E, U4 VNH5019A_E, U5 VNH5019A_E, U6 VNH5019A_E, U7 VNH5019A_E, U8 VNH5019A_E, U9 VNH5019A_E

Commit message: beginning layout, need to double check footprints and create BOM
Parts:
- moved R82 77.6 mm to (130.8, 28.6)
- moved R42 49.1 mm to (197.5, 100.3)
- moved D15 4.84 mm to (200.4, 144.1)
- moved R15 4.84 mm to (204.2, 144.1)
- moved D10 3.18 mm to (110.5, 23.5)
- moved D30 3.18 mm to (121.3, 23.5)
- moved D31 3.18 mm to (116.4, 22.9)
- moved R10 3.18 mm to (110.5, 27.3)
- moved D26 1.27 mm to (130.8, 25.4)
- moved R24 1.27 mm to (135.9, 25.4)
- moved R96 0.64 mm to (86.4, 95.2)
Changed lines of the file:
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@@
     (42 Eco1.User user)
     (43 Eco2.User user)
-    (44 Edge.Cuts user hide)
+    (44 Edge.Cuts user)
     (45 Margin user)
     (46 B.CrtYd user)
@@
   )
   (module Resistor_SMD:R_0603_1608Metric_Pad0.98x0.95mm_HandSolder (layer F.Cu)
-    (at 86.36 94.615 90)
+    (at 86.36 95.25 90)
     (descr "Resistor SMD 0603 (1608 Metric), square (rectangular) end terminal, IPC_7351 nominal with elongated pad for handsoldering. (Body size source: IPC-SM-782 page 72, https://www.pcb-3d.com/wordpress/wp-content/uploads/ipc-sm-782a_amendment_1_and_2.pdf), generated with kicad-footprint-generator")
     (tags "resistor handsolder")
@@
   )
   (module Resistor_SMD:R_0603_1608Metric_Pad0.98x0.95mm_HandSolder (layer F.Cu)
-    (at 98.564999 99.135001 270)
+    (at 130.81 28.575 270)
     (descr "Resistor SMD 0603 (1608 Metric), square (rectangular) end terminal, IPC_7351 nominal with elongated pad for handsoldering. (Body size source: IPC-SM-782 page 72, https://www.pcb-3d.com/wordpress/wp-content/uploads/ipc-sm-782a_amendment_1_and_2.pdf), generated with kicad-footprint-generator")
     (tags "resistor handsolder")
@@
   )
   (module Resistor_SMD:R_0603_1608Metric_Pad0.98x0.95mm_HandSolder (layer F.Cu)
-    (at 178.015001 145.355001)
+    (at 197.485 100.33)
     (descr "Resistor SMD 0603 (1608 Metric), square (rectangular) end terminal, IPC_7351 nominal with elongated pad for handsoldering. (Body size source: IPC-SM-782 page 72, https://www.pcb-3d.com/wordpress/wp-content/uploads/ipc-sm-782a_amendment_1_and_2.pdf), generated with kicad-footprint-generator")
     (tags "resistor handsolder")
@@
   )
   (module Resistor_SMD:R_0603_1608Metric_Pad0.98x0.95mm_HandSolder (layer F.Cu)
-    (at 135.89 26.67 270)
+    (at 135.89 25.4 270)
     (descr "Resistor SMD 0603 (1608 Metric), square (rectangular) end terminal, IPC_7351 nominal with elongated pad for handsoldering. (Body size source: IPC-SM-782 page 72, https://www.pcb-3d.com/wordpress/wp-content/uploads/ipc-sm-782a_amendment_1_and_2.pdf), generated with kicad-footprint-generator")
     (tags "resistor handsolder")
@@
   )
   (module Resistor_SMD:R_0603_1608Metric_Pad0.98x0.95mm_HandSolder (layer F.Cu)
-    (at 199.7475 142.24)
+    (at 204.1925 144.145)
     (descr "Resistor SMD 0603 (1608 Metric), square (rectangular) end terminal, IPC_7351 nominal with elongated pad for handsoldering. (Body size source: IPC-SM-782 page 72, https://www.pcb-3d.com/wordpress/wp-content/uploads/ipc-sm-782a_amendment_1_and_2.pdf), generated with kicad-footprint-generator")
     (tags "resistor handsolder")
@@
   )
   (module Resistor_SMD:R_0603_1608Metric_Pad0.98x0.95mm_HandSolder (layer F.Cu)
-    (at 110.49 30.48 270)
+    (at 110.49 27.305 270)
     (descr "Resistor SMD 0603 (1608 Metric), square (rectangular) end terminal, IPC_7351 nominal with elongated pad for handsoldering. (Body size source: IPC-SM-782 page 72, https://www.pcb-3d.com/wordpress/wp-content/uploads/ipc-sm-782a_amendment_1_and_2.pdf), generated with kicad-footprint-generator")
     (tags "resistor handsolder")
@@
   )
   (module LED_SMD:LED_0603_1608Metric_Pad1.05x0.95mm_HandSolder (layer F.Cu)
-    (at 116.394999 26.035 270)
+    (at 116.394999 22.86 270)
     (descr "LED SMD 0603 (1608 Metric), square (rectangular) end terminal, IPC_7351 nominal, (Body size source: http://www.tortai-tech.com/upload/download/2011102023233369053.pdf), generated with kicad-footprint-generator")
     (tags "LED handsolder")
@@
   )
   (module LED_SMD:LED_0603_1608Metric_Pad1.05x0.95mm_HandSolder (layer F.Cu)
-    (at 121.285 26.67 270)
+    (at 121.285 23.495 270)
     (descr "LED SMD 0603 (1608 Metric), square (rectangular) end terminal, IPC_7351 nominal, (Body size source: http://www.tortai-tech.com/upload/download/2011102023233369053.pdf), generated with kicad-footprint-generator")
     (tags "LED handsolder")
@@
   )
   (module LED_SMD:LED_0603_1608Metric_Pad1.05x0.95mm_HandSolder (layer F.Cu)
-    (at 130.81 26.67 90)
+    (at 130.81 25.4 90)
     (descr "LED SMD 0603 (1608 Metric), square (rectangular) end terminal, IPC_7351 nominal, (Body size source: http://www.tortai-tech.com/upload/download/2011102023233369053.pdf), generated with kicad-footprint-generator")
     (tags "LED handsolder")
@@
   )
   (module LED_SMD:LED_0603_1608Metric_Pad1.05x0.95mm_HandSolder (layer F.Cu)
-    (at 195.975 142.24)
+    (at 200.42 144.145)
     (descr "LED SMD 0603 (1608 Metric), square (rectangular) end terminal, IPC_7351 nominal, (Body size source: http://www.tortai-tech.com/upload/download/2011102023233369053.pdf), generated with kicad-footprint-generator")
     (tags "LED handsolder")
@@
   )
   (module LED_SMD:LED_0603_1608Metric_Pad1.05x0.95mm_HandSolder (layer F.Cu)
-    (at 110.49 26.67 270)
+    (at 110.49 23.495 270)
     (descr "LED SMD 0603 (1608 Metric), square (rectangular) end terminal, IPC_7351 nominal, (Body size source: http://www.tortai-tech.com/upload/download/2011102023233369053.pdf), generated with kicad-footprint-generator")
     (tags "LED handsolder")

Commit message: beginning layout, need to double check footprints and create BOM
Other:
- outline, holes or cut-outs redrawn
Changed lines of the file:
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@@
     (pad_to_mask_clearance 0)
     (aux_axis_origin 0 0)
-    (visible_elements 7FFFFFFF)
+    (visible_elements 7FFFF7FF)
     (pcbplotparams
       (layerselection 0x010fc_ffffffff)
@@
   (gr_line (start 64.135 28.575) (end 64.135 121.92) (layer Edge.Cuts) (width 0.05))
   (gr_line (start 262.255 23.495) (end 69.215 23.495) (layer Edge.Cuts) (width 0.05))
-  (gr_line (start 266.065 121.92) (end 266.065 28.575) (layer Edge.Cuts) (width 0.05))
+  (gr_line (start 267.335 121.92) (end 267.335 28.575) (layer Edge.Cuts) (width 0.05))
   (gr_line (start 69.215 127) (end 262.255 127) (layer Edge.Cuts) (width 0.05))
   (gr_arc (start 69.215 121.92) (end 64.135 121.92) (angle -90) (layer Edge.Cuts) (width 0.05))
   (gr_arc (start 69.215 28.575) (end 69.215 23.495) (angle -90) (layer Edge.Cuts) (width 0.05))
-  (gr_arc (start 260.985 28.575) (end 266.065 28.575) (angle -90) (layer Edge.Cuts) (width 0.05))
+  (gr_arc (start 262.255 28.575) (end 267.335 28.575) (angle -90) (layer Edge.Cuts) (width 0.05))
   (gr_arc (start 262.255 121.92) (end 262.255 127) (angle -90) (layer Edge.Cuts) (width 0.05))
 )

Commit message: beginning layout, need to double check footprints and create BOM
Parts:
- moved Q12 14.3 mm to (205.1, 31.8)
- moved R19 14.3 mm to (209.6, 31.8)
- moved Conn14 4.86 mm to (253.8, 65.2)
- moved U2 4.26 mm to (236.9, 52.1)
- moved R31 4.26 mm to (236.9, 57.1)
- moved Conn17 4.08 mm to (253.8, 78.9)
- moved Conn13 3.95 mm to (253.8, 51.5)
- moved Q14 3.81 mm to (244.2, 51.4)
- moved Q2 3.81 mm to (244.2, 42.3)
- moved Q3 3.81 mm to (244.2, 46.8)
- moved Conn19 3.70 mm to (212.4, 52.3)
- moved Conn9 3.70 mm to (212.4, 39.7)
- moved Conn16 3.40 mm to (253.8, 106.3)
- moved Conn10 3.38 mm to (253.8, 92.6)
- moved Conn18 3.17 mm to (253.8, 37.8)
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Changed lines of the file:
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@@
     (pad_to_mask_clearance 0)
     (aux_axis_origin 0 0)
-    (visible_elements 7FFFF7FF)
+    (visible_elements 7FFFFFFF)
     (pcbplotparams
       (layerselection 0x010fc_ffffffff)
@@
   )
   (module MRDT_Devices:OKI_Horizontal (layer F.Cu)
-    (at 234.95 48.26 180)
+    (at 236.855 52.07 180)
     (tags OKI)
     (fp_text reference U2 (at 0 -2.54) (layer F.SilkS) hide
@@
   )
   (module Resistor_SMD:R_0603_1608Metric_Pad0.98x0.95mm_HandSolder (layer F.Cu)
-    (at 234.95 53.34 270)
+    (at 236.855 57.15 270)
     (descr "Resistor SMD 0603 (1608 Metric), square (rectangular) end terminal, IPC_7351 nominal with elongated pad for handsoldering. (Body size source: IPC-SM-782 page 72, https://www.pcb-3d.com/wordpress/wp-content/uploads/ipc-sm-782a_amendment_1_and_2.pdf), generated with kicad-footprint-generator")
     (tags "resistor handsolder")
@@
   )
   (module Resistor_SMD:R_0603_1608Metric_Pad0.98x0.95mm_HandSolder (layer F.Cu)
-    (at 222.885 26.67)
+    (at 209.55 31.75)
     (descr "Resistor SMD 0603 (1608 Metric), square (rectangular) end terminal, IPC_7351 nominal with elongated pad for handsoldering. (Body size source: IPC-SM-782 page 72, https://www.pcb-3d.com/wordpress/wp-content/uploads/ipc-sm-782a_amendment_1_and_2.pdf), generated with kicad-footprint-generator")
     (tags "resistor handsolder")
@@
   )
   (module Package_TO_SOT_SMD:SOT-23 (layer F.Cu)
-    (at 244.215001 47.585001)
+    (at 244.215001 51.395001)
     (descr "SOT-23, Standard")
     (tags SOT-23)
@@
   )
   (module Package_TO_SOT_SMD:SOT-23 (layer F.Cu)
-    (at 218.44 26.67)
+    (at 205.105 31.75)
     (descr "SOT-23, Standard")
     (tags SOT-23)
@@
   )
   (module Package_TO_SOT_SMD:SOT-23 (layer F.Cu)
-    (at 244.215001 43.035001)
+    (at 244.215001 46.845001)
     (descr "SOT-23, Standard")
     (tags SOT-23)
@@
   )
   (module Package_TO_SOT_SMD:SOT-23 (layer F.Cu)
-    (at 244.215001 38.485001)
+    (at 244.215001 42.295001)
     (descr "SOT-23, Standard")
     (tags SOT-23)
@@
   )
   (module MRDT_Connectors:MOLEX_SL_02_Horizontal (layer F.Cu)
-    (at 227.584 116.332 270)
+    (at 226.949 117.475 270)
     (fp_text reference Conn20 (at 1.27 2.54 90) (layer F.SilkS) hide
       (effects (font (size 1 1) (thickness 0.15)))
@@
   )
   (module MRDT_Connectors:MOLEX_SL_02_Horizontal (layer F.Cu)
-    (at 210.486999 49.130001 270)
+    (at 212.391999 52.305001 270)
     (fp_text reference Conn19 (at 1.27 2.54 90) (layer F.SilkS) hide
       (effects (font (size 1 1) (thickness 0.15)))
@@
   )
   (module MRDT_Connectors:MOLEX_SL_03_Horizontal (layer F.Cu)
-    (at 251.251999 35.915001 270)
+    (at 253.791999 37.820001 270)
     (fp_text reference Conn18 (at 1.27 2.54 90) (layer F.SilkS) hide
       (effects (font (size 1 1) (thickness 0.15)))
@@
   )
   (module MRDT_Connectors:MOLEX_SL_03_Horizontal (layer F.Cu)
-    (at 251.46 75.565 270)
+    (at 253.791999 78.917499 270)
     (fp_text reference Conn17 (at 1.27 2.54 90) (layer F.SilkS) hide
       (effects (font (size 1 1) (thickness 0.15)))
@@
   )
   (module MRDT_Connectors:MOLEX_SL_02_Horizontal (layer F.Cu)
-    (at 251.079 104.267 270)
+    (at 253.791999 106.315831 270)
     (fp_text reference Conn16 (at 1.27 2.54 90) (layer F.SilkS) hide
       (effects (font (size 1 1) (thickness 0.15)))
@@
   )
   (module MRDT_Connectors:MOLEX_SL_02_Horizontal (layer F.Cu)
-    (at 251.079 116.84 270)
+    (at 253.791999 117.475 270)
     (fp_text reference Conn15 (at 1.27 2.54 90) (layer F.SilkS) hide
       (effects (font (size 1 1) (thickness 0.15)))
@@
   )
   (module MRDT_Connectors:MOLEX_SL_03_Horizontal (layer F.Cu)
-    (at 251.251999 61.075001 270)
+    (at 253.791999 65.218333 270)
     (fp_text reference Conn14 (at 1.27 2.54 90) (layer F.SilkS) hide
       (effects (font (size 1 1) (thickness 0.15)))
@@
   )
   (module MRDT_Connectors:MOLEX_SL_03_Horizontal (layer F.Cu)
-    (at 251.251999 48.495001 270)
+    (at 253.791999 51.519167 270)
     (fp_text reference Conn13 (at 1.27 2.54 90) (layer F.SilkS) hide
       (effects (font (size 1 1) (thickness 0.15)))
@@
   )
   (module MRDT_Connectors:MOLEX_SL_02_Horizontal (layer F.Cu)
-    (at 227.33 104.14 270)
+    (at 226.949 105.791 270)
     (fp_text reference Conn12 (at 1.27 2.54 90) (layer F.SilkS) hide
       (effects (font (size 1 1) (thickness 0.15)))
@@
   )
   (module MRDT_Connectors:MOLEX_SL_02_Horizontal (layer F.Cu)
-    (at 227.584 91.567 270)
+    (at 226.949 94.107 270)
     (fp_text reference Conn11 (at 1.27 2.54 90) (layer F.SilkS) hide
       (effects (font (size 1 1) (thickness 0.15)))
@@
   )
   (module MRDT_Connectors:MOLEX_SL_03_Horizontal (layer F.Cu)
-    (at 251.46 90.17 270)
+    (at 253.791999 92.616665 270)
     (fp_text reference Conn10 (at 1.27 2.54 90) (layer F.SilkS) hide
       (effects (font (size 1 1) (thickness 0.15)))
@@
   )
   (module MRDT_Connectors:MOLEX_SL_03_Horizontal (layer F.Cu)
-    (at 210.486999 36.550001 270)
+    (at 212.391999 39.725001 270)
     (fp_text reference Conn9 (at 1.27 2.54 90) (layer F.SilkS) hide
       (effects (font (size 1 1) (thickness 0.15)))

Commit message: beginning layout, need to double check footprints and create BOM
Parts:
- Conn11, Conn12, Conn19, Conn20: footprint MRDT_Connectors:MOLEX_SL_02_Horizontal -> MRDT_Connectors:MOLEX_SL_02_Vertical
- Conn9: footprint MRDT_Connectors:MOLEX_SL_03_Horizontal -> MRDT_Connectors:MOLEX_SL_03_Vertical
- moved Conn9 12.2 mm to (218.1, 28.9)
- moved Conn19 12.2 mm to (218.1, 41.5)
- moved Conn11 6.38 mm to (233.3, 94.7)
- moved Conn12 6.38 mm to (233.3, 106.4)
- moved Conn20 6.38 mm to (233.3, 118.1)

Commit message: began the layout
Parts:
- moved Conn19 76.2 mm to (219.4, 117.7)
- moved Conn9 76.2 mm to (219.4, 105.1)
- moved Q12 74.4 mm to (208.3, 106.0)
- moved R19 74.4 mm to (212.7, 106.0)
- moved D22 1.27 mm to (225.4, 88.3)
- moved D7 1.27 mm to (221.6, 83.8)
- moved R22 1.27 mm to (221.4, 91.0)
- moved R7 1.27 mm to (221.4, 88.5)
- moved Conn11 1.27 mm to (234.6, 94.7)
- moved Conn12 1.27 mm to (234.6, 106.4)
- moved Conn20 1.27 mm to (234.6, 118.1)
- moved D28 1.27 mm to (210.8, 95.9)
- moved R28 1.27 mm to (217.0, 96.0)
- moved R32 1.27 mm to (221.3, 93.5)
- moved R36 1.27 mm to (217.1, 88.5)
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
Commit message: layout
Parts:
- moved D18 115.2 mm to (171.4, 138.4)
- moved R18 115.2 mm to (166.9, 138.4)
- moved D17 111.8 mm to (237.5, 87.6)
- moved R17 111.8 mm to (233.7, 87.6)
- moved Q5 111.8 mm to (233.0, 83.3)
- moved D31 107.4 mm to (222.9, 36.8)
- moved R10 103.8 mm to (213.4, 41.3)
- moved D10 103.7 mm to (213.4, 36.8)
- moved D30 98.1 mm to (218.4, 36.8)
- moved R98 88.8 mm to (161.9, 61.0), turned to 0 degrees
- moved D20 87.8 mm to (171.8, 94.6)
- moved R20 87.8 mm to (175.3, 94.6)
- moved D29 76.8 mm to (118.7, 90.2), turned to 0 degrees
- moved R3 76.3 mm to (184.8, 24.1), turned to 0 degrees
- moved Q7 76.0 mm to (215.3, 86.4)
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
Commit message: layout
Parts:
- moved U1 148.6 mm to (188.6, 40.6)
- moved Q15 126.5 mm to (242.6, 118.7), turned to 90 degrees
- moved D32 85.3 mm to (86.4, 95.3)
- moved R87 78.7 mm to (201.0, 81.0), turned to 180 degrees
- moved R82 71.1 mm to (96.5, 90.8)
- moved D26 71.1 mm to (96.5, 87.6)
- moved R24 69.7 mm to (96.5, 83.8)
- moved R83 65.5 mm to (205.7, 80.6), turned to 180 degrees
- moved Q6 58.7 mm to (149.9, 90.2)
- moved D15 56.5 mm to (180.1, 83.8)
- moved R15 56.4 mm to (184.8, 83.8)
- moved R47 52.1 mm to (189.2, 87.0)
- moved D18 52.0 mm to (192.4, 90.8)
- moved R18 52.0 mm to (187.9, 90.8)
- moved R41 46.5 mm to (154.5, 102.0), turned to 90 degrees
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
Commit message: layout
Parts:
- moved Conn1 23.5 mm to (249.6, 6.99)
- moved Conn2 23.5 mm to (237.7, 6.68)
- moved Conn3 23.5 mm to (188.7, 6.84)
- moved Conn4 23.5 mm to (197.7, 6.84)
- moved Conn6 23.5 mm to (228.7, 6.68)
- moved Conn8 23.5 mm to (258.4, 6.99)
- moved Conn5 23.5 mm to (208.4, 6.76)
- moved Conn7 23.5 mm to (217.4, 6.76)
- moved R77 3.81 mm to (102.9, 99.7)
- moved U4 2.83 mm to (202.8, 105.0)
- moved U5 2.43 mm to (183.1, 105.0)
- moved R88 2.33 mm to (100.1, 99.7)
- moved U3 1.97 mm to (163.3, 105.0)
- moved Q31 1.67 mm to (148.0, 98.0)
- moved Q2 1.66 mm to (244.2, 40.6)
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