File: Hardware/ArmBoard_Hardware/Motor_Controller_7-Gripper.sch (KiCad schematic (older format))
At the start: 9 parts

Commit message: Added MotorToggles
Removed extra schematic files, added a MotorToggle sheet for the toggle buttons, sheet docs were updated
Parts:
- gave numbers to parts that had none: 9
Changed lines of the file:
@@
 $Descr A4 11693 8268
 encoding utf-8
-Sheet 3 4
-Title ""
-Date ""
-Rev ""
-Comp ""
-Comment1 ""
+Sheet 3 5
+Title "ArmBoard_Hardware"
+Date "2021-10-15"
+Rev "0"
+Comp "Mars Rover Design Team"
+Comment1 "Drawn By: Patrick Simoni / Tyler Lunyou"
 Comment2 ""
 Comment3 ""
@@
 AR Path="/62175536/619EFCE6/6211CA1F" Ref="U?"  Part="1"
 AR Path="/6352A0DC/6211CA1F" Ref="U?"  Part="1"
-AR Path="/63845F62/6211CA1F" Ref="U?"  Part="1"
-F 0 "U?" H 4200 5037 60  0000 C CNN
+AR Path="/63845F62/6211CA1F" Ref="U6"  Part="1"
+F 0 "U6" H 4200 5037 60  0000 C CNN
 F 1 "VNH5019A_E" H 4200 4931 60  0000 C CNN
 F 2 "" H 3600 4650 60  0001 C CNN
@@
 AR Path="/62175536/619EFCE6/6211CA25" Ref="Q?"  Part="1"
 AR Path="/6352A0DC/6211CA25" Ref="Q?"  Part="1"
-AR Path="/63845F62/6211CA25" Ref="Q?"  Part="1"
-F 0 "Q?" V 5450 3450 50  0000 C CNN
+AR Path="/63845F62/6211CA25" Ref="Q34"  Part="1"
+F 0 "Q34" V 5450 3450 50  0000 C CNN
 F 1 "BUK7M6R3-40EX" V 5350 3600 50  0000 C CNN
 F 2 "Package_TO_SOT_SMD:LFPAK33" H 5650 3175 50  0001 L CIN
@@
 AR Path="/62175536/619EFCE6/6211CA30" Ref="#PWR?"  Part="1"
 AR Path="/6352A0DC/6211CA30" Ref="#PWR?"  Part="1"
-AR Path="/63845F62/6211CA30" Ref="#PWR?"  Part="1"
-F 0 "#PWR?" H 3150 2000 50  0001 C CNN
+AR Path="/63845F62/6211CA30" Ref="#PWR0124"  Part="1"
+F 0 "#PWR0124" H 3150 2000 50  0001 C CNN
 F 1 "+3.3V" H 3000 2200 50  0000 C CNN
 F 2 "" H 3150 2150 50  0001 C CNN
@@
 AR Path="/62175536/619EFCE6/6211CA37" Ref="R?"  Part="1"
 AR Path="/6352A0DC/6211CA37" Ref="R?"  Part="1"
-AR Path="/63845F62/6211CA37" Ref="R?"  Part="1"
-F 0 "R?" H 3350 2250 50  0000 R CNN
+AR Path="/63845F62/6211CA37" Ref="R67"  Part="1"
+F 0 "R67" H 3350 2250 50  0000 R CNN
 F 1 "3.3k" H 3350 2350 50  0000 R CNN
 F 2 "" H 3150 2300 50  0001 C CNN
@@
 AR Path="/62175536/619EFCE6/6211CA3F" Ref="R?"  Part="1"
 AR Path="/6352A0DC/6211CA3F" Ref="R?"  Part="1"
-AR Path="/63845F62/6211CA3F" Ref="R?"  Part="1"
-F 0 "R?" V 3100 2450 50  0000 C CNN
+AR Path="/63845F62/6211CA3F" Ref="R66"  Part="1"
+F 0 "R66" V 3100 2450 50  0000 C CNN
 F 1 "1k" V 3000 2450 50  0000 C CNN
 F 2 "" H 3000 2450 50  0001 C CNN
@@
 AR Path="/62175536/619EFCE6/6211CA4A" Ref="#PWR?"  Part="1"
 AR Path="/6352A0DC/6211CA4A" Ref="#PWR?"  Part="1"
-AR Path="/63845F62/6211CA4A" Ref="#PWR?"  Part="1"
-F 0 "#PWR?" H 2900 3200 50  0001 C CNN
+AR Path="/63845F62/6211CA4A" Ref="#PWR0123"  Part="1"
+F 0 "#PWR0123" H 2900 3200 50  0001 C CNN
 F 1 "+3.3V" H 3000 3500 50  0000 C CNN
 F 2 "" H 2900 3350 50  0001 C CNN
@@
 AR Path="/62175536/619EFCE6/6211CA52" Ref="R?"  Part="1"
 AR Path="/6352A0DC/6211CA52" Ref="R?"  Part="1"
-AR Path="/63845F62/6211CA52" Ref="R?"  Part="1"
-F 0 "R?" H 2959 3546 50  0000 L CNN
+AR Path="/63845F62/6211CA52" Ref="R64"  Part="1"
+F 0 "R64" H 2959 3546 50  0000 L CNN
 F 1 "3.3k" H 2959 3455 50  0000 L CNN
 F 2 "" H 2900 3500 50  0001 C CNN
@@
 AR Path="/62175536/619EFCE6/6211CA59" Ref="R?"  Part="1"
 AR Path="/6352A0DC/6211CA59" Ref="R?"  Part="1"
-AR Path="/63845F62/6211CA59" Ref="R?"  Part="1"
-F 0 "R?" V 2850 3650 50  0000 C CNN
+AR Path="/63845F62/6211CA59" Ref="R63"  Part="1"
+F 0 "R63" V 2850 3650 50  0000 C CNN
 F 1 "1k" V 2750 3650 50  0000 C CNN
 F 2 "" H 2750 3650 50  0001 C CNN
@@
 AR Path="/62175536/619EFCE6/6211CA93" Ref="#PWR?"  Part="1"
 AR Path="/6352A0DC/6211CA93" Ref="#PWR?"  Part="1"
-AR Path="/63845F62/6211CA93" Ref="#PWR?"  Part="1"
-F 0 "#PWR?" H 4200 3400 50  0001 C CNN
+AR Path="/63845F62/6211CA93" Ref="#PWR0125"  Part="1"
+F 0 "#PWR0125" H 4200 3400 50  0001 C CNN
 F 1 "GND" H 4350 3550 50  0000 C CNN
 F 2 "" H 4200 3650 50  0001 C CNN
@@
 AR Path="/62175536/619EFCE6/6211CAA7" Ref="#PWR?"  Part="1"
 AR Path="/6352A0DC/6211CAA7" Ref="#PWR?"  Part="1"
-AR Path="/63845F62/6211CAA7" Ref="#PWR?"  Part="1"
-F 0 "#PWR?" H 5200 2900 50  0001 C CNN
+AR Path="/63845F62/6211CAA7" Ref="#PWR0126"  Part="1"
+F 0 "#PWR0126" H 5200 2900 50  0001 C CNN
 F 1 "+12VA" H 5215 3223 50  0000 C CNN
 F 2 "" H 5200 3050 50  0001 C CNN
@@
 AR Path="/62175536/619EFCE6/6211CAB3" Ref="#PWR?"  Part="1"
 AR Path="/6352A0DC/6211CAB3" Ref="#PWR?"  Part="1"
-AR Path="/63845F62/6211CAB3" Ref="#PWR?"  Part="1"
-F 0 "#PWR?" H 2200 2600 50  0001 C CNN
+AR Path="/63845F62/6211CAB3" Ref="#PWR0121"  Part="1"
+F 0 "#PWR0121" H 2200 2600 50  0001 C CNN
 F 1 "+3.3V" H 2300 2900 50  0000 C CNN
 F 2 "" H 2200 2750 50  0001 C CNN
@@
 AR Path="/62175536/619EFCE6/6211CABB" Ref="#PWR?"  Part="1"
 AR Path="/6352A0DC/6211CABB" Ref="#PWR?"  Part="1"
-AR Path="/63845F62/6211CABB" Ref="#PWR?"  Part="1"
-F 0 "#PWR?" H 2200 2750 50  0001 C CNN
+AR Path="/63845F62/6211CABB" Ref="#PWR0122"  Part="1"
+F 0 "#PWR0122" H 2200 2750 50  0001 C CNN
 F 1 "GND" H 2200 2850 50  0000 C CNN
 F 2 "" H 2200 3000 50  0001 C CNN
@@
 AR Path="/62175536/619EFCE6/6211CAC3" Ref="R?"  Part="1"
 AR Path="/6352A0DC/6211CAC3" Ref="R?"  Part="1"
-AR Path="/63845F62/6211CAC3" Ref="R?"  Part="1"
-F 0 "R?" V 2600 3000 50  0000 C CNN
+AR Path="/63845F62/6211CAC3" Ref="R62"  Part="1"
+F 0 "R62" V 2600 3000 50  0000 C CNN
 F 1 "1k" V 2700 3000 50  0000 C CNN
 F 2 "" H 2700 3000 50  0001 C CNN
@@
 AR Path="/62175536/619EFCE6/6211CAC9" Ref="R?"  Part="1"
 AR Path="/6352A0DC/6211CAC9" Ref="R?"  Part="1"
-AR Path="/63845F62/6211CAC9" Ref="R?"  Part="1"
-F 0 "R?" V 2600 2750 50  0000 C CNN
+AR Path="/63845F62/6211CAC9" Ref="R61"  Part="1"
+F 0 "R61" V 2600 2750 50  0000 C CNN
 F 1 "1k" V 2700 2750 50  0000 C CNN
 F 2 "" H 2700 2750 50  0001 C CNN
@@
 AR Path="/62175536/619EFCE6/6211CACF" Ref="R?"  Part="1"
 AR Path="/6352A0DC/6211CACF" Ref="R?"  Part="1"
-AR Path="/63845F62/6211CACF" Ref="R?"  Part="1"
-F 0 "R?" V 2850 2900 50  0000 C CNN
+AR Path="/63845F62/6211CACF" Ref="R65"  Part="1"
+F 0 "R65" V 2850 2900 50  0000 C CNN
 F 1 "1k" V 2950 2900 50  0000 C CNN
 F 2 "" H 2950 2900 50  0001 C CNN

Commit message: need to change the mosfet and the other footrpints under it
Parts:
- R100: renamed from R65; footprint (none) -> Resistor_SMD:R_0603_1608Metric_Pad0.98x0.95mm_HandSolder
- R101: renamed from R66; footprint (none) -> Resistor_SMD:R_0603_1608Metric_Pad0.98x0.95mm_HandSolder
- R102: renamed from R67; footprint (none) -> Resistor_SMD:R_0603_1608Metric_Pad0.98x0.95mm_HandSolder
- R96: renamed from R61; footprint (none) -> Resistor_SMD:R_0603_1608Metric_Pad0.98x0.95mm_HandSolder
- R97: renamed from R62; footprint (none) -> Resistor_SMD:R_0603_1608Metric_Pad0.98x0.95mm_HandSolder
- R98: renamed from R63; footprint (none) -> Resistor_SMD:R_0603_1608Metric_Pad0.98x0.95mm_HandSolder
- R99: renamed from R64; footprint (none) -> Resistor_SMD:R_0603_1608Metric_Pad0.98x0.95mm_HandSolder
- U9: renamed from U6; footprint (none) -> MRDT_ICs:MultiPowerSO_30
- renumbered Q34 to Q37
Changed lines of the file:
@@
 $Descr A4 11693 8268
 encoding utf-8
-Sheet 3 5
+Sheet 5 5
 Title "ArmBoard_Hardware"
 Date "2021-10-15"
@@
 AR Path="/62175536/619EFCE6/6211CA1F" Ref="U?"  Part="1"
 AR Path="/6352A0DC/6211CA1F" Ref="U?"  Part="1"
-AR Path="/63845F62/6211CA1F" Ref="U6"  Part="1"
-F 0 "U6" H 4200 5037 60  0000 C CNN
+AR Path="/63845F62/6211CA1F" Ref="U9"  Part="1"
+F 0 "U9" H 4200 5037 60  0000 C CNN
 F 1 "VNH5019A_E" H 4200 4931 60  0000 C CNN
-F 2 "" H 3600 4650 60  0001 C CNN
+F 2 "MRDT_ICs:MultiPowerSO_30" H 3600 4650 60  0001 C CNN
 F 3 "" H 3600 4650 60  0001 C CNN
 	1    3600 3350
@@
 AR Path="/62175536/619EFCE6/6211CA25" Ref="Q?"  Part="1"
 AR Path="/6352A0DC/6211CA25" Ref="Q?"  Part="1"
-AR Path="/63845F62/6211CA25" Ref="Q34"  Part="1"
-F 0 "Q34" V 5450 3450 50  0000 C CNN
+AR Path="/63845F62/6211CA25" Ref="Q37"  Part="1"
+F 0 "Q37" V 5450 3450 50  0000 C CNN
 F 1 "BUK7M6R3-40EX" V 5350 3600 50  0000 C CNN
 F 2 "Package_TO_SOT_SMD:LFPAK33" H 5650 3175 50  0001 L CIN
@@
 AR Path="/62175536/619EFCE6/6211CA30" Ref="#PWR?"  Part="1"
 AR Path="/6352A0DC/6211CA30" Ref="#PWR?"  Part="1"
-AR Path="/63845F62/6211CA30" Ref="#PWR0124"  Part="1"
-F 0 "#PWR0124" H 3150 2000 50  0001 C CNN
+AR Path="/63845F62/6211CA30" Ref="#PWR0142"  Part="1"
+F 0 "#PWR0142" H 3150 2000 50  0001 C CNN
 F 1 "+3.3V" H 3000 2200 50  0000 C CNN
 F 2 "" H 3150 2150 50  0001 C CNN
@@
 AR Path="/62175536/619EFCE6/6211CA37" Ref="R?"  Part="1"
 AR Path="/6352A0DC/6211CA37" Ref="R?"  Part="1"
-AR Path="/63845F62/6211CA37" Ref="R67"  Part="1"
-F 0 "R67" H 3350 2250 50  0000 R CNN
+AR Path="/63845F62/6211CA37" Ref="R102"  Part="1"
+F 0 "R102" H 3350 2250 50  0000 R CNN
 F 1 "3.3k" H 3350 2350 50  0000 R CNN
-F 2 "" H 3150 2300 50  0001 C CNN
+F 2 "Resistor_SMD:R_0603_1608Metric_Pad0.98x0.95mm_HandSolder" H 3150 2300 50  0001 C CNN
 F 3 "~" H 3150 2300 50  0001 C CNN
 	1    3150 2300
@@
 AR Path="/62175536/619EFCE6/6211CA3F" Ref="R?"  Part="1"
 AR Path="/6352A0DC/6211CA3F" Ref="R?"  Part="1"
-AR Path="/63845F62/6211CA3F" Ref="R66"  Part="1"
-F 0 "R66" V 3100 2450 50  0000 C CNN
+AR Path="/63845F62/6211CA3F" Ref="R101"  Part="1"
+F 0 "R101" V 3100 2450 50  0000 C CNN
 F 1 "1k" V 3000 2450 50  0000 C CNN
-F 2 "" H 3000 2450 50  0001 C CNN
+F 2 "Resistor_SMD:R_0603_1608Metric_Pad0.98x0.95mm_HandSolder" H 3000 2450 50  0001 C CNN
 F 3 "~" H 3000 2450 50  0001 C CNN
 	1    3000 2450
@@
 AR Path="/62175536/619EFCE6/6211CA4A" Ref="#PWR?"  Part="1"
 AR Path="/6352A0DC/6211CA4A" Ref="#PWR?"  Part="1"
-AR Path="/63845F62/6211CA4A" Ref="#PWR0123"  Part="1"
-F 0 "#PWR0123" H 2900 3200 50  0001 C CNN
+AR Path="/63845F62/6211CA4A" Ref="#PWR0141"  Part="1"
+F 0 "#PWR0141" H 2900 3200 50  0001 C CNN
 F 1 "+3.3V" H 3000 3500 50  0000 C CNN
 F 2 "" H 2900 3350 50  0001 C CNN
@@
 AR Path="/62175536/619EFCE6/6211CA52" Ref="R?"  Part="1"
 AR Path="/6352A0DC/6211CA52" Ref="R?"  Part="1"
-AR Path="/63845F62/6211CA52" Ref="R64"  Part="1"
-F 0 "R64" H 2959 3546 50  0000 L CNN
+AR Path="/63845F62/6211CA52" Ref="R99"  Part="1"
+F 0 "R99" H 2959 3546 50  0000 L CNN
 F 1 "3.3k" H 2959 3455 50  0000 L CNN
-F 2 "" H 2900 3500 50  0001 C CNN
+F 2 "Resistor_SMD:R_0603_1608Metric_Pad0.98x0.95mm_HandSolder" H 2900 3500 50  0001 C CNN
 F 3 "~" H 2900 3500 50  0001 C CNN
 	1    2900 3500
@@
 AR Path="/62175536/619EFCE6/6211CA59" Ref="R?"  Part="1"
 AR Path="/6352A0DC/6211CA59" Ref="R?"  Part="1"
-AR Path="/63845F62/6211CA59" Ref="R63"  Part="1"
-F 0 "R63" V 2850 3650 50  0000 C CNN
+AR Path="/63845F62/6211CA59" Ref="R98"  Part="1"
+F 0 "R98" V 2850 3650 50  0000 C CNN
 F 1 "1k" V 2750 3650 50  0000 C CNN
-F 2 "" H 2750 3650 50  0001 C CNN
+F 2 "Resistor_SMD:R_0603_1608Metric_Pad0.98x0.95mm_HandSolder" H 2750 3650 50  0001 C CNN
 F 3 "~" H 2750 3650 50  0001 C CNN
 	1    2750 3650
@@
 AR Path="/62175536/619EFCE6/6211CA93" Ref="#PWR?"  Part="1"
 AR Path="/6352A0DC/6211CA93" Ref="#PWR?"  Part="1"
-AR Path="/63845F62/6211CA93" Ref="#PWR0125"  Part="1"
-F 0 "#PWR0125" H 4200 3400 50  0001 C CNN
+AR Path="/63845F62/6211CA93" Ref="#PWR0143"  Part="1"
+F 0 "#PWR0143" H 4200 3400 50  0001 C CNN
 F 1 "GND" H 4350 3550 50  0000 C CNN
 F 2 "" H 4200 3650 50  0001 C CNN
@@
 AR Path="/62175536/619EFCE6/6211CAA7" Ref="#PWR?"  Part="1"
 AR Path="/6352A0DC/6211CAA7" Ref="#PWR?"  Part="1"
-AR Path="/63845F62/6211CAA7" Ref="#PWR0126"  Part="1"
-F 0 "#PWR0126" H 5200 2900 50  0001 C CNN
+AR Path="/63845F62/6211CAA7" Ref="#PWR0144"  Part="1"
+F 0 "#PWR0144" H 5200 2900 50  0001 C CNN
 F 1 "+12VA" H 5215 3223 50  0000 C CNN
 F 2 "" H 5200 3050 50  0001 C CNN
@@
 AR Path="/62175536/619EFCE6/6211CAB3" Ref="#PWR?"  Part="1"
 AR Path="/6352A0DC/6211CAB3" Ref="#PWR?"  Part="1"
-AR Path="/63845F62/6211CAB3" Ref="#PWR0121"  Part="1"
-F 0 "#PWR0121" H 2200 2600 50  0001 C CNN
+AR Path="/63845F62/6211CAB3" Ref="#PWR0139"  Part="1"
+F 0 "#PWR0139" H 2200 2600 50  0001 C CNN
 F 1 "+3.3V" H 2300 2900 50  0000 C CNN
 F 2 "" H 2200 2750 50  0001 C CNN
@@
 AR Path="/62175536/619EFCE6/6211CABB" Ref="#PWR?"  Part="1"
 AR Path="/6352A0DC/6211CABB" Ref="#PWR?"  Part="1"
-AR Path="/63845F62/6211CABB" Ref="#PWR0122"  Part="1"
-F 0 "#PWR0122" H 2200 2750 50  0001 C CNN
+AR Path="/63845F62/6211CABB" Ref="#PWR0140"  Part="1"
+F 0 "#PWR0140" H 2200 2750 50  0001 C CNN
 F 1 "GND" H 2200 2850 50  0000 C CNN
 F 2 "" H 2200 3000 50  0001 C CNN
@@
 AR Path="/62175536/619EFCE6/6211CAC3" Ref="R?"  Part="1"
 AR Path="/6352A0DC/6211CAC3" Ref="R?"  Part="1"
-AR Path="/63845F62/6211CAC3" Ref="R62"  Part="1"
-F 0 "R62" V 2600 3000 50  0000 C CNN
+AR Path="/63845F62/6211CAC3" Ref="R97"  Part="1"
+F 0 "R97" V 2600 3000 50  0000 C CNN
 F 1 "1k" V 2700 3000 50  0000 C CNN
-F 2 "" H 2700 3000 50  0001 C CNN
+F 2 "Resistor_SMD:R_0603_1608Metric_Pad0.98x0.95mm_HandSolder" H 2700 3000 50  0001 C CNN
 F 3 "~" H 2700 3000 50  0001 C CNN
 	1    2700 3000
@@
 AR Path="/62175536/619EFCE6/6211CAC9" Ref="R?"  Part="1"
 AR Path="/6352A0DC/6211CAC9" Ref="R?"  Part="1"
-AR Path="/63845F62/6211CAC9" Ref="R61"  Part="1"
-F 0 "R61" V 2600 2750 50  0000 C CNN
+AR Path="/63845F62/6211CAC9" Ref="R96"  Part="1"
+F 0 "R96" V 2600 2750 50  0000 C CNN
 F 1 "1k" V 2700 2750 50  0000 C CNN
-F 2 "" H 2700 2750 50  0001 C CNN
+F 2 "Resistor_SMD:R_0603_1608Metric_Pad0.98x0.95mm_HandSolder" H 2700 2750 50  0001 C CNN
 F 3 "~" H 2700 2750 50  0001 C CNN
 	1    2700 2750
@@
 AR Path="/62175536/619EFCE6/6211CACF" Ref="R?"  Part="1"
 AR Path="/6352A0DC/6211CACF" Ref="R?"  Part="1"
-AR Path="/63845F62/6211CACF" Ref="R65"  Part="1"
-F 0 "R65" V 2850 2900 50  0000 C CNN
+AR Path="/63845F62/6211CACF" Ref="R100"  Part="1"
+F 0 "R100" V 2850 2900 50  0000 C CNN
 F 1 "1k" V 2950 2900 50  0000 C CNN
-F 2 "" H 2950 2900 50  0001 C CNN
+F 2 "Resistor_SMD:R_0603_1608Metric_Pad0.98x0.95mm_HandSolder" H 2950 2900 50  0001 C CNN
 F 3 "~" H 2950 2900 50  0001 C CNN
 	1    2950 2900

Commit message: late night with the boy
Parts:
- removed Q37: BUK7M6R3-40EX, Package_TO_SOT_SMD:LFPAK33, symbol Transistor_FET:BUK7M6R3-40EX
- removed R100, R101, R96, R97, R98: 1k, Resistor_SMD:R_0603_1608Metric_Pad0.98x0.95mm_HandSolder, symbol Device:R_Small
- removed R102, R99: 3.3k, Resistor_SMD:R_0603_1608Metric_Pad0.98x0.95mm_HandSolder, symbol Device:R_Small
- removed U9: VNH5019A_E, MRDT_ICs:MultiPowerSO_30, symbol ArmBoard_Hardware-rescue:VNH5019A_E-MRDT_ICs
- added C11: C_Small, Capacitor_SMD:C_0603_1608Metric_Pad1.08x0.95mm_HandSolder, symbol Device:C_Small
- added R58: 20k, Resistor_SMD:R_0603_1608Metric_Pad0.98x0.95mm_HandSolder, symbol Device:R
- added R59, R60: 1k, Resistor_SMD:R_0603_1608Metric_Pad0.98x0.95mm_HandSolder, symbol Device:R_Small
- added U16: LTC6900, Package_TO_SOT_SMD:SOT-23-5_HandSoldering, symbol MRDT_Devices:LTC6900
- added U17: TB67H400AFNG,EL, MRDT_ICs:TB67H400AFNG,EL, symbol MRDT_ICs:TB67H400AFNG,EL
Connections:
- net labels added: +5V
- net labels removed: +3.3V, ENa_7, ENb_7
- wire segments 76 -> 55
- no-connect marks 0 -> 4

Commit message: Fixed Oscillators
Parts:
- C11: value C_Small -> .1uF
- U16: symbol MRDT_Devices:LTC6900 -> ArmBoard_Hardware-rescue:LTC6900-MRDT_Devices
- U17: symbol MRDT_ICs:TB67H400AFNG,EL -> ArmBoard_Hardware-rescue:TB67H400AFNG,EL-MRDT_ICs
Connections:
- net +5V: now also R58.1
- net GND: now also C11.2
Other:
- moved on the sheet: C11
Changed lines of the file:
@@
 Wire Wire Line
 	1395 1525 1400 1525
-Wire Wire Line
-	1395 1375 1395 1525
 $Comp
 L Device:C_Small C?
 U 1 1 6248952B
-P 1395 1275
+P 1275 1275
 AR Path="/63845F20/6248952B" Ref="C?"  Part="1"
 AR Path="/63845F62/6248952B" Ref="C11"  Part="1"
-F 0 "C11" H 1487 1321 50  0000 L CNN
-F 1 "C_Small" H 1487 1230 50  0000 L CNN
-F 2 "Capacitor_SMD:C_0603_1608Metric_Pad1.08x0.95mm_HandSolder" H 1395 1275 50  0001 C CNN
-F 3 "~" H 1395 1275 50  0001 C CNN
-	1    1395 1275
+F 0 "C11" H 1367 1321 50  0000 L CNN
+F 1 ".1uF" H 1367 1230 50  0000 L CNN
+F 2 "Capacitor_SMD:C_0603_1608Metric_Pad1.08x0.95mm_HandSolder" H 1275 1275 50  0001 C CNN
+F 3 "~" H 1275 1275 50  0001 C CNN
+	1    1275 1275
 	1    0    0    -1
 $EndComp
@@
 	2420 1425 2960 1425
 $Comp
-L MRDT_Devices:LTC6900 U?
+L ArmBoard_Hardware-rescue:LTC6900-MRDT_Devices U?
 U 1 1 62489547
 P 2030 1385
 AR Path="/63845F20/62489547" Ref="U?"  Part="1"
 AR Path="/63845F62/62489547" Ref="U16"  Part="1"
+AR Path="/62489547" Ref="U16"  Part="1"
 F 0 "U16" H 2100 1670 50  0000 C CNN
 F 1 "LTC6900" H 2100 1579 50  0000 C CNN
@@
 	3760 4325 3760 4200
 $Comp
-L MRDT_ICs:TB67H400AFNG,EL U?
+L ArmBoard_Hardware-rescue:TB67H400AFNG,EL-MRDT_ICs U?
 U 1 1 62489598
 P 3760 2775
@@
 Text GLabel 2810 3620 0    50   Output ~ 0
 OUTa_7
+Wire Wire Line
+	1275 1375 1275 1425
+Connection ~ 1275 1425
+Wire Wire Line
+	1395 1175 1275 1175
+Wire Wire Line
+	1395 1175 1395 1525
+Connection ~ 1395 1175
 $EndSCHEMATC

Commit message: armboard review
Parts:
- removed C11: .1uF, Capacitor_SMD:C_0603_1608Metric_Pad1.08x0.95mm_HandSolder, symbol Device:C_Small
- removed R58: 20k, Resistor_SMD:R_0603_1608Metric_Pad0.98x0.95mm_HandSolder, symbol Device:R
- removed U16: LTC6900, Package_TO_SOT_SMD:SOT-23-5_HandSoldering, symbol ArmBoard_Hardware-rescue:LTC6900-MRDT_Devices
Connections:
- net OSC: now reaches U17.1 (OSCM)
- no-connect marks 4 -> 3
Changed lines of the file:
@@
 Wire Wire Line
 	2235 2425 2235 2725
-Wire Wire Line
-	1605 1175 1780 1175
-Connection ~ 1605 1175
-Wire Wire Line
-	1605 1175 1605 1140
-Wire Wire Line
-	1395 1175 1605 1175
-Wire Wire Line
-	1780 1175 1780 1325
-$Comp
-L power:+5V #PWR?
-U 1 1 62489523
-P 1605 1140
-AR Path="/63845F20/62489523" Ref="#PWR?"  Part="1"
-AR Path="/63845F62/62489523" Ref="#PWR0107"  Part="1"
-F 0 "#PWR0107" H 1605 990 50  0001 C CNN
-F 1 "+5V" H 1620 1313 50  0000 C CNN
-F 2 "" H 1605 1140 50  0001 C CNN
-F 3 "" H 1605 1140 50  0001 C CNN
-	1    1605 1140
-	1    0    0    -1
-$EndComp
-Wire Wire Line
-	1395 1525 1400 1525
-$Comp
-L Device:C_Small C?
-U 1 1 6248952B
-P 1275 1275
-AR Path="/63845F20/6248952B" Ref="C?"  Part="1"
-AR Path="/63845F62/6248952B" Ref="C11"  Part="1"
-F 0 "C11" H 1367 1321 50  0000 L CNN
-F 1 ".1uF" H 1367 1230 50  0000 L CNN
-F 2 "Capacitor_SMD:C_0603_1608Metric_Pad1.08x0.95mm_HandSolder" H 1275 1275 50  0001 C CNN
-F 3 "~" H 1275 1275 50  0001 C CNN
-	1    1275 1275
-	1    0    0    -1
-$EndComp
-Wire Wire Line
-	1700 1525 1780 1525
-$Comp
-L Device:R R?
-U 1 1 62489532
-P 1550 1525
-AR Path="/63845F20/62489532" Ref="R?"  Part="1"
-AR Path="/63845F62/62489532" Ref="R58"  Part="1"
-F 0 "R58" V 1757 1525 50  0000 C CNN
-F 1 "20k" V 1666 1525 50  0000 C CNN
-F 2 "Resistor_SMD:R_0603_1608Metric_Pad0.98x0.95mm_HandSolder" V 1480 1525 50  0001 C CNN
-F 3 "~" H 1550 1525 50  0001 C CNN
-	1    1550 1525
-	0    -1   -1   0
-$EndComp
-Wire Wire Line
-	1275 1425 1780 1425
-NoConn ~ 1780 1625
-$Comp
-L power:GND #PWR?
-U 1 1 6248953A
-P 1275 1425
-AR Path="/6248953A" Ref="#PWR?"  Part="1"
-AR Path="/62175536/61C88AE8/6248953A" Ref="#PWR?"  Part="1"
-AR Path="/62175536/619EC506/6248953A" Ref="#PWR?"  Part="1"
-AR Path="/6352A127/6248953A" Ref="#PWR?"  Part="1"
-AR Path="/6352A1A0/6248953A" Ref="#PWR?"  Part="1"
-AR Path="/635FA3DE/6248953A" Ref="#PWR?"  Part="1"
-AR Path="/635FA457/6248953A" Ref="#PWR?"  Part="1"
-AR Path="/63845F20/6248953A" Ref="#PWR?"  Part="1"
-AR Path="/63845F62/6248953A" Ref="#PWR0106"  Part="1"
-F 0 "#PWR0106" H 1275 1175 50  0001 C CNN
-F 1 "GND" H 1150 1460 50  0000 C CNN
-F 2 "" H 1275 1425 50  0001 C CNN
-F 3 "" H 1275 1425 50  0001 C CNN
-	1    1275 1425
-	1    0    0    -1
-$EndComp
 $Comp
 L power:+5V #PWR?
@@
 Wire Wire Line
 	2420 1425 2960 1425
-$Comp
-L ArmBoard_Hardware-rescue:LTC6900-MRDT_Devices U?
-U 1 1 62489547
-P 2030 1385
-AR Path="/63845F20/62489547" Ref="U?"  Part="1"
-AR Path="/63845F62/62489547" Ref="U16"  Part="1"
-AR Path="/62489547" Ref="U16"  Part="1"
-F 0 "U16" H 2100 1670 50  0000 C CNN
-F 1 "LTC6900" H 2100 1579 50  0000 C CNN
-F 2 "Package_TO_SOT_SMD:SOT-23-5_HandSoldering" H 2030 1385 50  0001 C CNN
-F 3 "" H 2030 1385 50  0001 C CNN
-	1    2030 1385
-	1    0    0    -1
-$EndComp
 Wire Wire Line
 	2735 1825 2960 1825
@@
 Text GLabel 2810 3620 0    50   Output ~ 0
 OUTa_7
-Wire Wire Line
-	1275 1375 1275 1425
-Connection ~ 1275 1425
-Wire Wire Line
-	1395 1175 1275 1175
-Wire Wire Line
-	1395 1175 1395 1525
-Connection ~ 1395 1175
+Text GLabel 2420 1425 0    50   Input ~ 0
+OSC
 $EndSCHEMATC

Commit message: Rescued the Libaries
Parts:
- U17: symbol ArmBoard_Hardware-rescue:TB67H400AFNG,EL-MRDT_ICs -> MRDT_ICs:TB67H400AFNG,EL
Changed lines of the file:
@@
 	3760 4325 3760 4200
 $Comp
-L ArmBoard_Hardware-rescue:TB67H400AFNG,EL-MRDT_ICs U?
+L MRDT_ICs:TB67H400AFNG,EL U?
 U 1 1 62489598
 P 3760 2775
 AR Path="/63845F20/62489598" Ref="U?"  Part="1"
 AR Path="/63845F62/62489598" Ref="U17"  Part="1"
+AR Path="/62489598" Ref="U17"  Part="1"
 F 0 "U17" H 3760 4390 50  0000 C CNN
 F 1 "TB67H400AFNG,EL" H 3760 4299 50  0000 C CNN
