File: Hardware/ArmBoard_Hardware/Motor_Controller7.sch (KiCad schematic (older format))
At the start: 14 parts

Commit message: rev 2 finishing passes
Parts:
- gave numbers to parts that had none: 1
Changed lines of the file:
@@
 AR Path="/62D2CE1B/621FCE8E" Ref="#PWR?"  Part="1"
 AR Path="/62D4BAA1/621FCE8E" Ref="#PWR?"  Part="1"
-F 0 "#PWR?" H 4440 3800 50  0001 C CNN
+AR Path="/62C19165/621FCE8E" Ref="#PWR014"  Part="1"
+F 0 "#PWR014" H 4440 3800 50  0001 C CNN
 F 1 "GND" H 4445 3877 50  0000 C CNN
 F 2 "" H 4440 4050 50  0001 C CNN
@@
 AR Path="/62A5CC46/621FCE94" Ref="1k?"  Part="1"
 AR Path="/62AF9C52/621FCE94" Ref="1k?"  Part="1"
-AR Path="/62C19165/621FCE94" Ref="1k?"  Part="1"
+AR Path="/62C19165/621FCE94" Ref="1k42"  Part="1"
 AR Path="/62CA8FD7/621FCE94" Ref="1k?"  Part="1"
 AR Path="/62CBA1AC/621FCE94" Ref="1k?"  Part="1"
@@
 AR Path="/62D3BCB9/621FCE94" Ref="1k?"  Part="1"
 AR Path="/62D4BAA1/621FCE94" Ref="1k?"  Part="1"
-F 0 "1k?" V 4486 4050 50  0000 C CNN
+F 0 "1k42" V 4486 4050 50  0000 C CNN
 F 1 "R_Small" V 4485 4050 50  0001 C CNN
 F 2 "Resistor_SMD:R_0603_1608Metric_Pad0.98x0.95mm_HandSolder" H 4590 4050 50  0001 C CNN

Commit message: gerbs added and zipped
Parts:
- MC7: symbol ArmBoard_Hardware-rescue:VNH5019A_E-MRDT_ICs -> MRDT_ICs:VNH5019A_E
Changed lines of the file:
@@
 IN_A_7
 $Comp
-L ArmBoard_Hardware-rescue:VNH5019A_E-MRDT_ICs U?
+L MRDT_ICs:VNH5019A_E U?
 U 1 1 62E6C738
 P 4925 4600
