File: Hardware/Armboard_Hardware.kicad_pcb (KiCad board)
At the start: 2 copper layers, 142.7 x 155.4 mm, 315 parts, among them J1 RJ45_LED_Shielded, Q1 SI4156DY, Q10 SI4156DY, Q11 SI4156DY, Q12 SI4156DY, Q13 SI4156DY, Q14 SI4156DY, Q15 SI4156DY, Q16 SI4156DY, Q17 SI4156DY, Q18 SI4156DY, Q19 SI4156DY, Q2 SI4156DY, Q20 SI4156DY, Q21 SI4156DY, Q22 SI4156DY, Q23 SI4156DY, Q24 SI4156DY, Q25 SI4156DY, Q26 SI4156DY, Q27 SI4156DY, Q28 SI4156DY, Q29 BSS138, Q3 SI4156DY, Q30 SI4156DY, Q31 SI4156DY, Q32 SI4156DY, Q33 SI4156DY, Q34 SI4156DY, Q35 SI4156DY, Q36 SI4156DY, Q37 SI4156DY, Q4 SI4156DY, Q5 SI4156DY, Q6 SI4156DY, Q7 SI4156DY, Q8 SI4156DY, Q9 SI4156DY, SW1 SW_Push, SW10 SW_SPDT, SW2 SW_Push, SW3 SW_Push, SW4 SW_Push, SW5 SW_Push, SW6 SW_Push, SW7 SW_Push, SW8 SW_Push, SW9 SW_Push, U1 Teensy4.1_DEV-16771, U10 IRS2005S, U11 IRS2005S, U12 IRS2005S, U13 IRS2005S, U14 OKI, U15 IRS2005S, U16 IRS2005S, U17 IRS2005S, U18 IRS2005S, U19 IRS2005S, U2 IRS2005S, U20 IRS2005S, U21 74LVC2G04, U22 74LVC2G04, U23 74LVC2G04, U24 74LVC2G04, U25 74LVC2G04, U26 74LVC2G04, U27 74LVC2G04, U28 74LVC2G04, U29 74LVC2G04, U3 IRS2005S, U30 74HC148, U31 74HC148, U32 74HC00, U4 IRS2005S, U5 IRS2005S, U6 IRS2005S, U7 IRS2005S, U8 IRS2005S, U9 IRS2005S

Commit message: Fixed incorrect capacitor value
Parts:
- C33: value 110uF -> 100uF
Changed lines of the file:
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@@
       (effects (font (size 1 1) (thickness 0.15)))
     )
-    (fp_text value "110uF" (at 1.25 0 90) (layer "F.Fab")
+    (fp_text value "100uF" (at 1.25 0 90) (layer "F.Fab")
       (effects (font (size 1 1) (thickness 0.15)))
     )
